File: kicad/F-3188_CSR8645_breadbord_Adapter/F-3188_CSR8645_breadbord_Adapter.kicad_pcb (KiCad board)
At the start: 2 copper layers, 23.9 x 56.9 mm, 4 parts, among them J1 SCJ368R1NUS0B00G, P1 CONN_01X22, P2 CONN_01X21, U1 F-3188_CSR8645

Commit message: update
Other:
- board text added: "10"
- board text added: "11"
- board text added: "12"
- board text added: "18"
- board text added: "19"
- board text added: "1V8"
- board text added: "20"
- board text added: "21"
- board text added: "6"
- board text added: "7"
- board text added: "8"
- board text added: "9"
- board text added: "AGND"
- board text added: "AIO0"
- board text added: "AN"
- board text added: "AP"
- board text added: "BAT"
- board text added: "BAT SENSE"
- board text added: "BIAS"
- board text added: "BN"
- board text added: "BP"
- board text added: "CHG_EXT"
- board text added: "CLK"
- board text added: "CSB"
- board text added: "GND"
- board text added: "LED0"
- board text added: "LED1"
- board text added: "LED2"
- board text added: "LN"
- board text added: "LP"
- board text added: "MIC"
- board text added: "MISO"
- board text added: "MOSI"
- board text added: "PCM"
- board text added: "PIO"
- board text added: "PIO13"
- board text added: "POWER_RN"
- board text added: "RN"
- board text added: "RP"
- board text added: "RST#"
- board text added: "RX"
- board text added: "SPI"
- board text added: "SPK"
- board text added: "TX"
- board text added: "USB _P _N"
- board text added: "VBUS"
Changed lines of the file:
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@@
-(kicad_pcb (version 20160815) (host pcbnew 4.1.0-alpha+201608211231+7083~46~ubuntu16.04.1-product)
+(kicad_pcb (version 20170123) (host pcbnew no-vcs-found-9447181~59~ubuntu16.04.1)
   (general
-    (links 46)
-    (no_connects 0)
-    (area 132.766999 66.726999 156.843801 123.747601)
     (thickness 1.6)
-    (drawings 4)
+    (drawings 56)
     (tracks 307)
     (zones 0)
@@
     (zone_45_only yes)
     (trace_min 0.2)
-    (segment_width 0.2)
+    (segment_width 0.1)
     (edge_width 0.15)
     (via_size 0.6)
@@
     (uvia_dia 0.3)
     (uvia_drill 0.1)
-    (diff_pair_gap 0.25)
-    (diff_pair_width 0.2)
     (add_net /GND)
     (add_net "Net-(J1-Pad1)")
@@
     (descr "Through hole pin header")
     (tags "pin header")
-    (fp_text reference P1 (at 0 -5.1) (layer F.SilkS)
+    (fp_text reference P1 (at 0 -5.1) (layer F.SilkS) hide
       (effects (font (size 1 1) (thickness 0.15)))
     )
-    (fp_text value CONN_01X22 (at 0 -3.1) (layer F.Fab)
+    (fp_text value CONN_01X22 (at 0 -3.1) (layer F.Fab) hide
       (effects (font (size 1 1) (thickness 0.15)))
     )
@@
     (descr "Through hole pin header")
     (tags "pin header")
-    (fp_text reference P2 (at 0 -5.1) (layer F.SilkS)
+    (fp_text reference P2 (at 0 -5.1) (layer F.SilkS) hide
       (effects (font (size 1 1) (thickness 0.15)))
     )
-    (fp_text value CONN_01X21 (at 0 -3.1) (layer F.Fab)
+    (fp_text value CONN_01X21 (at 0 -3.1) (layer F.Fab) hide
       (effects (font (size 1 1) (thickness 0.15)))
     )
@@
     (pad "" np_thru_hole circle (at -5 0) (size 1.5 1.5) (drill 1.5) (layers *.Cu *.Mask B.SilkS))
   )
+  (gr_text AGND (at 150.114 68.58) (layer B.SilkS)
+    (effects (font (size 1.5 1.5) (thickness 0.3)) (justify mirror))
+  )
+  (gr_line (start 149.352 70.104) (end 149.352 79.502) (layer B.SilkS) (width 0.1))
+  (gr_text SPK (at 148.082 74.93 90) (layer B.SilkS)
+    (effects (font (size 1.5 1.5) (thickness 0.3)) (justify mirror))
+  )
+  (gr_text LP (at 151.13 71.12) (layer B.SilkS)
+    (effects (font (size 1.5 1.5) (thickness 0.3)) (justify mirror))
+  )
+  (gr_text LN (at 151.13 73.66) (layer B.SilkS)
+    (effects (font (size 1.5 1.5) (thickness 0.3)) (justify mirror))
+  )
+  (gr_text RP (at 151.13 76.2) (layer B.SilkS)
+    (effects (font (size 1.5 1.5) (thickness 0.3)) (justify mirror))
+  )
+  (gr_text RN (at 151.13 78.486) (layer B.SilkS)
+    (effects (font (size 1.5 1.5) (thickness 0.3)) (justify mirror))
+  )
+  (gr_text MIC (at 147.32 85.852 90) (layer B.SilkS)
+    (effects (font (size 1.5 1.5) (thickness 0.3)) (justify mirror))
+  )
+  (gr_line (start 148.336 80.264) (end 148.336 92.202) (layer B.SilkS) (width 0.1))
+  (gr_text BP (at 151.13 81.28) (layer B.SilkS)
+    (effects (font (size 1.5 1.5) (thickness 0.3)) (justify mirror))
+  )
+  (gr_text BN (at 151.13 83.82) (layer B.SilkS)
+    (effects (font (size 1.5 1.5) (thickness 0.3)) (justify mirror))
+  )
+  (gr_text AP (at 151.13 86.106) (layer B.SilkS)
+    (effects (font (size 1.5 1.5) (thickness 0.3)) (justify mirror))
+  )
+  (gr_text AN (at 151.13 88.9) (layer B.SilkS)
+    (effects (font (size 1.5 1.5) (thickness 0.3)) (justify mirror))
+  )
+  (gr_line (start 142.24 77.47) (end 142.24 89.916) (layer B.SilkS) (width 0.1))
+  (gr_text SPI (at 143.51 83.82 90) (layer B.SilkS)
+    (effects (font (size 1.5 1.5) (thickness 0.3)) (justify mirror))
+  )
+  (gr_line (start 151.13 93.218) (end 151.384 111.76) (layer B.SilkS) (width 0.1))
+  (gr_text PIO (at 150.114 103.886 90) (layer B.SilkS)
+    (effects (font (size 0.8 0.8) (thickness 0.1)) (justify mirror))
+  )
+  (gr_text BIAS (at 151.13 91.44) (layer B.SilkS)
+    (effects (font (size 1.5 1.5) (thickness 0.3)) (justify mirror))
+  )
+  (gr_text 21 (at 152.4 93.98) (layer B.SilkS)
+    (effects (font (size 1 1) (thickness 0.1)) (justify mirror))
+  )
+  (gr_text 20 (at 152.4 96.52) (layer B.SilkS)
+    (effects (font (size 1 1) (thickness 0.1)) (justify mirror))
+  )
+  (gr_text 19 (at 152.4 99.06) (layer B.SilkS)
+    (effects (font (size 1 1) (thickness 0.1)) (justify mirror))
+  )
+  (gr_text 18 (at 152.4 101.6) (layer B.SilkS)
+    (effects (font (size 1 1) (thickness 0.1)) (justify mirror))
+  )
+  (gr_text 8 (at 152.4 104.14) (layer B.SilkS)
+    (effects (font (size 1 1) (thickness 0.1)) (justify mirror))
+  )
+  (gr_text 7 (at 152.4 106.68) (layer B.SilkS)
+    (effects (font (size 1 1) (thickness 0.1)) (justify mirror))
+  )
+  (gr_text 6 (at 152.4 109.22) (layer B.SilkS)
+    (effects (font (size 1 1) (thickness 0.1)) (justify mirror))
+  )
+  (gr_text 9 (at 152.4 111.76) (layer B.SilkS)
+    (effects (font (size 1 1) (thickness 0.1)) (justify mirror))
+  )
+  (gr_text "USB\n_P\n_N" (at 152.654 114.808) (layer B.SilkS)
+    (effects (font (size 1 1) (thickness 0.1)) (justify mirror))
+  )
+  (gr_text PIO13 (at 153.924 121.412) (layer B.SilkS)
+    (effects (font (size 1 1) (thickness 0.1)) (justify mirror))
+  )
+  (gr_line (start 136.906 123.19) (end 136.906 115.824) (layer B.SilkS) (width 0.1))
+  (gr_text PIO (at 136.398 119.38 90) (layer B.SilkS)
+    (effects (font (size 0.8 0.8) (thickness 0.1)) (justify mirror))
+  )
+  (gr_text 12 (at 137.922 121.92) (layer B.SilkS)
+    (effects (font (size 1 1) (thickness 0.1)) (justify mirror))
+  )
+  (gr_text 11 (at 137.922 119.38) (layer B.SilkS)
+    (effects (font (size 1 1) (thickness 0.1)) (justify mirror))
+  )
+  (gr_text 10 (at 137.922 116.84) (layer B.SilkS)
+    (effects (font (size 1 1) (thickness 0.1)) (justify mirror))
+  )
+  (gr_text "BAT\nSENSE" (at 137.414 114.3) (layer B.SilkS)
+    (effects (font (size 0.8 0.8) (thickness 0.1)) (justify mirror))
+  )
+  (gr_text CHG_EXT (at 140.716 110.998) (layer B.SilkS)
+    (effects (font (size 1.5 1.5) (thickness 0.3)) (justify mirror))
+  )
+  (gr_text GND (at 138.684 108.966) (layer B.SilkS)
+    (effects (font (size 1.5 1.5) (thickness 0.3)) (justify mirror))
+  )
+  (gr_text 1V8 (at 138.684 106.426) (layer B.SilkS)
+    (effects (font (size 1.5 1.5) (thickness 0.3)) (justify mirror))
+  )
+  (gr_text POWER_RN (at 141.732 104.14) (layer B.SilkS)
+    (effects (font (size 1.5 1.5) (thickness 0.3)) (justify mirror))
+  )
+  (gr_text BAT (at 138.684 101.6) (layer B.SilkS)
+    (effects (font (size 1.5 1.5) (thickness 0.3)) (justify mirror))
+  )
+  (gr_text RST# (at 138.684 99.06) (layer B.SilkS)
+    (effects (font (size 1.5 1.5) (thickness 0.3)) (justify mirror))
+  )
+  (gr_text VBUS (at 138.684 96.52) (layer B.SilkS)
+    (effects (font (size 1.5 1.5) (thickness 0.3)) (justify mirror))
+  )
+  (gr_text RX (at 138.938 93.98) (layer B.SilkS)
+    (effects (font (size 1.5 1.5) (thickness 0.3)) (justify mirror))
+  )
+  (gr_text TX (at 138.938 91.44) (layer B.SilkS)
+    (effects (font (size 1.5 1.5) (thickness 0.3)) (justify mirror))
+  )
+  (gr_text PCM (at 139.446 88.9) (layer B.SilkS)
+    (effects (font (size 1.5 1.5) (thickness 0.3)) (justify mirror))
+  )
+  (gr_text MOSI (at 138.938 86.36) (layer B.SilkS)
+    (effects (font (size 1.5 1.5) (thickness 0.3)) (justify mirror))
+  )
+  (gr_text CLK (at 139.192 83.566) (layer B.SilkS)
+    (effects (font (size 1.5 1.5) (thickness 0.3)) (justify mirror))
+  )
+  (gr_text CSB (at 138.938 81.28) (layer B.SilkS)
+    (effects (font (size 1.5 1.5) (thickness 0.3)) (justify mirror))
+  )
+  (gr_text MISO (at 138.938 78.74) (layer B.SilkS)
+    (effects (font (size 1.5 1.5) (thickness 0.3)) (justify mirror))
+  )
+  (gr_text AIO0 (at 139.192 76.2) (layer B.SilkS)
+    (effects (font (size 1.5 1.5) (thickness 0.3)) (justify mirror))
+  )
+  (gr_text LED0 (at 139.192 73.66) (layer B.SilkS)
+    (effects (font (size 1.5 1.5) (thickness 0.3)) (justify mirror))
+  )
+  (gr_text LED1 (at 139.192 71.12) (layer B.SilkS)
+    (effects (font (size 1.5 1.5) (thickness 0.3)) (justify mirror))
+  )
+  (gr_text LED2 (at 139.192 68.58) (layer B.SilkS)
+    (effects (font (size 1.5 1.5) (thickness 0.3)) (justify mirror))
+  )
   (gr_line (start 132.842 66.802) (end 156.7688 66.802) (angle 90) (layer Edge.Cuts) (width 0.15))
