File: kicad/F-3188_CSR8645_breadbord_Adapter/F-3188_CSR8645_breadbord_Adapter.sch (KiCad schematic (older format))
At the start: 4 parts, among them J1 SCJ368R1NUS0B00G, P1 CONN_01X22, P2 CONN_01X21, U1 F-3188_CSR8645

Commit message: update
Parts:
- added D1, D2: LED1, LEDs:LED_1206, symbol LED
- added J2: ON, Connectors:GS2, symbol GS2
- added R1, R2: 10k, Resistors_SMD:R_0805, symbol R
- added R3, R4: 1k, Resistors_SMD:R_0805, symbol R
- added SW1: RESET, Buttons_Switches_SMD:SW_SPST_FSMSM, symbol SW_Push
- added SW2: POWER_ON, Buttons_Switches_SMD:SW_SPST_FSMSM, symbol SW_Push
Connections:
- net GND: now also SW1.2
- net RST#: now reaches P1.13 (P13), U1.13 (RST#)
- net RST#: now also R1.2, SW1.1
- net BAT: now reaches P1.14 (P14), U1.14 (BAT)
- net BAT: now also R1.1, R2.1, R3.1, R4.1
- net POWER_ON: now reaches P1.15 (P15), U1.15 (POWER_RN)
- net POWER_ON: now also J2.1 (G1), SW2.2
- net LED1: now reaches P1.2 (P2), U1.2 (LED1)
- net LED1: now also D1.1 (K)
- net LED0: now reaches P1.3 (P3), U1.3 (LED0)
- net LED0: now also D2.1 (K)
- net HL: now reaches J1.2, P2.4 (P4), U1.40 (SPK_R_P1)
- net HL: now also J1.3
- net HGND: now reaches J1.1, P2.3 (P3), U1.41 (SPK_L_N1)
- net HR: now reaches J1.5, P2.2 (P2), U1.42 (SPK_L_P1)
- net HR: now also J1.4
- new net: D2.2 (A), R4.2
- new net: D1.2 (A), R3.2
- new net: J2.2 (G2), R2.2, SW2.1
Other:
- moved on the sheet: J1
