File: kicad/MB-CM15113-btm-68D_breakout_adapter/MB-CM15113-btm-68D_breakout_adapter.sch (KiCad schematic (older format))
At the start: 12 parts, among them P1 CONN_01X16, P2 CONN_01X05, P3 CONN_01X16, U1 MB-CM15113

Commit message: update
Parts:
- added C1: 15pF, Capacitors_SMD:C_0805_HandSoldering, symbol C
- added C2: 100n, Capacitors_SMD:C_0805_HandSoldering, symbol C
- added L1: 15nH, Choke_SMD:Choke_SMD_1206_Standard, symbol L
- P1, P3: value CONN_01X16 -> CONN_01X15; footprint Pin_Headers:Pin_Header_Straight_1x16 -> Pin_Headers:Pin_Header_Straight_1x15_Pitch2.54mm; symbol CONN_01X16 -> CONN_01X15
- SW1: renamed from SW?; value SW_PUSH -> RESET
- SW2: renamed from SW?; value SW_PUSH -> ON/OFF
- gave numbers to parts that had none: 6
Connections:
- net labels added: GND
- wire segments 54 -> 77
