File: kicad/MB-CM15113-btm-68D_breakout_adapter/MB-CM15113-btm-68D_breakout_adapter.sch (KiCad schematic (older format))
At the start: 15 parts, among them P1 CONN_01X15, P2 CONN_01X05, P3 CONN_01X15, SW1 RESET, SW2 ON/OFF, U1 MB-CM15113

Commit message: update
Parts:
- C1, C2: symbol C -> MB-CM15113-btm-68D_breakout_adapter-rescue:C
- D1, D2: symbol D -> MB-CM15113-btm-68D_breakout_adapter-rescue:D
- L1: symbol L -> MB-CM15113-btm-68D_breakout_adapter-rescue:L
- P1, P3: symbol CONN_01X15 -> MB-CM15113-btm-68D_breakout_adapter-rescue:CONN_01X15
- P2: symbol CONN_01X05 -> MB-CM15113-btm-68D_breakout_adapter-rescue:CONN_01X05
- R1, R2, R3, R4: symbol R -> MB-CM15113-btm-68D_breakout_adapter-rescue:R
- SW1, SW2: symbol SW_PUSH -> MB-CM15113-btm-68D_breakout_adapter-rescue:SW_PUSH
- U1: symbol MB-CM15113 -> MB-CM15113-btm-68D_breakout_adapter-rescue:MB-CM15113
Changed lines of the file:
@@
-EESchema Schematic File Version 2
-LIBS:power
-LIBS:device
-LIBS:transistors
-LIBS:conn
-LIBS:linear
-LIBS:regul
-LIBS:74xx
-LIBS:cmos4000
-LIBS:adc-dac
-LIBS:memory
-LIBS:xilinx
-LIBS:microcontrollers
-LIBS:dsp
-LIBS:microchip
-LIBS:analog_switches
-LIBS:motorola
-LIBS:texas
-LIBS:intel
-LIBS:audio
-LIBS:interface
-LIBS:digital-audio
-LIBS:philips
-LIBS:display
-LIBS:cypress
-LIBS:siliconi
-LIBS:opto
-LIBS:atmel
-LIBS:contrib
-LIBS:valves
-LIBS:MB-CM15113
-LIBS:audio_source-cache
+EESchema Schematic File Version 4
 LIBS:MB-CM15113-btm-68D_breakout_adapter-cache
-EELAYER 26 0
+EELAYER 29 0
 EELAYER END
 $Descr A4 11693 8268
@@
 $EndDescr
 $Comp
-L MB-CM15113 U1
+L MB-CM15113-btm-68D_breakout_adapter-rescue:MB-CM15113 U1
 U 1 1 55EC62E4
 P 5500 2850
@@
 $EndComp
 $Comp
-L CONN_01X15 P1
+L MB-CM15113-btm-68D_breakout_adapter-rescue:CONN_01X15 P1
 U 1 1 55EC634B
 P 4050 2850
@@
 $EndComp
 $Comp
-L CONN_01X15 P3
+L MB-CM15113-btm-68D_breakout_adapter-rescue:CONN_01X15 P3
 U 1 1 55EC639E
 P 8300 2850
@@
 $EndComp
 $Comp
-L CONN_01X05 P2
+L MB-CM15113-btm-68D_breakout_adapter-rescue:CONN_01X05 P2
 U 1 1 55EC6792
 P 6450 1650
@@
 $EndComp
 $Comp
-L R R2
+L MB-CM15113-btm-68D_breakout_adapter-rescue:R R2
 U 1 1 57ECF44A
 P 6300 4300
@@
 $EndComp
 $Comp
-L R R3
+L MB-CM15113-btm-68D_breakout_adapter-rescue:R R3
 U 1 1 57ECF4C4
 P 6600 4300
@@
 $EndComp
 $Comp
-L D D1
+L MB-CM15113-btm-68D_breakout_adapter-rescue:D D1
 U 1 1 57ECF6CA
 P 6300 3900
@@
 $EndComp
 $Comp
-L D D2
+L MB-CM15113-btm-68D_breakout_adapter-rescue:D D2
 U 1 1 57ECF843
 P 6600 3900
@@
 $EndComp
 $Comp
-L SW_PUSH SW2
+L MB-CM15113-btm-68D_breakout_adapter-rescue:SW_PUSH SW2
 U 1 1 57ED00C6
 P 7050 4150
@@
 $EndComp
 $Comp
-L R R4
+L MB-CM15113-btm-68D_breakout_adapter-rescue:R R4
 U 1 1 57ED0215
 P 7300 4300
@@
 $EndComp
 $Comp
-L SW_PUSH SW1
+L MB-CM15113-btm-68D_breakout_adapter-rescue:SW_PUSH SW1
 U 1 1 57ED066C
 P 4400 4150
@@
 $EndComp
 $Comp
-L R R1
+L MB-CM15113-btm-68D_breakout_adapter-rescue:R R1
 U 1 1 57ED0675
 P 4650 4300
@@
 $EndComp
 $Comp
-L L L1
+L MB-CM15113-btm-68D_breakout_adapter-rescue:L L1
 U 1 1 599EED00
 P 7550 2650
@@
 $EndComp
 $Comp
-L C C1
+L MB-CM15113-btm-68D_breakout_adapter-rescue:C C1
 U 1 1 599EF23C
 P 7250 1900
@@
 $EndComp
 $Comp
-L C C2
+L MB-CM15113-btm-68D_breakout_adapter-rescue:C C2
 U 1 1 599EFBD4
 P 7850 4000
@@
 $EndComp
 $Comp
-L GND #PWR01
+L power1:GND #PWR01
 U 1 1 599F0545
 P 4200 3950
@@
 	4250 3050 4750 3050
 Wire Wire Line
-	4750 3150 4250 3150
-Wire Wire Line
-	6200 3250 8100 3250
-Wire Wire Line
-	6200 3150 8100 3150
-Wire Wire Line
-	6200 3050 8100 3050
-Wire Wire Line
-	6200 2950 8100 2950
+	4750 3150 4650 3150
+Wire Wire Line
+	6200 3250 6300 3250
+Wire Wire Line
+	6200 3150 6600 3150
+Wire Wire Line
+	6200 3050 7050 3050
+Wire Wire Line
+	6200 2950 6450 2950
 Wire Wire Line
 	6200 2850 8100 2850
@@
 	6200 2750 8100 2750
 Wire Wire Line
-	6200 2550 8100 2550
+	6200 2550 6650 2550
 Wire Wire Line
 	6200 2450 8100 2450
 Wire Wire Line
-	6200 2350 8100 2350
+	6200 2350 6550 2350
 Wire Wire Line
 	6200 2250 8100 2250
@@
 	6300 4450 6300 4550
 Wire Wire Line
-	6300 4550 6600 4550
+	6300 4550 6450 4550
 Wire Wire Line
 	6600 4550 6600 4450
@@
 	4400 4450 4400 4550
 Wire Wire Line
-	4400 4550 4650 4550
+	4400 4550 4500 4550
 Wire Wire Line
 	4650 4550 4650 4450
@@
 Connection ~ 4500 3550
 Wire Wire Line
-	6200 2150 8100 2150
+	6200 2150 6250 2150
 Connection ~ 6250 2150
 Wire Wire Line
 	7700 2650 8100 2650
 Wire Wire Line
-	7400 2650 6200 2650
+	7400 2650 7250 2650
 Wire Wire Line
 	7250 2050 7250 2650
@@
 Connection ~ 7850 2950
 Wire Wire Line
-	7650 3350 7650 4300
+	7650 3350 7650 3800
 Wire Wire Line
 	7650 4300 7850 4300
@@
 	4200 3950 4200 3800
 Wire Wire Line
-	4200 3800 7650 3800
-Wire Wire Line
-	4750 3250 4250 3250
+	4200 3800 4400 3800
+Wire Wire Line
+	4750 3250 4700 3250
 Wire Wire Line
 	4250 3350 4600 3350
@@
 Connection ~ 4700 3250
 Wire Wire Line
-	4750 3550 4450 3550
+	4750 3550 4500 3550
 Wire Wire Line
 	4450 3550 4450 3450
@@
 	4350 3650 4750 3650
 Wire Wire Line
-	4400 3250 4400 3850
+	4400 3250 4400 3800
 Connection ~ 4400 3800
 Connection ~ 4400 3250
@@
 Wire Wire Line
 	7900 3450 6200 3450
+Wire Wire Line
+	6650 2550 7000 2550
+Wire Wire Line
+	6550 2350 8100 2350
+Wire Wire Line
+	6300 3250 8100 3250
+Wire Wire Line
+	6600 3150 8100 3150
+Wire Wire Line
+	6450 2950 7300 2950
+Wire Wire Line
+	6450 4550 6600 4550
+Wire Wire Line
+	7050 3050 8100 3050
+Wire Wire Line
+	7300 2950 7850 2950
+Wire Wire Line
+	4650 3150 4250 3150
+Wire Wire Line
+	4500 4550 4650 4550
+Wire Wire Line
+	4500 3550 4450 3550
+Wire Wire Line
+	6250 2150 8100 2150
+Wire Wire Line
+	7250 2650 6200 2650
+Wire Wire Line
+	7000 2550 8100 2550
+Wire Wire Line
+	7850 2950 8100 2950
+Wire Wire Line
+	4700 3250 4400 3250
+Wire Wire Line
+	4400 3800 7650 3800
+Wire Wire Line
+	4400 3800 4400 3850
+Wire Wire Line
+	4400 3250 4250 3250
+Wire Wire Line
+	7650 3800 7650 4300
 $EndSCHEMATC
