File: kicad/S3860M-S_breadboard_adapter/S3860M-S_breadboard_adapter.sch (KiCad schematic (older format))
At the start: 11 parts, among them J1 SCJ368R1NUS0B00G, P1 CONN_01X12, P2 CONN_01X12, U1 S3860M-S

Commit message: to fcking much changes to commit it separatly, lets go with everything in one commit, git will love me for sure :D
Parts:
- added C1: 100n, Capacitors_SMD.pretty:C_1206_HandSoldering, symbol c:C
- D1, D2: symbol LED-RESCUE-S3860M-S_breadboard_adapter -> S3860M-S_breadboard_adapter-rescue:LED-RESCUE-S3860M-S_breadboard_adapter
- J1: symbol SCJ368R1NUS0B00G -> phonejack:SCJ368R1NUS0B00G
- ON/OFF/PLAY1, RESET1: symbol SW_PUSH -> S3860M-S_breadboard_adapter-rescue:SW_PUSH-RESCUE-S3860M-S_breadboard_adapter
- P1: symbol CONN_01X12 -> S3860M-S_breadboard_adapter-rescue:CONN_01X12-RESCUE-S3860M-S_breadboard_adapter
- P2: symbol CONN_01X11 -> S3860M-S_breadboard_adapter-rescue:CONN_01X11-RESCUE-S3860M-S_breadboard_adapter
- R1, R2, R3: symbol R -> S3860M-S_breadboard_adapter-rescue:R-RESCUE-S3860M-S_breadboard_adapter
- U1: symbol S3860M-S -> S3860M-S_breadboard_adapter-rescue:S3860M-S-RESCUE-S3860M-S_breadboard_adapter
Connections:
- net labels added: GND
- wire segments 63 -> 82
Changed lines of the file:
@@
-EESchema Schematic File Version 2
-LIBS:S3860M-S_breadboard_adapter-rescue
-LIBS:power
-LIBS:device
-LIBS:transistors
-LIBS:conn
-LIBS:linear
-LIBS:regul
-LIBS:74xx
-LIBS:cmos4000
-LIBS:adc-dac
-LIBS:memory
-LIBS:xilinx
-LIBS:microcontrollers
-LIBS:dsp
-LIBS:microchip
-LIBS:analog_switches
-LIBS:motorola
-LIBS:texas
-LIBS:intel
-LIBS:audio
-LIBS:interface
-LIBS:digital-audio
-LIBS:philips
-LIBS:display
-LIBS:cypress
-LIBS:siliconi
-LIBS:opto
-LIBS:atmel
-LIBS:contrib
-LIBS:valves
-LIBS:phonejack
-LIBS:SOYO-BT24G03
-LIBS:S3860M-S
-LIBS:open-project
+EESchema Schematic File Version 4
 LIBS:S3860M-S_breadboard_adapter-cache
 EELAYER 26 0
@@
 $EndDescr
 $Comp
-L S3860M-S U1
+L S3860M-S_breadboard_adapter-rescue:S3860M-S-RESCUE-S3860M-S_breadboard_adapter U1
 U 1 1 5576DBD3
 P 5650 3750
@@
 $EndComp
 $Comp
-L SCJ368R1NUS0B00G J1
+L phonejack:SCJ368R1NUS0B00G J1
 U 1 1 5576DC76
 P 5650 2550
@@
 $EndComp
 $Comp
-L CONN_01X11 P2
+L S3860M-S_breadboard_adapter-rescue:CONN_01X11-RESCUE-S3860M-S_breadboard_adapter P2
 U 1 1 5576DF5A
 P 9300 3800
@@
 $EndComp
 $Comp
-L SW_PUSH RESET1
+L S3860M-S_breadboard_adapter-rescue:SW_PUSH-RESCUE-S3860M-S_breadboard_adapter RESET1
 U 1 1 56C45A37
 P 5400 4950
@@
 $EndComp
 $Comp
-L R R1
+L S3860M-S_breadboard_adapter-rescue:R-RESCUE-S3860M-S_breadboard_adapter R1
 U 1 1 56C47B10
 P 5400 5200
@@
 $EndComp
 $Comp
-L SW_PUSH ON/OFF/PLAY1
+L S3860M-S_breadboard_adapter-rescue:SW_PUSH-RESCUE-S3860M-S_breadboard_adapter ON/OFF/PLAY1
 U 1 1 56C4875B
 P 5700 5700
@@
 $EndComp
 $Comp
-L R R2
+L S3860M-S_breadboard_adapter-rescue:R-RESCUE-S3860M-S_breadboard_adapter R2
 U 1 1 56C48674
 P 5550 5850
@@
 $EndComp
 $Comp
-L R R3
+L S3860M-S_breadboard_adapter-rescue:R-RESCUE-S3860M-S_breadboard_adapter R3
 U 1 1 56C48760
 P 5550 6150
@@
 $EndComp
 $Comp
-L LED-RESCUE-S3860M-S_breadboard_adapter D1
+L S3860M-S_breadboard_adapter-rescue:LED-RESCUE-S3860M-S_breadboard_adapter D1
 U 1 1 56C487CC
 P 6100 5850
@@
 $EndComp
 $Comp
-L LED-RESCUE-S3860M-S_breadboard_adapter D2
+L S3860M-S_breadboard_adapter-rescue:LED-RESCUE-S3860M-S_breadboard_adapter D2
 U 1 1 56C488F4
 P 6100 6150
@@
 $EndComp
 $Comp
-L CONN_01X12 P1
+L S3860M-S_breadboard_adapter-rescue:CONN_01X12-RESCUE-S3860M-S_breadboard_adapter P1
 U 1 1 5576DE6D
 P 3400 3850
@@
 	6250 3800 9100 3800
 Wire Wire Line
-	3600 3300 5050 3300
-Wire Wire Line
-	3600 3400 5050 3400
-Wire Wire Line
-	3600 3500 5050 3500
+	3600 3300 4900 3300
+Wire Wire Line
+	3600 3400 4950 3400
+Wire Wire Line
+	3600 3500 5000 3500
 Wire Wire Line
 	3600 3600 5050 3600
@@
 	3600 3700 5050 3700
 Wire Wire Line
-	3600 3800 5050 3800
-Wire Wire Line
-	3600 3900 5050 3900
+	3600 3800 4850 3800
+Wire Wire Line
+	3600 3900 4800 3900
 Wire Wire Line
 	3600 4000 5050 4000
@@
 	5400 5700 5000 5700
 Wire Wire Line
-	5000 4400 5000 6500
+	5000 4400 5000 5700
 Connection ~ 5000 4400
 Wire Wire Line
@@
 	6300 5850 6400 5850
 Wire Wire Line
-	6400 5850 6400 6500
+	6400 5850 6400 6150
 Wire Wire Line
 	6400 6150 6300 6150
@@
 	5250 5200 4950 5200
 Wire Wire Line
-	5700 4950 9000 4950
+	5700 4950 5800 4950
 Wire Wire Line
 	9000 4950 9000 4000
@@
 Connection ~ 9050 4300
 Wire Wire Line
-	3600 4400 5050 4400
+	3600 4400 5000 4400
 Wire Wire Line
 	4800 6150 4800 3900
@@
 Connection ~ 4850 3800
 Wire Wire Line
-	3600 4300 5050 4300
+	3600 4300 4000 4300
 Wire Wire Line
 	3600 4100 5050 4100
 Wire Wire Line
-	3600 4200 5050 4200
+	3600 4200 3800 4200
 Wire Wire Line
 	9100 3900 6250 3900
@@
 	8250 4100 8250 4000
 Wire Wire Line
-	8250 4000 9100 4000
+	8250 4000 9000 4000
 Wire Wire Line
 	9100 4100 8400 4100
@@
 	8550 4200 9100 4200
 Wire Wire Line
-	8650 4300 9100 4300
+	8650 4300 9050 4300
 Wire Wire Line
 	8650 4400 8650 4300
@@
 	3800 5350 3800 4200
 Connection ~ 3800 4200
+Wire Wire Line
+	5000 3500 5050 3500
+Wire Wire Line
+	4950 3400 5050 3400
+Wire Wire Line
+	4900 3300 5050 3300
+Wire Wire Line
+	4950 4300 5050 4300
+Wire Wire Line
+	5000 4400 5050 4400
+Wire Wire Line
+	5000 5700 5000 6500
+Wire Wire Line
+	6400 6150 6400 6500
+Wire Wire Line
+	5800 4950 9000 4950
+Wire Wire Line
+	9000 4000 9100 4000
+Wire Wire Line
+	9050 4300 9100 4300
+Wire Wire Line
+	4800 3900 5050 3900
+Wire Wire Line
+	4850 3800 5050 3800
+Wire Wire Line
+	3800 4200 4250 4200
+Text Label 4400 4200 0    50   ~ 0
+GND
+$Comp
+L c:C C1
+U 1 1 5A910B1E
+P 4250 4650
+F 0 "C1" H 4379 4703 60  0000 L CNN
+F 1 "100n" H 4379 4597 60  0000 L CNN
+F 2 "Capacitors_SMD.pretty:C_1206_HandSoldering" H 4250 4650 50  0001 C CNN
+F 3 "" H 4250 4650 50  0001 C CNN
+	1    4250 4650
+	1    0    0    -1
+$EndComp
+Wire Wire Line
+	4250 4450 4250 4200
+Connection ~ 4250 4200
+Wire Wire Line
+	4250 4200 5050 4200
+Wire Wire Line
+	4250 4850 4250 4950
+Wire Wire Line
+	4250 4950 4000 4950
+Wire Wire Line
+	4000 4950 4000 4300
+Connection ~ 4000 4300
+Wire Wire Line
+	4000 4300 4950 4300
 $EndSCHEMATC

Commit message: version 2.0
Parts:
- removed J1: SCJ368R1NUS0B00G, jacks:3.5mm_stereo_jack_PJ320B, symbol phonejack:SCJ368R1NUS0B00G
- added C2: 4u7, Capacitors_SMD.pretty:C_1206_HandSoldering, symbol c:C
- added C3: 2u2/6.5V, Capacitors_SMD.pretty:C_0805_HandSoldering, symbol c:C
- added C4: 220p/optional, Capacitors_SMD.pretty:C_0805_HandSoldering, symbol c:C
- added C5, C6, C7: 2u2, Capacitors_SMD.pretty:C_1206_HandSoldering, symbol c:C
- added J1: OUT, jacks:3.5mm_stereo_jack_PJ320B, symbol jacks:PJ-320B
- added J2: MIC, jacks:3.5mm_stereo_jack_PJ320B, symbol jacks:PJ-320B
- added L1: 15n, Choke_SMD.pretty:Choke_SMD_1206_Handsoldering, symbol Device:L
- added R4: 2k2, Resistors_SMD:R_0805_HandSoldering, symbol S3860M-S_breadboard_adapter-rescue:R-RESCUE-S3860M-S_breadboard_adapter
- added R5: 2k, Resistors_SMD:R_0805_HandSoldering, symbol S3860M-S_breadboard_adapter-rescue:R-RESCUE-S3860M-S_breadboard_adapter
- added SW1: PREVIOUS, Buttons_Switches_SMD:SW_SPST_FSMSM, symbol S3860M-S_breadboard_adapter-rescue:SW_PUSH-RESCUE-S3860M-S_breadboard_adapter
- added SW2: NEXT, Buttons_Switches_SMD:SW_SPST_FSMSM, symbol S3860M-S_breadboard_adapter-rescue:SW_PUSH-RESCUE-S3860M-S_breadboard_adapter
- added SW3: VOL-, Buttons_Switches_SMD:SW_SPST_FSMSM, symbol S3860M-S_breadboard_adapter-rescue:SW_PUSH-RESCUE-S3860M-S_breadboard_adapter
- added SW4: VOL+, Buttons_Switches_SMD:SW_SPST_FSMSM, symbol S3860M-S_breadboard_adapter-rescue:SW_PUSH-RESCUE-S3860M-S_breadboard_adapter
- C1: footprint Capacitors_SMD.pretty:C_1206_HandSoldering -> Capacitors_SMD.pretty:C_0805_HandSoldering
- DG1: renamed from D1; value LED -> GREEN
- DR2: renamed from D2; value LED -> RED
- P1: footprint Pin_Headers:Pin_Header_Straight_1x12 -> Pin_Headers:Pin_Header_Straight_1x12_Pitch2.54mm; symbol S3860M-S_breadboard_adapter-rescue:CONN_01X12-RESCUE-S3860M-S_breadboard_adapter -> Connector_Generic:Conn_01x12_Male
- P2: footprint Pin_Headers:Pin_Header_Straight_1x11 -> Pin_Headers:Pin_Header_Straight_1x12_Pitch2.54mm; symbol S3860M-S_breadboard_adapter-rescue:CONN_01X11-RESCUE-S3860M-S_breadboard_adapter -> Connector_Generic:Conn_01x12_Male
- SW6: renamed from RESET1; value 1 -> RESET
- renumbered R2 to R1, R3 to R2, R1 to R3, ON/OFF/PLAY1 to SW5
Connections:
- net labels added: 1V8, AOL, AOM, AOR, LED1, LED2, MFB1, MIC+, MICBIAS, MUTE, NEXT, ONKEY, PREVIOUS, RESET, UART_RX, UART_TX, VBAT, VBUCK, VCC, VOL+, VOL-, VPP
- wire segments 82 -> 79
- no-connect marks 0 -> 1
Other:
- note added: "this is at blk "datasheet"\nI put it here just in case\ns3860-m "datasheet"\nis missing this parts"
- moved on the sheet: C1, DG1, DR2, R1, R2, R3, SW5, SW6, U1

Commit message: update
Parts:
- C5, C6, C7: value 2u2 -> 10uF
- R4: value 2k2 -> 2k
Connections:
- net MIC+: no longer C2.1, L1.1, L1.2
- net MICBIAS: now also C2.1, L1.2; no longer R4.2
- new net: L1.1, R4.2
Other:
- moved on the sheet: C2, L1
Changed lines of the file:
@@
 P 3200 3650
 F 0 "C3" V 3100 3750 60  0000 L CNN
-F 1 "2u2/6.5V" V 2950 3600 60  0000 L CNN
+F 1 "2u2/6.5V" V 3000 3450 60  0000 L CNN
 F 2 "Capacitors_SMD.pretty:C_0805_HandSoldering" H 3200 3650 50  0001 C CNN
 F 3 "" H 3200 3650 50  0001 C CNN
@@
 P 3250 3250
 F 0 "R4" V 3042 3250 50  0000 C CNN
-F 1 "2k2" V 3134 3250 50  0000 C CNN
+F 1 "2k" V 3134 3250 50  0000 C CNN
 F 2 "Resistors_SMD:R_0805_HandSoldering" V 3134 3250 50  0001 C CNN
 F 3 "" H 3250 3250 50  0000 C CNN
@@
 	0    1    1    0
 $EndComp
-Wire Wire Line
-	3100 3250 2300 3250
 Wire Wire Line
 	3400 3650 3700 3650
@@
 Wire Wire Line
 	4100 4050 4200 4050
-Text Label 2300 3250 0    50   ~ 0
+Text Label 1900 3250 0    50   ~ 0
 MICBIAS
 Text Label 1900 3650 0    50   ~ 0
@@
 P 3250 1550
 F 0 "C6" V 3300 1650 60  0000 L CNN
-F 1 "2u2" V 3300 1300 60  0000 L CNN
+F 1 "10uF" V 3300 1300 60  0000 L CNN
 F 2 "Capacitors_SMD.pretty:C_1206_HandSoldering" H 3250 1550 50  0001 C CNN
 F 3 "" H 3250 1550 50  0001 C CNN
@@
 P 3250 1750
 F 0 "C7" V 3300 1850 60  0000 L CNN
-F 1 "2u2" V 3300 1500 60  0000 L CNN
+F 1 "10uF" V 3300 1500 60  0000 L CNN
 F 2 "Capacitors_SMD.pretty:C_1206_HandSoldering" H 3250 1750 50  0001 C CNN
 F 3 "" H 3250 1750 50  0001 C CNN
@@
 P 3250 1950
 F 0 "C5" V 3300 2050 60  0000 L CNN
-F 1 "2u2" V 3300 1700 60  0000 L CNN
+F 1 "10uF" V 3300 1700 60  0000 L CNN
 F 2 "Capacitors_SMD.pretty:C_1206_HandSoldering" H 3250 1950 50  0001 C CNN
 F 3 "" H 3250 1950 50  0001 C CNN
@@
 L Device:L L1
 U 1 1 5BD6EF23
-P 2600 3650
-F 0 "L1" V 2419 3650 50  0000 C CNN
-F 1 "15n" V 2510 3650 50  0000 C CNN
-F 2 "Choke_SMD.pretty:Choke_SMD_1206_Handsoldering" H 2600 3650 50  0001 C CNN
-F 3 "~" H 2600 3650 50  0001 C CNN
-	1    2600 3650
+P 2650 3250
+F 0 "L1" V 2469 3250 50  0000 C CNN
+F 1 "15n" V 2560 3250 50  0000 C CNN
+F 2 "Choke_SMD.pretty:Choke_SMD_1206_Handsoldering" H 2650 3250 50  0001 C CNN
+F 3 "~" H 2650 3250 50  0001 C CNN
+	1    2650 3250
 	0    1    1    0
 $EndComp
-Wire Wire Line
-	2750 3650 3000 3650
-Wire Wire Line
-	2450 3650 2250 3650
 $Comp
 L c:C C2
 U 1 1 5BD76587
-P 2250 4000
-F 0 "C2" H 1950 3950 60  0000 L CNN
-F 1 "4u7" H 1900 3800 60  0000 L CNN
-F 2 "Capacitors_SMD.pretty:C_1206_HandSoldering" H 2250 4000 50  0001 C CNN
-F 3 "" H 2250 4000 50  0001 C CNN
-	1    2250 4000
-	1    0    0    -1
-$EndComp
-Wire Wire Line
-	2250 3800 2250 3650
-Connection ~ 2250 3650
-Wire Wire Line
-	2250 3650 1900 3650
+P 2350 3550
+F 0 "C2" H 2500 3650 60  0000 L CNN
+F 1 "4u7" H 2500 3550 60  0000 L CNN
+F 2 "Capacitors_SMD.pretty:C_1206_HandSoldering" H 2350 3550 50  0001 C CNN
+F 3 "" H 2350 3550 50  0001 C CNN
+	1    2350 3550
+	1    0    0    -1
+$EndComp
 $Comp
 L power:GND #PWR0104
 U 1 1 5BD79283
-P 2250 4400
-F 0 "#PWR0104" H 2250 4150 50  0001 C CNN
-F 1 "GND" H 2255 4227 50  0000 C CNN
-F 2 "" H 2250 4400 50  0001 C CNN
-F 3 "" H 2250 4400 50  0001 C CNN
-	1    2250 4400
-	1    0    0    -1
-$EndComp
-Wire Wire Line
-	2250 4200 2250 4400
-Text Label 2800 3650 0    50   ~ 0
-MIC+
-Wire Notes Line
-	2750 3400 2750 4650
-Wire Notes Line
-	2100 4650 2100 3400
-Text Notes 1800 5000 0    50   ~ 0
+P 2350 3950
+F 0 "#PWR0104" H 2350 3700 50  0001 C CNN
+F 1 "GND" H 2355 3777 50  0000 C CNN
+F 2 "" H 2350 3950 50  0001 C CNN
+F 3 "" H 2350 3950 50  0001 C CNN
+	1    2350 3950
+	1    0    0    -1
+$EndComp
+Wire Wire Line
+	2350 3750 2350 3950
+Wire Notes Line
+	2850 3000 2850 4250
+Wire Notes Line
+	2200 4250 2200 3000
+Text Notes 1900 4600 0    50   ~ 0
 this is at blk "datasheet"\nI put it here just in case\ns3860-m "datasheet"\nis missing this parts
 Wire Notes Line
-	2100 3400 2750 3400
-Wire Notes Line
-	2100 4650 2750 4650
+	2200 3000 2850 3000
+Wire Notes Line
+	2200 4250 2850 4250
 Wire Wire Line
 	6650 2550 7350 2550
@@
 Wire Wire Line
 	8550 2150 9350 2150
+Wire Wire Line
+	1900 3250 2350 3250
+Wire Wire Line
+	2800 3250 3100 3250
+Wire Wire Line
+	1900 3650 3000 3650
+Wire Wire Line
+	2350 3350 2350 3250
+Connection ~ 2350 3250
+Wire Wire Line
+	2350 3250 2500 3250
 $EndSCHEMATC
