File: kicad/S3860M-S_breadboard_adapter/S3860M-S_breadboard_adapter.kicad_pcb (KiCad board)
At the start: 2 copper layers, 26.5 x 31.6 mm, 17 parts, among them J1 SCJ368R1NUS0B00G, P1 CONN_01X12, P2 CONN_01X12, U1 S3860M-S

Commit message: to fcking much changes to commit it separatly, lets go with everything in one commit, git will love me for sure :D
Parts:
- removed GND1: GND, open-project:S_JUMPER_3
- removed ONKEY1: ONKEY, open-project:S_JUMPER_3
- removed RST1: RST, open-project:S_JUMPER_3
- removed VBUCK1: VBUCK, open-project:S_JUMPER_3
- removed VOL+1: VOL+, open-project:S_JUMPER_3
- removed VOL-1: VOL-, open-project:S_JUMPER_3
- added C1: 100n, Capacitors_SMD.pretty:C_1206_HandSoldering, F.Cu at (101.8, 103.6)
- moved R1 3.42 mm to (93.4, 103.7)
- moved J1 3.11 mm to (97.9, 119.9)
Connections:
- ON/OFF/PLAY1 pad 2: /ONKEY -> Net-(ON/OFF/PLAY1-Pad2)
- P1 pad 4: /VBUCK -> Net-(P1-Pad4)
- P2 pad 10: /VOL+ -> Net-(P2-Pad10)
- P2 pad 11: /ONKEY -> Net-(ON/OFF/PLAY1-Pad2)
- P2 pad 8: /RESET -> Net-(P2-Pad8)
- P2 pad 9: /VOL- -> Net-(P2-Pad9)
- R1 pad 1: /RESET -> Net-(P2-Pad8)
- RESET1 pad 2: /RESET -> Net-(P2-Pad8)
- U1 pad 10: Net-(GND1-Pad3) -> Net-(P1-Pad4)
- U1 pad 11: Net-(GND1-Pad1) -> /GND
- U1 pad 14: Net-(ONKEY1-Pad3) -> Net-(ON/OFF/PLAY1-Pad2)
- U1 pad 15: Net-(RST1-Pad1) -> Net-(P2-Pad10)
- U1 pad 16: Net-(ONKEY1-Pad1) -> Net-(P2-Pad9)
- U1 pad 17: Net-(RST1-Pad3) -> Net-(P2-Pad8)
- U1 pad 18: Net-(U1-Pad18) -> (no net)
Routing:
- net /ONKEY: track 23.6 -> 0.00 mm
- net /RESET: track 22.2 -> 0.00 mm
- net /GND: track 0.58 -> 22.6 mm, vias 0 -> 1
- net Net-(GND1-Pad1): track 18.1 -> 0.00 mm, vias 2 -> 0
- net Net-(ON/OFF/PLAY1-Pad2): track 0.00 -> 17.1 mm, vias 0 -> 1
- net Net-(P2-Pad8): track 0.00 -> 17.1 mm, vias 0 -> 1
- net Net-(ONKEY1-Pad1): track 17.1 -> 0.00 mm, vias 2 -> 0
- net Net-(RST1-Pad3): track 16.5 -> 0.00 mm, vias 2 -> 0
- net Net-(U1-Pad18): track 15.5 -> 0.00 mm, vias 1 -> 0
- net Net-(RST1-Pad1): track 15.5 -> 0.00 mm, vias 2 -> 0
- net Net-(GND1-Pad3): track 14.9 -> 0.00 mm
- net Net-(C1-Pad2): track 44.0 -> 32.3 mm, vias 0 -> 2
- net Net-(ONKEY1-Pad3): track 9.76 -> 0.00 mm, vias 1 -> 0
- net Net-(P2-Pad10): track 0.00 -> 9.31 mm
- net Net-(P1-Pad4): track 0.00 -> 8.94 mm
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Other:
- board text added: "1V8"
- board text added: "GND"
- board text added: "VBAT"
- board text added: "VOL+"
- board text added: "VOL-"
- board text removed: "+"
- board text removed: "-"
- board text removed: "GND VBAT 1V8"
- board text removed: "MODULE SELECT"
- board text removed: "S3860M-S"
- board text removed: "XS3868"
