File: kicad/arduino_based_cdc_emulator/atmega88/arduino_based_cdc_emu.kicad_pcb (KiCad board)
At the start: 2 copper layers, 25.4 x 23.2 mm, 14 parts, among them IC1 ATMEGA88-A, P1 CONN_1, P2 CONN_2, P3 CONN_3, U1 78L05, X1 20MHz

Commit message: update
Parts:
- removed C1, C2: 22p, Capacitors_SMD:C_1206_HandSoldering
- removed C3, C4: 100n, Capacitors_SMD:C_1206_HandSoldering
- removed IC1: ATMEGA88-A, SMD_Packages:TQFP-32
- removed P1: CONN_1, Pin_Headers:Pin_Header_Straight_1x05
- removed P2: CONN_2, Pin_Headers:Pin_Header_Straight_1x05
- removed P3: CONN_3, Pin_Headers:Pin_Header_Straight_1x01
- removed R1, R2, R3, R4: 3k3, Resistors_SMD:R_1206_HandSoldering
- removed U1: 78L05, my_modules:SOT-223-REGULATOR
- removed X1: 20MHz, Crystals_Oscillators_SMD:Q_49U3HMS
Routing:
- net GND: track 106.8 -> 0.00 mm
- net +5V: track 40.8 -> 0.00 mm
- net /DataOut: track 34.1 -> 0.00 mm
- net +12V: track 20.1 -> 0.00 mm
- net Net-(C2-Pad2): track 17.5 -> 0.00 mm
- net Net-(IC1-Pad15): track 17.2 -> 0.00 mm
- net Net-(C1-Pad2): track 14.8 -> 0.00 mm
- net /RESET: track 11.9 -> 0.00 mm
- net TX: track 11.5 -> 0.00 mm
- net RX: track 10.5 -> 0.00 mm
- net /MISO: track 9.94 -> 0.00 mm
- net Net-(IC1-Pad32): track 8.87 -> 0.00 mm
- net Net-(IC1-Pad17): track 8.83 -> 0.00 mm
- net /Clock: track 7.78 -> 0.00 mm
- net /DataIn: track 4.40 -> 0.00 mm
Other:
- board outline removed
