File: kicad/arduino_based_cdc_emulator/atmega88/arduino_based_cdc_emu.sch (KiCad schematic (older format))
At the start: 25 parts, among them IC1 ATMEGA88-A, P1 CONN_1, P2 CONN_2, P3 CONN_3, Q1 Q_NPN_EBC, Q2 Q_NPN_EBC, Q3 Q_NPN_EBC, U1 78L05, X1 16MHz

Commit message: update
Parts:
- removed C1, C2: 22p, Capacitors_SMD:C_0805, symbol C-RESCUE-arduino_based_cdc_emu
- removed D1: 1N4148, Diodes_SMD:DO-214AA, symbol D
- removed Q1, Q2, Q3: Q_NPN_EBC, symbol Q_NPN_BEC
- removed R1, R2: 3k3, Resistors_SMD:R_0805, symbol R-RESCUE-arduino_based_cdc_emu
- removed R5, R7, R9: 3k3, Resistors_SMD:R_0805_HandSoldering, symbol R-RESCUE-arduino_based_cdc_emu
- removed R6, R8: 47k, Resistors_SMD:R_0805_HandSoldering, symbol R-RESCUE-arduino_based_cdc_emu
- removed X1: 16MHz, Crystals_Oscillators_SMD:Q_49U3HMS, symbol CRYSTAL
- added D? (x2): 1N4148, Diodes_SMD:DO-214AA, symbol D
- added JP?: Jumper_NC_Dual, Pin_Headers:Pin_Header_Straight_1x03_Pitch2.54mm, symbol Jumper_NC_Dual
- added R? (x2): 3k3, Resistors_SMD:R_0805, symbol R-RESCUE-arduino_based_cdc_emu
- added Y?: Resonator_Small, modules:MURATA_CSTCE_V53, symbol Resonator_Small
Connections:
- wire segments 71 -> 62
Other:
- moved on the sheet: R4
