File: kicad/arduino_based_cdc_emulator/atmega88/arduino_based_cdc_emu.sch (KiCad schematic (older format))
At the start: 17 parts, among them IC1 ATMEGA88-A, P1 CONN_1, P2 CONN_2, P3 CONN_3, U1 78L05

Commit message: to fcking much changes to commit it separatly, lets go with everything in one commit, git will love me for sure :D
Parts:
- C3, C4: symbol C-RESCUE-arduino_based_cdc_emu -> arduino_based_cdc_emu-rescue:C-RESCUE-arduino_based_cdc_emu
- C5: symbol CP -> arduino_based_cdc_emu-rescue:CP-RESCUE-arduino_based_cdc_emu
- D2, D? (x2): symbol D -> arduino_based_cdc_emu-rescue:D-RESCUE-arduino_based_cdc_emu
- IC1: symbol ATMEGA88-A -> arduino_based_cdc_emu-rescue:ATMEGA88-A-RESCUE-arduino_based_cdc_emu
- JP?: symbol Jumper_NC_Dual -> arduino_based_cdc_emu-rescue:Jumper_NC_Dual-RESCUE-arduino_based_cdc_emu
- P1: symbol CONN_5 -> arduino_based_cdc_emu-rescue:CONN_5-RESCUE-arduino_based_cdc_emu
- P2: symbol CONN_01X05 -> arduino_based_cdc_emu-rescue:CONN_01X05-RESCUE-arduino_based_cdc_emu
- P3: symbol CONN_01X01 -> arduino_based_cdc_emu-rescue:CONN_01X01-RESCUE-arduino_based_cdc_emu
- R3, R4, R? (x2): symbol R-RESCUE-arduino_based_cdc_emu -> arduino_based_cdc_emu-rescue:R-RESCUE-arduino_based_cdc_emu
- U1: symbol 78L05 -> arduino_based_cdc_emu-rescue:78L05-RESCUE-arduino_based_cdc_emu
- Y?: symbol Resonator_Small -> arduino_based_cdc_emu-rescue:Resonator_Small-RESCUE-arduino_based_cdc_emu
Connections:
- wire segments 62 -> 70
Changed lines of the file:
@@
-EESchema Schematic File Version 2
-LIBS:arduino_based_cdc_emu-rescue
-LIBS:power
-LIBS:device
-LIBS:transistors
-LIBS:conn
-LIBS:linear
-LIBS:regul
-LIBS:74xx
-LIBS:cmos4000
-LIBS:adc-dac
-LIBS:memory
-LIBS:xilinx
-LIBS:microcontrollers
-LIBS:dsp
-LIBS:microchip
-LIBS:analog_switches
-LIBS:motorola
-LIBS:texas
-LIBS:intel
-LIBS:audio
-LIBS:interface
-LIBS:digital-audio
-LIBS:philips
-LIBS:display
-LIBS:cypress
-LIBS:siliconi
-LIBS:opto
-LIBS:atmel
-LIBS:contrib
-LIBS:valves
+EESchema Schematic File Version 4
 LIBS:arduino_based_cdc_emu-cache
 EELAYER 26 0
@@
 $EndDescr
 $Comp
-L +5V #PWR01
+L power:+5V #PWR01
 U 1 1 53207304
 P 4900 5400
@@
 $EndComp
 $Comp
-L R-RESCUE-arduino_based_cdc_emu R3
+L arduino_based_cdc_emu-rescue:R-RESCUE-arduino_based_cdc_emu R3
 U 1 1 532072FD
 P 4900 5700
@@
 DataOut
 $Comp
-L GND-RESCUE-arduino_based_cdc_emu #PWR02
+L arduino_based_cdc_emu-rescue:GND-RESCUE-arduino_based_cdc_emu #PWR02
 U 1 1 530C945D
 P 9550 2400
@@
 $EndComp
 $Comp
-L CONN_5 P1
+L arduino_based_cdc_emu-rescue:CONN_5-RESCUE-arduino_based_cdc_emu P1
 U 1 1 530C9435
 P 10050 2150
@@
 $EndComp
 $Comp
-L +12V #PWR03
+L power:+12V #PWR03
 U 1 1 530C8041
 P 2400 5500
@@
 $EndComp
 $Comp
-L +5V #PWR04
+L power:+5V #PWR04
 U 1 1 530C8014
 P 3850 5550
@@
 $EndComp
 $Comp
-L GND-RESCUE-arduino_based_cdc_emu #PWR05
+L arduino_based_cdc_emu-rescue:GND-RESCUE-arduino_based_cdc_emu #PWR05
 U 1 1 530C800A
 P 3200 6250
@@
 $EndComp
 $Comp
-L 78L05 U1
+L arduino_based_cdc_emu-rescue:78L05-RESCUE-arduino_based_cdc_emu U1
 U 1 1 530C7FFF
 P 3200 5700
@@
 $EndComp
 $Comp
-L GND-RESCUE-arduino_based_cdc_emu #PWR06
+L arduino_based_cdc_emu-rescue:GND-RESCUE-arduino_based_cdc_emu #PWR06
 U 1 1 530C7FEB
 P 3850 6250
@@
 $EndComp
 $Comp
-L GND-RESCUE-arduino_based_cdc_emu #PWR07
+L arduino_based_cdc_emu-rescue:GND-RESCUE-arduino_based_cdc_emu #PWR07
 U 1 1 530C7FE7
 P 2500 6250
@@
 $EndComp
 $Comp
-L C-RESCUE-arduino_based_cdc_emu C4
+L arduino_based_cdc_emu-rescue:C-RESCUE-arduino_based_cdc_emu C4
 U 1 1 530C7FE2
 P 3850 5900
@@
 $EndComp
 $Comp
-L C-RESCUE-arduino_based_cdc_emu C3
+L arduino_based_cdc_emu-rescue:C-RESCUE-arduino_based_cdc_emu C3
 U 1 1 530C7FD9
 P 2500 5900
@@
 $EndComp
 $Comp
-L R-RESCUE-arduino_based_cdc_emu R4
+L arduino_based_cdc_emu-rescue:R-RESCUE-arduino_based_cdc_emu R4
 U 1 1 530C77E3
 P 6050 4900
@@
 $EndComp
 $Comp
-L +5V #PWR08
+L power:+5V #PWR08
 U 1 1 530C77C0
 P 1450 1850
@@
 $EndComp
 $Comp
-L GND-RESCUE-arduino_based_cdc_emu #PWR09
+L arduino_based_cdc_emu-rescue:GND-RESCUE-arduino_based_cdc_emu #PWR09
 U 1 1 530C77A6
 P 1450 4500
@@
 $EndComp
 $Comp
-L ATMEGA88-A IC1
+L arduino_based_cdc_emu-rescue:ATMEGA88-A-RESCUE-arduino_based_cdc_emu IC1
 U 1 1 530C76C5
 P 2400 3150
@@
 $EndComp
 $Comp
-L +12V #PWR011
+L power:+12V #PWR011
 U 1 1 543549B8
 P 9350 1750
@@
 $EndComp
 $Comp
-L CONN_01X05 P2
+L arduino_based_cdc_emu-rescue:CONN_01X05-RESCUE-arduino_based_cdc_emu P2
 U 1 1 54357812
 P 9150 4800
@@
 TX
 $Comp
-L GND-RESCUE-arduino_based_cdc_emu #PWR012
+L arduino_based_cdc_emu-rescue:GND-RESCUE-arduino_based_cdc_emu #PWR012
 U 1 1 54358932
 P 8750 5100
@@
 RESET
 $Comp
-L +5V #PWR013
+L power:+5V #PWR013
 U 1 1 554857A3
 P 8750 4400
@@
 	8050 1950 8950 1950
 Wire Wire Line
-	3850 5550 3850 5700
+	3850 5550 3850 5650
 Wire Wire Line
 	3400 2650 4900 2650
@@
 	3400 3850 4850 3850
 Wire Wire Line
-	2400 5650 2800 5650
+	2400 5650 2500 5650
 Wire Wire Line
 	3200 5950 3200 6250
@@
 	1450 2650 1500 2650
 Wire Wire Line
-	1450 1850 1450 2650
+	1450 1850 1450 2050
 Wire Wire Line
 	1500 2350 1450 2350
@@
 	1500 4150 1450 4150
 Wire Wire Line
-	1450 4150 1450 4500
+	1450 4150 1450 4250
 Wire Wire Line
 	1500 4250 1450 4250
@@
 	8750 4600 8750 4400
 $Comp
-L CONN_01X01 P3
+L arduino_based_cdc_emu-rescue:CONN_01X01-RESCUE-arduino_based_cdc_emu P3
 U 1 1 5548A42E
 P 9150 5750
@@
 MISO
 $Comp
-L CP C5
+L arduino_based_cdc_emu-rescue:CP-RESCUE-arduino_based_cdc_emu C5
 U 1 1 560D753D
 P 4900 6300
@@
 RESET
 Wire Wire Line
-	4900 5950 4900 6150
-$Comp
-L GND-RESCUE-arduino_based_cdc_emu #PWR014
+	4900 5950 4900 6000
+$Comp
+L arduino_based_cdc_emu-rescue:GND-RESCUE-arduino_based_cdc_emu #PWR014
 U 1 1 560D79D0
 P 4900 6600
@@
 	3850 6100 3850 6250
 $Comp
-L Jumper_NC_Dual JP?
+L arduino_based_cdc_emu-rescue:Jumper_NC_Dual-RESCUE-arduino_based_cdc_emu JP?
 U 1 1 58C14056
 P 5550 4350
@@
 	4850 4350 5300 4350
 $Comp
-L GND-RESCUE-arduino_based_cdc_emu #PWR010
+L arduino_based_cdc_emu-rescue:GND-RESCUE-arduino_based_cdc_emu #PWR010
 U 1 1 530C7791
 P 5350 2950
@@
 $EndComp
 $Comp
-L Resonator_Small Y?
+L arduino_based_cdc_emu-rescue:Resonator_Small-RESCUE-arduino_based_cdc_emu Y?
 U 1 1 58C19400
 P 5000 2750
@@
 	5350 2750 5350 2950
 $Comp
-L D D2
+L arduino_based_cdc_emu-rescue:D-RESCUE-arduino_based_cdc_emu D2
 U 1 1 5685E033
 P 9100 2150
@@
 $EndComp
 $Comp
-L D D?
+L arduino_based_cdc_emu-rescue:D-RESCUE-arduino_based_cdc_emu D?
 U 1 1 58C1A494
 P 8650 2050
@@
 $EndComp
 $Comp
-L D D?
+L arduino_based_cdc_emu-rescue:D-RESCUE-arduino_based_cdc_emu D?
 U 1 1 58C16D80
 P 9100 1950
@@
 	8950 2150 8050 2150
 $Comp
-L R-RESCUE-arduino_based_cdc_emu R?
+L arduino_based_cdc_emu-rescue:R-RESCUE-arduino_based_cdc_emu R?
 U 1 1 58C1746A
 P 3800 2550
@@
 $EndComp
 $Comp
-L R-RESCUE-arduino_based_cdc_emu R?
+L arduino_based_cdc_emu-rescue:R-RESCUE-arduino_based_cdc_emu R?
 U 1 1 58C1758C
 P 3800 2350
@@
 Wire Wire Line
 	4050 2350 4200 2350
+Wire Wire Line
+	1450 2350 1450 2650
+Wire Wire Line
+	1450 2150 1450 2350
+Wire Wire Line
+	1450 2050 1450 2150
+Wire Wire Line
+	1450 4250 1450 4350
+Wire Wire Line
+	1450 4350 1450 4500
+Wire Wire Line
+	4900 6000 4900 6150
+Wire Wire Line
+	3850 5650 3850 5700
+Wire Wire Line
+	2500 5650 2800 5650
 $EndSCHEMATC
