File: kicad/regulated_power_supply/regulated_power_supply.kicad_pcb (KiCad board)
At the start: 2 copper layers, 139.1 x 38.5 mm, 47 parts, among them P1 CONN_01X03, P2 CONN_01X02, Q1 Q_NPN_BCE, SW1 SPST, T1 2N3055, U1 TL072, U2 LM723

Commit message: update
Parts:
- moved C6 3.21 mm to (172.5, 37.6), turned to 0 degrees
- moved Rv1 2.29 mm to (161.5, 50.3)
- moved D7 0.82 mm to (165.6, 52.1)
- moved D6 0.79 mm to (165.6, 49.3)
Routing:
- net Net-(C6-Pad1): track 39.4 -> 42.6 mm
- net Net-(R2-Pad1): track 23.9 -> 26.8 mm
- net Net-(C7-Pad2): track 37.5 -> 40.2 mm
- net Net-(D6-Pad2): track 8.05 -> 9.72 mm
- net Net-(D7-Pad2): track 7.63 -> 8.89 mm
- net /Vout: track 111.1 -> 110.6 mm
