File: kicad/regulated_power_supply/regulated_power_supply.sch (KiCad schematic (older format))
At the start: 47 parts, among them P1 CONN_01X03, P2 CONN_01X02, Q1 Q_NPN_BCE, SW1 SPST, T1 2N3055, U1 TL072, U2 LM723

Commit message: update
Parts:
- D5: symbol LED -> LED-RESCUE-regulated_power_supply
Changed lines of the file:
@@
 LIBS:valves
 LIBS:regulated_power_supply-cache
-EELAYER 25 0
+EELAYER 26 0
 EELAYER END
 $Descr A4 11693 8268
@@
 $EndComp
 $Comp
-L LED D5
+L LED-RESCUE-regulated_power_supply D5
 U 1 1 56730594
 P 2100 4450
