File: kicad/SOIC28_breadboard_adapter/SOIC28_breadboard_adapter.kicad_pcb (KiCad board)
At the start: 2 copper layers, 21.8 x 65 mm, 6 parts, among them IC1 AT90S1200-Y, P1 CONN_01X14, P2 CONN_01X14, P3 CONN_01X10, P4 CONN_01X14, U1 HM62256BLFP-4SLT

Commit message: to fcking much changes to commit it separatly, lets go with everything in one commit, git will love me for sure :D
Parts:
- removed IC1: AT90S1200-Y, Housings_SOIC:SOIC-20_7.5x12.8mm_Pitch1.27mm
- removed P3: CONN_01X10, Pin_Headers:Pin_Header_Straight_1x10
- removed P4: CONN_01X14, Pin_Headers:Pin_Header_Straight_1x10
- added U2: HM62256BLFP-4SLT, Housings_SOIC.pretty:SOIC-28_7.5x17.9mm_Pitch1.27mm, B.Cu at (174.0, 120.7)
Connections:
- P1 pad 1: Net-(P1-Pad1) -> GND
- P2 pad 1: Net-(P2-Pad1) -> GND
- P2 pad 14: VCC -> GND
- P2 pad 5: Net-(P2-Pad5) -> Net-(P1-Pad2)
- U1 pad 1: Net-(P1-Pad1) -> GND
- U1 pad 15: Net-(P2-Pad1) -> GND
- U1 pad 19: Net-(P2-Pad5) -> Net-(P1-Pad2)
- U1 pad 28: VCC -> GND
Routing:
- net GND: track 12.1 -> 80.6 mm
- net Net-(P1-Pad2): track 12.6 -> 30.3 mm
- net Net-(P2-Pad1): track 13.9 -> 0.00 mm
- net Net-(P1-Pad1): track 13.0 -> 0.00 mm
- net VCC: track 12.9 -> 0.00 mm
- net Net-(IC1-Pad20): track 9.09 -> 0.00 mm
- net Net-(IC1-Pad1): track 8.94 -> 0.00 mm
- net Net-(IC1-Pad11): track 8.94 -> 0.00 mm
- net Net-(IC1-Pad10): track 8.94 -> 0.00 mm
- net Net-(P2-Pad11): track 6.92 -> 14.2 mm
- net Net-(P1-Pad13): track 12.2 -> 19.3 mm
- net Net-(IC1-Pad9): track 6.92 -> 0.00 mm
- net Net-(IC1-Pad2): track 6.92 -> 0.00 mm
- net Net-(IC1-Pad19): track 6.92 -> 0.00 mm
- net Net-(IC1-Pad12): track 6.78 -> 0.00 mm
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Other:
- board size 21.8 x 65 mm -> 21.8 x 37.1 mm
