File: kicad/SOIC28_breadboard_adapter/SOIC28_breadboard_adapter.sch (KiCad schematic (older format))
At the start: 6 parts, among them IC1 AT90S1200-Y, P1 CONN_01X14, P2 CONN_01X14, P3 CONN_01X10, P4 CONN_01X14, U1 HM62256BLFP-4SLT

Commit message: to fcking much changes to commit it separatly, lets go with everything in one commit, git will love me for sure :D
Parts:
- removed IC1: AT90S1200-Y, Housings_SOIC:SOIC-20_7.5x12.8mm_Pitch1.27mm, symbol AT90S1200-Y
- removed P3: CONN_01X10, Pin_Headers:Pin_Header_Straight_1x10, symbol CONN_01X10
- removed P4: CONN_01X14, Pin_Headers:Pin_Header_Straight_1x10, symbol CONN_01X10
- added U2: HM62256BLFP-4SLT, Housings_SOIC:SOIC-28_7.5x17.9mm_Pitch1.27mm, symbol SOIC28_breadboard_adapter-rescue:HM62256BLFP-4SLT-RESCUE-SOIC28_breadboard_adap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
- P1, P2: symbol CONN_01X14 -> SOIC28_breadboard_adapter-rescue:CONN_01X14-RESCUE-SOIC28_breadboard_adapter
- U1: symbol HM62256BLFP-4SLT -> SOIC28_breadboard_adapter-rescue:HM62256BLFP-4SLT-RESCUE-SOIC28_breadboard_adapter
Connections:
- wire segments 95 -> 179
