File: kicad/ardpicprog/ardpicprog.sch (KiCad schematic (older format))
At the start: 33 parts, among them P1 CONN_01X06, P2 CONN_01X02, Q1 BC548, SW1 SW_PUSH, U1 PIC16F627, U2 MC34063, U3 LM78L12ACZ

Commit message: to fcking much changes to commit it separatly, lets go with everything in one commit, git will love me for sure :D
Parts:
- C1, C2, C3, C4, C5, C6, C7: symbol C-RESCUE-ardpicprog -> ardpicprog-rescue:C-RESCUE-ardpicprog
- D1, D3: symbol LED -> ardpicprog-rescue:LED-RESCUE-ardpicprog
- D2: symbol DIODESCH -> ardpicprog-rescue:DIODESCH-RESCUE-ardpicprog
- D4, D5: symbol DIODE -> ardpicprog-rescue:DIODE-RESCUE-ardpicprog
- JP1: symbol JUMPER3 -> ardpicprog-rescue:JUMPER3-RESCUE-ardpicprog
- L1: symbol INDUCTOR -> ardpicprog-rescue:INDUCTOR-RESCUE-ardpicprog
- P1: symbol CONN_01X06 -> ardpicprog-rescue:CONN_01X06-RESCUE-ardpicprog
- P2: symbol CONN_01X02 -> ardpicprog-rescue:CONN_01X02-RESCUE-ardpicprog
- Q1: symbol BC548 -> ardpicprog-rescue:BC548-RESCUE-ardpicprog
- R1, R10, R11, R2, R3, R4, R5, R6, R7, R8, R9: symbol R-RESCUE-ardpicprog -> ardpicprog-rescue:R-RESCUE-ardpicprog
- SHIELD1: symbol ARDUINO_SHIELD -> ardpicprog-rescue:ARDUINO_SHIELD-RESCUE-ardpicprog
- SW1: symbol SW_PUSH -> ardpicprog-rescue:SW_PUSH-RESCUE-ardpicprog
- U1: symbol PIC16F627 -> ardpicprog-rescue:PIC16F627-RESCUE-ardpicprog
- U2: symbol MC34063 -> ardpicprog-rescue:MC34063-RESCUE-ardpicprog
- U3: symbol LM78L12ACZ -> ardpicprog-rescue:LM78L12ACZ-RESCUE-ardpicprog
Connections:
- wire segments 104 -> 123
