File: kicad/ardpicprog/ardpicprog_smd.kicad_pcb (KiCad board)
At the start: 2 copper layers, 69.2 x 53.9 mm, 37 parts, among them P1 CONN_01X06, P2 CONN_01X02, Q1 BC548, SW1 SW_PUSH, U1 PIC16F627, U2 MC34063, U3 LM78L12ACZ

Commit message: update
Parts:
- turned SW1 to 0 degrees
Routing:
- net RESET: track 35.4 -> 33.0 mm
