File: kicad/arduino_atmega88/arduino_atmega88.sch (KiCad schematic (older format))
At the start: 21 parts, among them IC1 ATMEGA88A-A, P1 CONN_6, P4 CONN_7, SW1 SW_PUSH, U1 78L05, X1 16MHz

Commit message: to fcking much changes to commit it separatly, lets go with everything in one commit, git will love me for sure :D
Parts:
- C1, C2, C3, C4, C5, C6: symbol C-RESCUE-arduino_atmega88 -> arduino_atmega88-rescue:C-RESCUE-arduino_atmega88
- D1, D2: symbol LED-RESCUE-arduino_atmega88 -> arduino_atmega88-rescue:LED-RESCUE-arduino_atmega88
- D3, D4: symbol DIODE -> arduino_atmega88-rescue:DIODE-RESCUE-arduino_atmega88
- IC1: symbol ATMEGA88A-A -> arduino_atmega88-rescue:ATMEGA88A-A-RESCUE-arduino_atmega88
- P1: symbol CONN_6 -> arduino_atmega88-rescue:CONN_6-RESCUE-arduino_atmega88
- P4: symbol CONN_7 -> arduino_atmega88-rescue:CONN_7-RESCUE-arduino_atmega88
- R1, R2, R3, R4: symbol R-RESCUE-arduino_atmega88 -> arduino_atmega88-rescue:R-RESCUE-arduino_atmega88
- SHIELD1: symbol ARDUINO_SHIELD -> arduino_shieldsNCL:ARDUINO_SHIELD
- SW1: symbol SW_PUSH -> arduino_atmega88-rescue:SW_PUSH-RESCUE-arduino_atmega88
- U1: symbol 78L05 -> arduino_atmega88-rescue:78L05-RESCUE-arduino_atmega88
- X1: symbol CRYSTAL -> arduino_atmega88-rescue:CRYSTAL-RESCUE-arduino_atmega88
Connections:
- wire segments 118 -> 130
Changed lines of the file:
@@
-EESchema Schematic File Version 2
-LIBS:arduino_atmega88-rescue
-LIBS:power
-LIBS:device
-LIBS:transistors
-LIBS:conn
-LIBS:linear
-LIBS:regul
-LIBS:74xx
-LIBS:cmos4000
-LIBS:adc-dac
-LIBS:memory
-LIBS:xilinx
-LIBS:microcontrollers
-LIBS:dsp
-LIBS:microchip
-LIBS:analog_switches
-LIBS:motorola
-LIBS:texas
-LIBS:intel
-LIBS:audio
-LIBS:interface
-LIBS:digital-audio
-LIBS:philips
-LIBS:display
-LIBS:cypress
-LIBS:siliconi
-LIBS:opto
-LIBS:atmel
-LIBS:contrib
-LIBS:valves
-LIBS:arduino_shieldsNCL
+EESchema Schematic File Version 4
 LIBS:arduino_atmega88-cache
-EELAYER 25 0
+EELAYER 26 0
 EELAYER END
 $Descr A4 11693 8268
@@
 	2150 3800 1750 3800
 Wire Wire Line
-	1750 3950 1750 3600
+	1750 3950 1750 3800
 Wire Wire Line
 	1750 3600 2150 3600
@@
 	5500 2300 5500 2350
 Wire Wire Line
-	5000 2950 4050 2950
+	5000 2950 4900 2950
 Wire Wire Line
 	5250 1400 5250 1550
@@
 	4650 1950 4650 2100
 Wire Wire Line
-	4650 2100 4050 2100
+	4650 2100 4500 2100
 Wire Wire Line
 	4050 3700 4350 3700
@@
 	4050 3800 4350 3800
 Wire Wire Line
-	4050 2200 5250 2200
-Wire Wire Line
-	5250 2200 5250 1950
+	4050 2200 4700 2200
+Wire Wire Line
+	5250 2200 5250 2100
 Connection ~ 5250 2100
 Wire Wire Line
@@
 	4900 2350 4900 2400
 Wire Wire Line
-	4900 2900 4900 3050
+	4900 2900 4900 2950
 Wire Wire Line
 	9400 1700 9750 1700
@@
 	7000 2200 7000 2150
 Wire Wire Line
-	7500 2400 6750 2400
+	7500 2400 7400 2400
 Wire Wire Line
 	6750 2400 6750 2500
@@
 	2150 1800 1750 1800
 Wire Wire Line
-	1750 1800 1750 1400
+	1750 1800 1750 1600
 Connection ~ 1750 1500
 Wire Wire Line
@@
 	1650 5350 1800 5350
 Wire Wire Line
-	1650 5000 1650 5550
+	1650 5000 1650 5350
 Connection ~ 1650 5350
 Wire Wire Line
@@
 	8400 5700 8400 5600
 Wire Wire Line
-	2800 5350 2600 5350
-$Comp
-L DIODE D3
+	2800 5350 2700 5350
+$Comp
+L arduino_atmega88-rescue:DIODE-RESCUE-arduino_atmega88 D3
 U 1 1 5335B1E9
 P 3000 5350
@@
 $EndComp
 $Comp
-L DIODE D4
+L arduino_atmega88-rescue:DIODE-RESCUE-arduino_atmega88 D4
 U 1 1 5335A8D7
 P 8650 5700
@@
 $EndComp
 $Comp
-L GND-RESCUE-arduino_atmega88 #PWR01
+L arduino_atmega88-rescue:GND-RESCUE-arduino_atmega88 #PWR01
 U 1 1 5335A5BD
 P 2200 6100
@@
 $EndComp
 $Comp
-L GND-RESCUE-arduino_atmega88 #PWR02
+L arduino_atmega88-rescue:GND-RESCUE-arduino_atmega88 #PWR02
 U 1 1 5335A5B8
 P 2700 6100
@@
 $EndComp
 $Comp
-L GND-RESCUE-arduino_atmega88 #PWR03
+L arduino_atmega88-rescue:GND-RESCUE-arduino_atmega88 #PWR03
 U 1 1 5335A5B7
 P 1650 6100
@@
 Vin
 $Comp
-L +5V #PWR04
+L power1:+5V #PWR04
 U 1 1 5335A59A
 P 3300 5100
@@
 $EndComp
 $Comp
-L 78L05 U1
+L arduino_atmega88-rescue:78L05-RESCUE-arduino_atmega88 U1
 U 1 1 5335A58C
 P 2200 5400
@@
 $EndComp
 $Comp
-L C-RESCUE-arduino_atmega88 C6
+L arduino_atmega88-rescue:C-RESCUE-arduino_atmega88 C6
 U 1 1 5335A584
 P 2700 5800
@@
 $EndComp
 $Comp
-L C-RESCUE-arduino_atmega88 C5
+L arduino_atmega88-rescue:C-RESCUE-arduino_atmega88 C5
 U 1 1 5335A581
 P 1650 5750
@@
 $EndComp
 $Comp
-L CONN_6 P1
+L arduino_atmega88-rescue:CONN_6-RESCUE-arduino_atmega88 P1
 U 1 1 53318F84
 P 5250 5500
@@
 $EndComp
 $Comp
-L +5V #PWR05
+L power1:+5V #PWR05
 U 1 1 53318048
 P 8050 4550
@@
 $EndComp
 $Comp
-L LED-RESCUE-arduino_atmega88 D2
+L arduino_atmega88-rescue:LED-RESCUE-arduino_atmega88 D2
 U 1 1 53318026
 P 8050 5600
@@
 $EndComp
 $Comp
-L R-RESCUE-arduino_atmega88 R2
+L arduino_atmega88-rescue:R-RESCUE-arduino_atmega88 R2
 U 1 1 53318025
 P 8050 5000
@@
 $EndComp
 $Comp
-L GND-RESCUE-arduino_atmega88 #PWR06
+L arduino_atmega88-rescue:GND-RESCUE-arduino_atmega88 #PWR06
 U 1 1 53318024
 P 8050 6000
@@
 SCK
 $Comp
-L GND-RESCUE-arduino_atmega88 #PWR07
+L arduino_atmega88-rescue:GND-RESCUE-arduino_atmega88 #PWR07
 U 1 1 53317FD6
 P 7200 6000
@@
 $EndComp
 $Comp
-L R-RESCUE-arduino_atmega88 R1
+L arduino_atmega88-rescue:R-RESCUE-arduino_atmega88 R1
 U 1 1 53317FCD
 P 7200 5000
@@
 $EndComp
 $Comp
-L LED-RESCUE-arduino_atmega88 D1
+L arduino_atmega88-rescue:LED-RESCUE-arduino_atmega88 D1
 U 1 1 53317FC2
 P 7200 5600
@@
 DTR
 $Comp
-L +3.3V-RESCUE-arduino_atmega88 #PWR08
+L arduino_atmega88-rescue:+3.3V-RESCUE-arduino_atmega88 #PWR08
 U 1 1 53317D04
 P 8800 6000
@@
 $EndComp
 $Comp
-L +5V #PWR09
+L power1:+5V #PWR09
 U 1 1 53317CF8
 P 8400 5600
@@
 RX
 $Comp
-L GND-RESCUE-arduino_atmega88 #PWR010
+L arduino_atmega88-rescue:GND-RESCUE-arduino_atmega88 #PWR010
 U 1 1 53317C3C
 P 9000 5200
@@
 MOSI
 $Comp
-L GND-RESCUE-arduino_atmega88 #PWR011
+L arduino_atmega88-rescue:GND-RESCUE-arduino_atmega88 #PWR011
 U 1 1 53317586
 P 4300 5950
@@
 $EndComp
 $Comp
-L +5V #PWR012
+L power1:+5V #PWR012
 U 1 1 53317583
 P 4300 5150
@@
 MISO
 $Comp
-L CONN_7 P4
+L arduino_atmega88-rescue:CONN_7-RESCUE-arduino_atmega88 P4
 U 1 1 533174DE
 P 9750 5700
@@
 $EndComp
 $Comp
-L GND-RESCUE-arduino_atmega88 #PWR013
+L arduino_atmega88-rescue:GND-RESCUE-arduino_atmega88 #PWR013
 U 1 1 53317494
 P 1750 3950
@@
 A6
 $Comp
-L +5V #PWR014
+L power1:+5V #PWR014
 U 1 1 533171DD
 P 1750 1400
@@
 AREF
 $Comp
-L GND-RESCUE-arduino_atmega88 #PWR015
+L arduino_atmega88-rescue:GND-RESCUE-arduino_atmega88 #PWR015
 U 1 1 53317195
 P 1750 2650
@@
 $EndComp
 $Comp
-L C-RESCUE-arduino_atmega88 C1
+L arduino_atmega88-rescue:C-RESCUE-arduino_atmega88 C1
 U 1 1 5331718F
 P 1750 2350
@@
 AREF
 $Comp
-L GND-RESCUE-arduino_atmega88 #PWR016
+L arduino_atmega88-rescue:GND-RESCUE-arduino_atmega88 #PWR016
 U 1 1 53317146
 P 10050 1850
@@
 Vin
 $Comp
-L GND-RESCUE-arduino_atmega88 #PWR017
+L arduino_atmega88-rescue:GND-RESCUE-arduino_atmega88 #PWR017
 U 1 1 533170E1
 P 6750 2500
@@
 $EndComp
 $Comp
-L +5V #PWR018
+L power1:+5V #PWR018
 U 1 1 533170C3
 P 6850 2150
@@
 $EndComp
 $Comp
-L +3.3V-RESCUE-arduino_atmega88 #PWR019
+L arduino_atmega88-rescue:+3.3V-RESCUE-arduino_atmega88 #PWR019
 U 1 1 533170BB
 P 7000 2150
@@
 RX
 $Comp
-L GND-RESCUE-arduino_atmega88 #PWR020
+L arduino_atmega88-rescue:GND-RESCUE-arduino_atmega88 #PWR020
 U 1 1 53316F0E
 P 4900 3750
@@
 $EndComp
 $Comp
-L SW_PUSH SW1
+L arduino_atmega88-rescue:SW_PUSH-RESCUE-arduino_atmega88 SW1
 U 1 1 53316EFA
 P 4900 3350
@@
 $EndComp
 $Comp
-L +5V #PWR021
+L power1:+5V #PWR021
 U 1 1 53316DF1
 P 5500 2300
@@
 $EndComp
 $Comp
-L R-RESCUE-arduino_atmega88 R3
+L arduino_atmega88-rescue:R-RESCUE-arduino_atmega88 R3
 U 1 1 53316DE9
 P 4900 2650
@@
 DTR
 $Comp
-L C-RESCUE-arduino_atmega88 C3
+L arduino_atmega88-rescue:C-RESCUE-arduino_atmega88 C3
 U 1 1 53316DBF
 P 5200 2950
@@
 A0
 $Comp
-L GND-RESCUE-arduino_atmega88 #PWR022
+L arduino_atmega88-rescue:GND-RESCUE-arduino_atmega88 #PWR022
 U 1 1 53316CEE
 P 5250 1400
@@
 $EndComp
 $Comp
-L GND-RESCUE-arduino_atmega88 #PWR023
+L arduino_atmega88-rescue:GND-RESCUE-arduino_atmega88 #PWR023
 U 1 1 53316CAD
 P 4650 1400
@@
 $EndComp
 $Comp
-L C-RESCUE-arduino_atmega88 C4
+L arduino_atmega88-rescue:C-RESCUE-arduino_atmega88 C4
 U 1 1 53316C9F
 P 5250 1750
@@
 $EndComp
 $Comp
-L C-RESCUE-arduino_atmega88 C2
+L arduino_atmega88-rescue:C-RESCUE-arduino_atmega88 C2
 U 1 1 53316C9B
 P 4650 1750
@@
 $EndComp
 $Comp
-L CRYSTAL X1
+L arduino_atmega88-rescue:CRYSTAL-RESCUE-arduino_atmega88 X1
 U 1 1 53316C89
 P 4950 2100
@@
 D8
 $Comp
-L ATMEGA88A-A IC1
+L arduino_atmega88-rescue:ATMEGA88A-A-RESCUE-arduino_atmega88 IC1
 U 1 1 53316A2F
 P 3050 2600
@@
 $EndComp
 $Comp
-L ARDUINO_SHIELD SHIELD1
+L arduino_shieldsNCL:ARDUINO_SHIELD SHIELD1
 U 1 1 5331693A
 P 8450 2500
@@
 $EndComp
 $Comp
-L R-RESCUE-arduino_atmega88 R4
+L arduino_atmega88-rescue:R-RESCUE-arduino_atmega88 R4
 U 1 1 5452671C
 P 4600 2500
@@
 Wire Wire Line
 	8800 5800 8800 6000
+Wire Wire Line
+	1750 1600 1750 1500
+Wire Wire Line
+	1750 3800 1750 3700
+Wire Wire Line
+	4900 2950 4050 2950
+Wire Wire Line
+	4900 2950 4900 3050
+Wire Wire Line
+	5250 2100 5250 1950
+Wire Wire Line
+	7400 2400 6750 2400
+Wire Wire Line
+	1750 3700 1750 3600
+Wire Wire Line
+	1750 1500 1750 1400
+Wire Wire Line
+	1650 5350 1650 5550
+Wire Wire Line
+	2700 5350 2600 5350
+Wire Wire Line
+	4700 2200 5250 2200
+Wire Wire Line
+	4500 2100 4050 2100
 $EndSCHEMATC
