File: kicad/arduino_based_cdc_emulator/atmega88_k9spud/arduino_based_cdc_emu.sch (KiCad schematic (older format))
At the start: 14 parts, among them IC1 ATMEGA88-A, P1 CONN_5, P2 CONN_2, U1 78L05, X1 20MHz

Commit message: to fcking much changes to commit it separatly, lets go with everything in one commit, git will love me for sure :D
Parts:
- 2u2: symbol CP -> arduino_based_cdc_emu-rescue:CP-RESCUE-arduino_based_cdc_emu
- C1, C2, C3, C4: symbol C-RESCUE-arduino_based_cdc_emu -> arduino_based_cdc_emu-rescue:C-RESCUE-arduino_based_cdc_emu
- IC1: symbol ATMEGA88-A-RESCUE-arduino_based_cdc_emu -> arduino_based_cdc_emu-rescue:ATMEGA88-A-RESCUE-arduino_based_cdc_emu
- P1: symbol CONN_5 -> arduino_based_cdc_emu-rescue:CONN_5-RESCUE-arduino_based_cdc_emu
- P2: symbol CONN_01X03 -> arduino_based_cdc_emu-rescue:CONN_01X03-RESCUE-arduino_based_cdc_emu
- R1, R2, R3, R4: symbol R-RESCUE-arduino_based_cdc_emu -> arduino_based_cdc_emu-rescue:R-RESCUE-arduino_based_cdc_emu
- U1: symbol 78L05 -> arduino_based_cdc_emu-rescue:78L05-RESCUE-arduino_based_cdc_emu
- X1: symbol CRYSTAL -> arduino_based_cdc_emu-rescue:CRYSTAL-RESCUE-arduino_based_cdc_emu
Connections:
- wire segments 45 -> 55
Changed lines of the file:
@@
-EESchema Schematic File Version 2
-LIBS:arduino_based_cdc_emu-rescue
-LIBS:power
-LIBS:device
-LIBS:transistors
-LIBS:conn
-LIBS:linear
-LIBS:regul
-LIBS:74xx
-LIBS:cmos4000
-LIBS:adc-dac
-LIBS:memory
-LIBS:xilinx
-LIBS:microcontrollers
-LIBS:dsp
-LIBS:microchip
-LIBS:analog_switches
-LIBS:motorola
-LIBS:texas
-LIBS:intel
-LIBS:audio
-LIBS:interface
-LIBS:digital-audio
-LIBS:philips
-LIBS:display
-LIBS:cypress
-LIBS:siliconi
-LIBS:opto
-LIBS:atmel
-LIBS:contrib
-LIBS:valves
+EESchema Schematic File Version 4
 LIBS:arduino_based_cdc_emu-cache
-EELAYER 25 0
+EELAYER 26 0
 EELAYER END
 $Descr A4 11693 8268
@@
 Connection ~ 3850 4950
 Wire Wire Line
-	3750 4950 4250 4950
+	3750 4950 3850 4950
 Wire Wire Line
 	4250 4950 4250 5200
 Wire Wire Line
-	4250 5550 3750 5550
+	4250 5550 3850 5550
 Connection ~ 3850 5550
 Connection ~ 3350 5550
@@
 	8650 5850 8650 6050
 Wire Wire Line
-	8550 5450 8950 5450
+	8550 5450 8650 5450
 Wire Wire Line
 	9350 5750 9350 6050
@@
 	7300 4150 6850 4150
 Wire Wire Line
-	6850 5300 7500 5300
+	6850 5300 7300 5300
 Wire Wire Line
 	6350 5300 6150 5300
 $Comp
-L +5V #PWR01
+L power:+5V #PWR01
 U 1 1 53207304
 P 7300 5250
@@
 $EndComp
 $Comp
-L R-RESCUE-arduino_based_cdc_emu R3
+L arduino_based_cdc_emu-rescue:R-RESCUE-arduino_based_cdc_emu R3
 U 1 1 532072FD
 P 6600 5300
@@
 DataOut
 $Comp
-L CONN_5 P1
+L arduino_based_cdc_emu-rescue:CONN_5-RESCUE-arduino_based_cdc_emu P1
 U 1 1 530C9435
 P 10100 3150
@@
 $EndComp
 $Comp
-L +12V #PWR02
+L power:+12V #PWR02
 U 1 1 530C8041
 P 8550 5300
@@
 $EndComp
 $Comp
-L +5V #PWR03
+L power:+5V #PWR03
 U 1 1 530C8014
 P 10000 5350
@@
 $EndComp
 $Comp
-L 78L05 U1
+L arduino_based_cdc_emu-rescue:78L05-RESCUE-arduino_based_cdc_emu U1
 U 1 1 530C7FFF
 P 9350 5500
@@
 $EndComp
 $Comp
-L C-RESCUE-arduino_based_cdc_emu C4
+L arduino_based_cdc_emu-rescue:C-RESCUE-arduino_based_cdc_emu C4
 U 1 1 530C7FE2
 P 10000 5650
@@
 $EndComp
 $Comp
-L C-RESCUE-arduino_based_cdc_emu C3
+L arduino_based_cdc_emu-rescue:C-RESCUE-arduino_based_cdc_emu C3
 U 1 1 530C7FD9
 P 8650 5650
@@
 $EndComp
 $Comp
-L R-RESCUE-arduino_based_cdc_emu R2
+L arduino_based_cdc_emu-rescue:R-RESCUE-arduino_based_cdc_emu R2
 U 1 1 530C78F0
 P 6600 4350
@@
 $EndComp
 $Comp
-L R-RESCUE-arduino_based_cdc_emu R1
+L arduino_based_cdc_emu-rescue:R-RESCUE-arduino_based_cdc_emu R1
 U 1 1 530C77F4
 P 6600 4150
@@
 $EndComp
 $Comp
-L R-RESCUE-arduino_based_cdc_emu R4
+L arduino_based_cdc_emu-rescue:R-RESCUE-arduino_based_cdc_emu R4
 U 1 1 530C77E3
 P 6600 5650
@@
 $EndComp
 $Comp
-L +5V #PWR04
+L power:+5V #PWR04
 U 1 1 530C77C0
 P 4200 3650
@@
 $EndComp
 $Comp
-L C-RESCUE-arduino_based_cdc_emu C2
+L arduino_based_cdc_emu-rescue:C-RESCUE-arduino_based_cdc_emu C2
 U 1 1 530C7707
 P 3550 5550
@@
 $EndComp
 $Comp
-L C-RESCUE-arduino_based_cdc_emu C1
+L arduino_based_cdc_emu-rescue:C-RESCUE-arduino_based_cdc_emu C1
 U 1 1 530C7703
 P 3550 4950
@@
 $EndComp
 $Comp
-L CRYSTAL X1
+L arduino_based_cdc_emu-rescue:CRYSTAL-RESCUE-arduino_based_cdc_emu X1
 U 1 1 530C76D9
 P 3850 5250
@@
 $EndComp
 $Comp
-L ATMEGA88-A-RESCUE-arduino_based_cdc_emu IC1
+L arduino_based_cdc_emu-rescue:ATMEGA88-A-RESCUE-arduino_based_cdc_emu IC1
 U 1 1 530C76C5
 P 5150 4950
@@
 $EndComp
 $Comp
-L +12V #PWR05
+L power:+12V #PWR05
 U 1 1 543549B8
 P 9050 3200
@@
 $EndComp
 Wire Wire Line
-	4200 4450 4200 3650
+	4200 4450 4200 4150
 Wire Wire Line
 	4250 4150 4200 4150
@@
 	4250 5950 4200 5950
 Wire Wire Line
-	4200 5950 4200 6300
+	4200 5950 4200 6050
 Wire Wire Line
 	4250 6050 4200 6050
@@
 	10000 5450 9750 5450
 $Comp
-L CONN_01X03 P2
+L arduino_based_cdc_emu-rescue:CONN_01X03-RESCUE-arduino_based_cdc_emu P2
 U 1 1 54357812
 P 9950 4400
@@
 NoConn ~ 6150 3850
 $Comp
-L GND #PWR06
+L power:GND #PWR06
 U 1 1 564E2443
 P 4200 6300
@@
 $EndComp
 $Comp
-L GND #PWR07
+L power:GND #PWR07
 U 1 1 564E2722
 P 3350 5700
@@
 $EndComp
 $Comp
-L GND #PWR08
+L power:GND #PWR08
 U 1 1 564E291B
 P 8650 6050
@@
 $EndComp
 $Comp
-L GND #PWR09
+L power:GND #PWR09
 U 1 1 564E2BE7
 P 9350 6050
@@
 $EndComp
 $Comp
-L GND #PWR010
+L power:GND #PWR010
 U 1 1 564E2C19
 P 10000 6050
@@
 $EndComp
 $Comp
-L GND #PWR011
+L power:GND #PWR011
 U 1 1 564E2EC9
 P 9550 4600
@@
 $EndComp
 $Comp
-L GND #PWR012
+L power:GND #PWR012
 U 1 1 564E3127
 P 9600 3400
@@
 $EndComp
 $Comp
-L GND #PWR013
+L power:GND #PWR013
 U 1 1 564E32CC
 P 7500 5900
@@
 $EndComp
 $Comp
-L CP 2u2
+L arduino_based_cdc_emu-rescue:CP-RESCUE-arduino_based_cdc_emu 2u2
 U 1 1 564E32FE
 P 7500 5550
@@
 	4250 4450 4200 4450
 Wire Wire Line
-	3350 4950 3350 5700
+	3350 4950 3350 5550
+Wire Wire Line
+	3850 4950 4250 4950
+Wire Wire Line
+	3850 5550 3750 5550
+Wire Wire Line
+	3350 5550 3350 5700
+Wire Wire Line
+	4200 4150 4200 3950
+Wire Wire Line
+	4200 3950 4200 3850
+Wire Wire Line
+	4200 3850 4200 3650
+Wire Wire Line
+	4200 6050 4200 6150
+Wire Wire Line
+	4200 6150 4200 6300
+Wire Wire Line
+	8650 5450 8950 5450
+Wire Wire Line
+	7300 5300 7500 5300
 $EndSCHEMATC
