File: kicad/arduino_based_cdc_emulator/atmegax8_with_bluetooth/atmegax8_with_bluetooth.kicad_pcb (KiCad board)
At the start: 2 copper layers, 40.9 x 35.7 mm, 66 parts, among them IC1 ATMEGA88-A, P1 CONN_9, P2 SPI, Q1 BC817-40, U1 78L05, U2 S3860M-S, U3 LM358, X1 16MHz

Commit message: to fcking much changes to commit it separatly, lets go with everything in one commit, git will love me for sure :D
Parts:
- removed C1, C2: 22p, Capacitors_SMD:C_0805_HandSoldering
- removed L2: 15n, SMD_Packages:SMD-1206_Pol
- removed X1: 16MHz, Crystals:Crystal_HC49-SD_SMD
- added C26: 10n, Capacitors_SMD:C_0805_HandSoldering, B.Cu at (80.1, 145.1)
- added C27: 1u/10V, Capacitors_SMD:C_0805_HandSoldering, F.Cu at (79.2, 143.4)
- added C28: 100n, Capacitors_SMD:C_0805_HandSoldering, B.Cu at (86.4, 147.6)
- added D2: LED, LEDs:LED_0805_HandSoldering, B.Cu at (102.1, 142.4)
- added D3: LED, LEDs:LED_0805_HandSoldering, B.Cu at (100.0, 142.4)
- added P3: CONN_4, Pin_Headers.pretty:Pin_Header_Straight_1x04, F.Cu at (107.6, 147.5)
- added R31: 1k, Resistors_SMD:R_0805_HandSoldering, B.Cu at (99.9, 147.4)
- added Y1: Crystal_GND2, modules:MURATA_CSTCE_V53, F.Cu at (87.1, 166.2)
- C19: footprint Capacitors_SMD:c_elec_5x5.8 -> Capacitors_SMD:CP_Elec_5x5.8
- C24, P2, R7: moved to F.Cu
- L1: value INDUCTOR -> 330u
- R25: value 4k7 -> 1k2
- R26: value 330 -> 1k; moved to B.Cu
- R27: value 2k7(3k3) -> 1k2
- U2: value S3860M-S -> F-6188; footprint my_modules:S3860M-S -> modules:F-6188_nosilk
- moved C24 27.1 mm to (96.2, 167.8), turned to 0 degrees
- moved R25 26.8 mm to (79.0, 151.7), turned to 180 degrees
- moved P2 24.4 mm to (102.0, 165.2), turned to 0 degrees
- moved R7 21.3 mm to (95.4, 165.6), turned to 0 degrees
- moved R26 8.43 mm to (102.1, 147.4), turned to 90 degrees
- moved R6 6.22 mm to (89.4, 165.1), turned to 270 degrees
- moved R19 4.53 mm to (98.9, 142.9)
- moved R5 4.04 mm to (91.6, 165.1), turned to 90 degrees
- moved U2 3.39 mm to (94.0, 152.1)
- moved D1 2.33 mm to (97.4, 144.8), turned to 270 degrees
- moved R13 1.74 mm to (97.7, 148.9)
- moved R14 1.74 mm to (97.6, 146.8)
- moved C19 1.60 mm to (86.6, 151.8), turned to 0 degrees
- moved R9 1.53 mm to (77.2, 143.5)
- moved R11 1.04 mm to (75.2, 143.5)
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Connections:
- net /MIC_IN renamed /MIC_IN2
- C19 pad 2: /BTAGND -> /BTOUTRN
- C21 pad 2: /BTAGND -> /BTOUTLN
- C23 pad 1: /MIC -> /MICP
- IC1 pad 24: /BT_ENABLE -> (no net)
- P1 pad 5: GND -> /MIC_IN1
- R25 pad 1: Net-(R25-Pad1) -> GND
- R25 pad 2: GND -> /MIC_IN1
- R26 pad 1: Net-(R25-Pad1) -> /LED1
- R26 pad 2: /BT_ENABLE -> Net-(D2-Pad2)
- R27 pad 2: Net-(L2-Pad2) -> /MIC_BIAS
- U2 pad 1: (no net) -> GND
- U2 pad 10: (no net) -> TX
- U2 pad 11: GND -> RX
- U2 pad 12: +BATT -> (no net)
- U2 pad 13: (no net) -> /LED1
- U2 pad 14: (no net) -> /LED2
- U2 pad 16: (no net) -> GND
- U2 pad 17: /BT_RESET -> GND
- U2 pad 18: (no net) -> /IN_DETECT
- U2 pad 19: Net-(R25-Pad1) -> /INR
- U2 pad 2: /BTAGND -> (no net)
- U2 pad 20: RX -> /INL
- U2 pad 21: TX -> /MICN
- U2 pad 22: (no net) -> /MICP
- U2 pad 23: (no net) -> /MIC_BIAS
- U2 pad 24: (no net) -> /BTOUTLN
- U2 pad 25: (no net) -> /BTOUTL
- U2 pad 3: /BTOUTL -> GND
- U2 pad 4: /BTOUTR -> (no net)
- U2 pad 5: /MIC -> (no net)
- U2 pad 6: /MIC_BIAS -> (no net)
- U2 pad 8: (no net) -> /BT_RESET
Routing:
- net GND: track 169.3 -> 106.1 mm, vias 0 -> 4
- net /MICP: track 0.00 -> 44.9 mm, vias 0 -> 2
- net /BTOUTRN: track 0.00 -> 39.8 mm, vias 0 -> 2
- net +BATT: track 20.7 -> 60.1 mm, vias 0 -> 2
- net /MICN: track 0.00 -> 39.3 mm, vias 0 -> 3
- net /MOSI: track 45.1 -> 9.68 mm
- net /MISO: track 35.4 -> 4.28 mm
- net TX: track 30.7 -> 2.51 mm, vias 1 -> 0
- net /SCK: track 35.9 -> 8.14 mm, vias 0 -> 2
- net /BTOUTR: track 7.47 -> 34.5 mm, vias 0 -> 2
- net /MIC: track 26.9 -> 0.00 mm
- net /BTAGND: track 26.5 -> 0.00 mm
- net /BTOUTLN: track 0.00 -> 26.2 mm, vias 0 -> 2
- net RX: track 26.1 -> 0.00 mm, vias 1 -> 0
- net +5V: track 94.3 -> 70.5 mm, vias 6 -> 5
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Other:
- board size 40.9 x 35.7 mm -> 110.5 x 172.6 mm
