File: kicad/arduino_based_cdc_emulator/atmegax8_with_bluetooth/atmegax8_with_bluetooth.sch (KiCad schematic (older format))
At the start: 66 parts, among them IC1 ATMEGA88-A, P1 CONN_9, P2 SPI, Q1 BC817-40, U1 78L05, U2 S3860M-S, U3 LM358, X1 16MHz

Commit message: to fcking much changes to commit it separatly, lets go with everything in one commit, git will love me for sure :D
Parts:
- removed C1, C2: 22p, Capacitors_SMD:C_0805_HandSoldering, symbol C
- removed L2: 15n, SMD_Packages:SMD-1206_Pol, symbol INDUCTOR
- removed Q1: BC817-40, TO_SOT_Packages_SMD:SOT-23, symbol BC817-40
- removed R25: 4k7, Resistors_SMD:R_0805_HandSoldering, symbol R
- removed R26: 330, Resistors_SMD:R_0805_HandSoldering, symbol R
- removed R28: 47k, Resistors_SMD:R_0805_HandSoldering, symbol R
- removed R30: 10k, Resistors_SMD:R_0805_HandSoldering, symbol R
- removed U2: S3860M-S, my_modules:S3860M-S, symbol S3860M-S
- removed X1: 16MHz, Crystals:Crystal_HC49-SD_SMD, symbol Crystal
- added C26: 10n, Capacitors_SMD:C_0805_HandSoldering, symbol atmegax8_with_bluetooth-rescue:C-RESCUE-atmegax8_with_bluetooth
- added C27: 1u/10V, Capacitors_SMD:C_0805_HandSoldering, symbol atmegax8_with_bluetooth-rescue:C-RESCUE-atmegax8_with_bluetooth
- added C28: 100n, Capacitors_SMD:C_0805_HandSoldering, symbol atmegax8_with_bluetooth-rescue:C-RESCUE-atmegax8_with_bluetooth
- added D2, D3: LED, LEDs:LED_0805_HandSoldering, symbol atmegax8_with_bluetooth-rescue:LED-RESCUE-atmegax8_with_bluetooth
- added D?: D_Zener, Diodes_SMD.pretty:MiniMELF_Handsoldering, symbol Device:D_Zener
- added JP?: Jumper_3_Bridged12, symbol Jumper:Jumper_3_Bridged12
- added P3: CONN_4, Pin_Headers.pretty:Pin_Header_Straight_1x04, symbol atmegax8_with_bluetooth-rescue:Conn_01x04-RESCUE-atmegax8_with_bluetooth
- added R25: 1k2, Resistors_SMD:R_0805_HandSoldering, symbol atmegax8_with_bluetooth-rescue:R-RESCUE-atmegax8_with_bluetooth
- added R26, R31: 1k, Resistors_SMD:R_0805_HandSoldering, symbol atmegax8_with_bluetooth-rescue:R-RESCUE-atmegax8_with_bluetooth
- added U2: F-6188, modules:F-6188_nosilk, symbol F-6188:F-6188
- added Y1: Crystal_GND2, modules:MURATA_CSTCE_V53, symbol Device:Crystal_GND2
- C10, C11, C13, C14, C20, C21, C24, C25, C6, C9: symbol CP -> atmegax8_with_bluetooth-rescue:CP-RESCUE-atmegax8_with_bluetooth
- C12, C15, C16, C17, C18, C22, C23, C3, C4, C5, C7, C8: symbol C -> atmegax8_with_bluetooth-rescue:C-RESCUE-atmegax8_with_bluetooth
- C19: footprint Capacitors_SMD:c_elec_5x5.8 -> Capacitors_SMD:CP_Elec_5x5.8; symbol CP -> atmegax8_with_bluetooth-rescue:CP-RESCUE-atmegax8_with_bluetooth
- D1: symbol D -> atmegax8_with_bluetooth-rescue:D-RESCUE-atmegax8_with_bluetooth
- IC1: symbol ATMEGA88-A -> atmegax8_with_bluetooth-rescue:ATMEGA88-A-RESCUE-atmegax8_with_bluetooth
- L1: value INDUCTOR -> 330u; symbol INDUCTOR -> atmegax8_with_bluetooth-rescue:INDUCTOR-RESCUE-atmegax8_with_bluetooth
- P1: value CONN_9 -> CONN_10; footprint Pin_Headers:Pin_Header_Straight_1x11 -> Pin_Headers:Pin_Header_Straight_1x12; symbol CONN_01X11 -> gencon:CONN_12
- P2: symbol CONN_02X03 -> atmegax8_with_bluetooth-rescue:CONN_02X03-RESCUE-atmegax8_with_bluetooth
- R1, R10, R11, R12, R13, R14, R15, R16, R17, R18, R19, R2, R20, R21, R22, R23, R24, R29, R3, R4, R5, R6, R7, R8, R9: symbol R -> atmegax8_with_bluetooth-rescue:R-RESCUE-atmegax8_with_bluetooth
- R27: value 2k7(3k3) -> 1k2; symbol R -> atmegax8_with_bluetooth-rescue:R-RESCUE-atmegax8_with_bluetooth
- U1: symbol 78L05 -> atmegax8_with_bluetooth-rescue:78L05-RESCUE-atmegax8_with_bluetooth
- U3: symbol LM358 -> atmegax8_with_bluetooth-rescue:LM358-RESCUE-atmegax8_with_bluetooth
Connections:
- net labels added: BTOUTLN, BTOUTRN, INL, INR, IN_DETECT, MICN, MICP, MIC_IN1, MIC_IN2, MUTE
- net labels removed: BTAGND, BT_ENABLE, MIC, MIC_IN
- wire segments 186 -> 262
- no-connect marks 17 -> 16
