File: kicad/arduino_based_cdc_emulator/atmegax8_with_bluetooth/atmegax8_with_bluetooth.sch (KiCad schematic (older format))
At the start: 69 parts, among them IC1 ATMEGA88-A, P1 CONN_10, P2 SPI, P3 CONN_4, U1 78L05, U2 F-6188, U3 LM358, Y1 Crystal_GND2

Commit message: update
Parts:
- P1: symbol gencon:CONN_12 -> atmegax8_with_bluetooth-rescue:CONN_12-gencon
- U2: symbol F-6188:F-6188 -> atmegax8_with_bluetooth-rescue:F-6188-F-6188
Changed lines of the file:
@@
 EESchema Schematic File Version 4
 LIBS:atmegax8_with_bluetooth-cache
-EELAYER 26 0
+EELAYER 29 0
 EELAYER END
 $Descr A3 16535 11693
@@
 DataOut
 $Comp
-L gencon:CONN_12 P1
+L atmegax8_with_bluetooth-rescue:CONN_12-gencon P1
 U 1 1 530C9435
 P 8300 9900
@@
 MIC_IN2
 $Comp
-L F-6188:F-6188 U2
+L atmegax8_with_bluetooth-rescue:F-6188-F-6188 U2
 U 1 1 59FC4A54
 P 9850 7600

Commit message: changes to bt version, but it is not good, do not use this setup
Parts:
- removed C24: 2u2, Capacitors_Tantalum_SMD:TantalC_SizeA_EIA-3216_HandSoldering, symbol atmegax8_with_bluetooth-rescue:CP-RESCUE-atmegax8_with_bluetooth
- removed C25: 2u1, Capacitors_Tantalum_SMD:TantalC_SizeA_EIA-3216_HandSoldering, symbol atmegax8_with_bluetooth-rescue:CP-RESCUE-atmegax8_with_bluetooth
- removed D?: D_Zener, Diodes_SMD.pretty:MiniMELF_Handsoldering, symbol Device:D_Zener
- removed JP?: Jumper_3_Bridged12, symbol Jumper:Jumper_3_Bridged12
- removed R29: 10k, Resistors_SMD:R_0805_HandSoldering, symbol atmegax8_with_bluetooth-rescue:R-RESCUE-atmegax8_with_bluetooth
- removed U1: 78L05, my_modules:SOT-223-REGULATOR, symbol atmegax8_with_bluetooth-rescue:78L05-RESCUE-atmegax8_with_bluetooth
- added C1, C24: 100n, Capacitors_SMD:C_0805_HandSoldering, symbol atmegax8_with_bluetooth-rescue:C-RESCUE-atmegax8_with_bluetooth
- added J1: Ant, modules:1pin_smd, symbol Connector_Generic:Conn_01x01
- added J2: TMS, modules:1pin_smd, symbol Connector_Generic:Conn_01x01
- added J3: TCK, modules:1pin_smd, symbol Connector_Generic:Conn_01x01
- added J4: TDO, modules:1pin_smd, symbol Connector_Generic:Conn_01x01
- added J5: TDI, modules:1pin_smd, symbol Connector_Generic:Conn_01x01
- added P4: SERIAL, Pin_Headers:Pin_Header_Straight_1x02_Pitch2.54mm, symbol Connector:Conn_01x02_Male
- added P5: CONN_4, Pin_Headers.pretty:Pin_Header_Straight_1x03, symbol Connector:Conn_01x03_Male
- added U4, U5: MAX809, TO_SOT_Packages_SMD.pretty:SOT-23, symbol MAX809_810:MAX809
- C10: value 100m/25V -> 100u/16V; footprint Capacitors_SMD:c_elec_6.3x7.7 -> Capacitors_Tantalum_SMD:CP_Tantalum_Case-D_EIA-7343-31_Hand; symbol atmegax8_with_bluetooth-rescue:CP-RESCUE-atmegax8_with_bluetooth -> Device:CP
- C11: value 47m/25V -> 100m/16V; footprint Capacitors_Tantalum_SMD:TantalC_SizeD_EIA-7343_HandSoldering -> Capacitors_Tantalum_SMD:CP_Tantalum_Case-D_EIA-7343-31_Hand
- C22: footprint Capacitors_SMD:C_1206_HandSoldering -> Capacitors_Tantalum_SMD.pretty:TantalC_SizeA_EIA-3216_Wave; symbol atmegax8_with_bluetooth-rescue:C-RESCUE-atmegax8_with_bluetooth -> Device:CP
- C23, C27: footprint Capacitors_SMD:C_0805_HandSoldering -> Capacitors_SMD:C_1206_HandSoldering; symbol atmegax8_with_bluetooth-rescue:C-RESCUE-atmegax8_with_bluetooth -> Device:C
- D1: footprint Diodes_SMD:MiniMELF_Handsoldering -> Diodes_SMD:D_MiniMELF
- P1: footprint Pin_Headers:Pin_Header_Straight_1x12 -> Pin_Headers:Pin_Header_Straight_1x12_Pitch2.54mm
- R3, R7: value 3k3 -> 100
- R5: value 27 -> 20
- Y1: value Crystal_GND2 -> 16MHz
Connections:
- net +12V: now also P1.5; no longer C3.1, P1.7
- net +5V: now also C1.1, C24.1, P5.1 (Pin_1), U5.3 (VCC); no longer R3.2
- net +BATT: now also U4.3 (VCC); no longer R7.2
- net ARESET: now also R3.2; no longer R3.1
- net BTOUTL: now also C20.1; no longer C6.1
- net BTOUTLN: now also C19.2; no longer C21.2
- net BTOUTR: now also C6.1; no longer C20.1
- net BTOUTRN: now also C21.2; no longer C19.2
- net BT_RESET: now also R7.2; no longer R7.1
- net CDC_ENA_12V: now also C3.1, P5.3 (Pin_3)
- net GND: now also C1.2, C24.2, P5.2 (Pin_2), U4.1 (GND), U5.1 (GND); no longer C10.2
- net GNDA: now also C10.2
- net MIC_IN1: now also P1.7; no longer P1.6
- net MIC_IN2: now also P1.6; no longer P1.5
- net at IC1.12 ((PCINT0/CLKO/ICP1)PB0): now also R4.1
- net at IC1.30 ((PCINT16/RXD)PD0), R13.1: now also P4.2 (Pin_2)
- net at IC1.31 ((PCINT17/TXD)PD1), R14.1: now also P4.1 (Pin_1)
- net at U2.2 (ANT): now also J1.1 (Pin_1)
- net at U2.4 (TMS/GPIO19): now also J2.1 (Pin_1)
- net at U2.5 (TCK/GPIO18): now also J3.1 (Pin_1)
- net at U2.6 (TDO/GPIO21): now also J4.1 (Pin_1)
- net at U2.7 (TDI/GPIO20): now also J5.1 (Pin_1)
- new net: R3.1, U5.2 (RESET)
- new net: R7.1, U4.2 (RESET)
Other:
- moved on the sheet: C14, C15, C16, C17, C18, C19, C20, C21, C23, C26, C27, C28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
