File: kicad/audio_preamplifier/audio_preamplifier.sch (KiCad schematic (older format))
At the start: 22 parts, among them P2 CONN_01X03, P3 CONN_01X03, U3 TL072

Commit message: to fcking much changes to commit it separatly, lets go with everything in one commit, git will love me for sure :D
Parts:
- C1, C4, C5, C6, C7, C8, C9: symbol CP -> audio_preamplifier-rescue:CP
- C11: symbol C -> audio_preamplifier-rescue:C
- L1: symbol INDUCTOR -> audio_preamplifier-rescue:INDUCTOR
- P2: symbol CONN_01X03 -> audio_preamplifier-rescue:CONN_01X03
- P3: symbol CONN_01X05 -> audio_preamplifier-rescue:CONN_01X05
- R10, R11, R12, R13, R14, R15, R16, R17, R8, R9: symbol R -> audio_preamplifier-rescue:R
- U3: symbol TL072-RESCUE-audio_preamplifier -> audio_preamplifier-rescue:TL072-RESCUE-audio_preamplifier
Changed lines of the file:
@@
-EESchema Schematic File Version 2
-LIBS:audio_preamplifier-rescue
-LIBS:power
-LIBS:device
-LIBS:transistors
-LIBS:conn
-LIBS:linear
-LIBS:regul
-LIBS:74xx
-LIBS:cmos4000
-LIBS:adc-dac
-LIBS:memory
-LIBS:xilinx
-LIBS:microcontrollers
-LIBS:dsp
-LIBS:microchip
-LIBS:analog_switches
-LIBS:motorola
-LIBS:texas
-LIBS:intel
-LIBS:audio
-LIBS:interface
-LIBS:digital-audio
-LIBS:philips
-LIBS:display
-LIBS:cypress
-LIBS:siliconi
-LIBS:opto
-LIBS:atmel
-LIBS:contrib
-LIBS:valves
+EESchema Schematic File Version 4
 LIBS:audio_preamplifier-cache
-EELAYER 25 0
+EELAYER 26 0
 EELAYER END
 $Descr A4 11693 8268
@@
 $EndDescr
 $Comp
-L AGND #PWR01
+L audio_preamplifier-rescue:AGND #PWR01
 U 1 1 52EA33C9
 P 3700 6700
@@
 $EndComp
 $Comp
-L AGND #PWR02
+L audio_preamplifier-rescue:AGND #PWR02
 U 1 1 52EA33C7
 P 2700 6650
@@
 $EndComp
 $Comp
-L AGND #PWR03
+L audio_preamplifier-rescue:AGND #PWR03
 U 1 1 52EA31C6
 P 8100 4000
@@
 $EndComp
 $Comp
-L AGND #PWR04
+L audio_preamplifier-rescue:AGND #PWR04
 U 1 1 52E92164
 P 3750 4550
@@
 $EndComp
 $Comp
-L AGND #PWR05
+L audio_preamplifier-rescue:AGND #PWR05
 U 1 1 52E92160
 P 3800 2550
@@
 $EndComp
 $Comp
-L AGND #PWR06
+L audio_preamplifier-rescue:AGND #PWR06
 U 1 1 52E91F4E
 P 2150 2500
@@
 $EndComp
 $Comp
-L AGND #PWR07
+L audio_preamplifier-rescue:AGND #PWR07
 U 1 1 52E91F46
 P 2100 4550
@@
 $EndComp
 $Comp
-L AGND #PWR08
+L audio_preamplifier-rescue:AGND #PWR08
 U 1 1 52E91F01
 P 5700 6850
@@
 $EndComp
 $Comp
-L C C11
+L audio_preamplifier-rescue:C C11
 U 1 1 52E79ACE
 P 4150 6300
@@
 $EndComp
 $Comp
-L INDUCTOR L1
+L audio_preamplifier-rescue:INDUCTOR L1
 U 1 1 52E771D7
 P 3150 5900
@@
 $EndComp
 $Comp
-L CP C1
+L audio_preamplifier-rescue:CP C1
 U 1 1 52E771C6
 P 2700 6250
@@
 $EndComp
 $Comp
-L CP C4
+L audio_preamplifier-rescue:CP C4
 U 1 1 52E56B09
 P 3700 6300
@@
 $EndComp
 $Comp
-L AGND #PWR09
+L audio_preamplifier-rescue:AGND #PWR09
 U 1 1 52E56AD2
 P 7500 3500
@@
 $EndComp
 $Comp
-L AGND #PWR010
+L audio_preamplifier-rescue:AGND #PWR010
 U 1 1 52E56ACB
 P 7400 2400
@@
 $EndComp
 $Comp
-L +12V #PWR011
+L audio_preamplifier-rescue:+12V #PWR011
 U 1 1 52D3D406
 P 7250 3550
@@
 right_out
 $Comp
-L +12V #PWR012
+L audio_preamplifier-rescue:+12V #PWR012
 U 1 1 52D3D226
 P 2700 5800
@@
 left_out
 $Comp
-L CP C5
+L audio_preamplifier-rescue:CP C5
 U 1 1 52D3D19D
 P 5400 6450
@@
 $EndComp
 $Comp
-L R R9
+L audio_preamplifier-rescue:R R9
 U 1 1 52D3D170
 P 5700 6500
@@
 $EndComp
 $Comp
-L R R8
+L audio_preamplifier-rescue:R R8
 U 1 1 52D3D16C
 P 5700 5850
@@
 $EndComp
 $Comp
-L CP C8
+L audio_preamplifier-rescue:CP C8
 U 1 1 52D3D12D
 P 4750 1850
@@
 $EndComp
 $Comp
-L CP C9
+L audio_preamplifier-rescue:CP C9
 U 1 1 52D3D123
 P 4850 3800
@@
 $EndComp
 $Comp
-L R R11
+L audio_preamplifier-rescue:R R11
 U 1 1 52D3CF9F
 P 2100 4150
@@
 $EndComp
 $Comp
-L R R10
+L audio_preamplifier-rescue:R R10
 U 1 1 52D3CF9C
 P 2150 2200
@@
 $EndComp
 $Comp
-L R R13
+L audio_preamplifier-rescue:R R13
 U 1 1 52D3CF91
 P 2800 4800
@@
 $EndComp
 $Comp
-L R R12
+L audio_preamplifier-rescue:R R12
 U 1 1 52D3CF88
 P 2850 2700
@@
 $EndComp
 $Comp
-L R R15
+L audio_preamplifier-rescue:R R15
 U 1 1 52D3CE54
 P 3350 4850
@@
 $EndComp
 $Comp
-L R R14
+L audio_preamplifier-rescue:R R14
 U 1 1 52D3CE47
 P 3400 2700
@@
 $EndComp
 $Comp
-L R R17
+L audio_preamplifier-rescue:R R17
 U 1 1 52D3CE44
 P 4250 4400
@@
 $EndComp
 $Comp
-L R R16
+L audio_preamplifier-rescue:R R16
 U 1 1 52D3CE2F
 P 4150 2350
@@
 $EndComp
 $Comp
-L CP C7
+L audio_preamplifier-rescue:CP C7
 U 1 1 52D3C91A
 P 2500 3700
@@
 $EndComp
 $Comp
-L CP C6
+L audio_preamplifier-rescue:CP C6
 U 1 1 52D3C8BA
 P 2550 1750
@@
 $EndComp
 $Comp
-L TL072-RESCUE-audio_preamplifier U3
+L audio_preamplifier-rescue:TL072-RESCUE-audio_preamplifier U3
 U 2 1 52D3B907
 P 3850 3800
@@
 $EndComp
 $Comp
-L TL072-RESCUE-audio_preamplifier U3
+L audio_preamplifier-rescue:TL072-RESCUE-audio_preamplifier U3
 U 1 1 52D3B8FE
 P 3900 1850
@@
 $EndComp
 $Comp
-L CONN_01X05 P3
+L audio_preamplifier-rescue:CONN_01X05 P3
 U 1 1 54F9D72B
 P 8400 3550
@@
 $EndComp
 $Comp
-L CONN_01X03 P2
+L audio_preamplifier-rescue:CONN_01X03 P2
 U 1 1 54F9D9C9
 P 8350 2250
@@
 $EndComp
 $Comp
-L AGND #PWR013
+L audio_preamplifier-rescue:AGND #PWR013
 U 1 1 560EBEB5
 P 4150 6700
@@
 	5400 6600 5400 6800
 Wire Wire Line
-	4400 1850 4600 1850
-Wire Wire Line
-	2650 3700 3350 3700
+	4400 1850 4500 1850
+Wire Wire Line
+	2650 3700 2800 3700
 Wire Wire Line
 	3400 2850 3400 3100
 Wire Wire Line
-	3400 1950 3400 2550
-Wire Wire Line
-	4350 3800 4700 3800
-Wire Wire Line
-	5700 6650 5700 6850
+	3400 1950 3400 2350
+Wire Wire Line
+	4350 3800 4550 3800
+Wire Wire Line
+	5700 6650 5700 6800
 Wire Wire Line
 	4900 1850 5100 1850
 Wire Wire Line
-	1500 3700 2350 3700
+	1500 3700 2100 3700
 Wire Wire Line
 	8150 3550 8200 3550
@@
 	3700 6450 3700 6700
 Wire Wire Line
-	2700 5800 2700 6100
-Wire Wire Line
-	3450 5900 4950 5900
+	2700 5800 2700 5900
+Wire Wire Line
+	3450 5900 3700 5900
 Wire Wire Line
 	4150 5900 4150 6150
@@
 Connection ~ 4500 1850
 Wire Wire Line
-	3350 3900 3350 4700
+	3350 3900 3350 4400
 Wire Wire Line
 	3350 4400 4100 4400
@@
 	5400 6200 5400 6300
 Wire Wire Line
-	5400 6200 6400 6200
-Wire Wire Line
-	5700 6000 5700 6350
+	5400 6200 5700 6200
+Wire Wire Line
+	5700 6000 5700 6200
 Connection ~ 5700 6200
 Wire Wire Line
@@
 	3350 5000 3350 5200
 Wire Wire Line
-	2850 3100 3950 3100
+	2850 3100 3400 3100
 Text Label 3950 3100 2    60   ~ 0
 virtual_gnd
@@
 Connection ~ 3400 3100
 Wire Wire Line
-	2800 5200 3900 5200
+	2800 5200 3350 5200
 Wire Wire Line
 	2100 4300 2100 4550
@@
 	3750 3300 3750 3400
 Wire Wire Line
-	1550 1750 2400 1750
-Wire Wire Line
-	2700 1750 3400 1750
+	1550 1750 2150 1750
+Wire Wire Line
+	2700 1750 2850 1750
 Wire Wire Line
 	8100 3650 8200 3650
 Wire Wire Line
 	7250 3750 8200 3750
+Wire Wire Line
+	2700 5900 2700 6100
+Wire Wire Line
+	3700 5900 4150 5900
+Wire Wire Line
+	4150 5900 4950 5900
+Wire Wire Line
+	3400 2350 3400 2550
+Wire Wire Line
+	4500 1850 4600 1850
+Wire Wire Line
+	3350 4400 3350 4700
+Wire Wire Line
+	4550 3800 4700 3800
+Wire Wire Line
+	5700 6800 5700 6850
+Wire Wire Line
+	5700 6200 6400 6200
+Wire Wire Line
+	5700 6200 5700 6350
+Wire Wire Line
+	3350 5200 3900 5200
+Wire Wire Line
+	2800 3700 3350 3700
+Wire Wire Line
+	2850 1750 3400 1750
+Wire Wire Line
+	3400 3100 3950 3100
+Wire Wire Line
+	2100 3700 2350 3700
+Wire Wire Line
+	2150 1750 2400 1750
 $EndSCHEMATC
