File: kicad/audio_preamplifier/audio_preamplifier.sch (KiCad schematic (older format))
At the start: 22 parts, among them P2 CONN_01X03, P3 CONN_01X03, U3 TL072

Commit message: update
Parts:
- C1: value 100m/25V -> 47m/25V; footprint Capacitors_SMD:c_elec_6.3x7.7 -> Capacitors_Tantalum_SMD:CP_Tantalum_Case-D_EIA-7343-31_Hand
- C11: footprint Capacitors_SMD:C_1206_HandSoldering -> Capacitors_SMD:C_0805_HandSoldering
- C4: footprint Capacitors_Tantalum_SMD:TantalC_SizeD_EIA-7343_HandSoldering -> Capacitors_Tantalum_SMD:CP_Tantalum_Case-D_EIA-7343-31_Hand
- C6, C7: footprint Capacitors_SMD:c_elec_5x5.8 -> Capacitors_SMD:CP_Elec_5x5.8
- C8, C9: value 47m/25V -> 10m/16V; footprint Capacitors_SMD:c_elec_5x5.8 -> Capacitors_SMD:CP_Elec_5x5.8
- L1: footprint (none) -> Inductors.pretty:Inductor_1212
- P2: footprint Pin_Headers:Pin_Header_Straight_1x03 -> Pin_Headers:Pin_Header_Straight_1x03_Pitch2.54mm
- P3: footprint Pin_Headers:Pin_Header_Straight_1x05 -> Pin_Headers:Pin_Header_Straight_1x05_Pitch2.54mm
- R10, R11, R12, R13, R14, R15, R16, R17, R8, R9: footprint Resistors_SMD:R_1206_HandSoldering -> Resistors_SMD:R_0805_HandSoldering
- U3: footprint (none) -> Housings_SOIC:SOIC-8_3.9x4.9mm_Pitch1.27mm
Changed lines of the file:
@@
 EESchema Schematic File Version 4
 LIBS:audio_preamplifier-cache
-EELAYER 26 0
+EELAYER 29 0
 EELAYER END
 $Descr A4 11693 8268
@@
 F 0 "C11" H 4200 6400 50  0000 L CNN
 F 1 "100n" H 4200 6200 50  0000 L CNN
-F 2 "Capacitors_SMD:C_1206_HandSoldering" H 4150 6300 60  0001 C CNN
+F 2 "Capacitors_SMD:C_0805_HandSoldering" H 4150 6300 60  0001 C CNN
 F 3 "" H 4150 6300 60  0001 C CNN
 	1    4150 6300
@@
 F 0 "L1" V 3100 5900 40  0000 C CNN
 F 1 "330uH" V 3250 5900 40  0000 C CNN
-F 2 "" H 3150 5900 60  0001 C CNN
+F 2 "Inductors.pretty:Inductor_1212" H 3150 5900 60  0001 C CNN
 F 3 "" H 3150 5900 60  0001 C CNN
 	1    3150 5900
@@
 P 2700 6250
 F 0 "C1" H 2750 6350 50  0000 L CNN
-F 1 "100m/25V" H 2750 6150 50  0000 L CNN
-F 2 "Capacitors_SMD:c_elec_6.3x7.7" H 2700 6250 60  0001 C CNN
+F 1 "47m/25V" H 2750 6150 50  0000 L CNN
+F 2 "Capacitors_Tantalum_SMD:CP_Tantalum_Case-D_EIA-7343-31_Hand" H 2700 6250 60  0001 C CNN
 F 3 "" H 2700 6250 60  0001 C CNN
 	1    2700 6250
@@
 F 0 "C4" H 3750 6400 50  0000 L CNN
 F 1 "47m/25V" H 3750 6200 50  0000 L CNN
-F 2 "Capacitors_Tantalum_SMD:TantalC_SizeD_EIA-7343_HandSoldering" H 3700 6300 60  0001 C CNN
+F 2 "Capacitors_Tantalum_SMD:CP_Tantalum_Case-D_EIA-7343-31_Hand" H 3700 6300 60  0001 C CNN
 F 3 "" H 3700 6300 60  0001 C CNN
 	1    3700 6300
@@
 F 0 "R9" V 5780 6500 50  0000 C CNN
 F 1 "10k" V 5700 6500 50  0000 C CNN
-F 2 "Resistors_SMD:R_1206_HandSoldering" H 5700 6500 60  0001 C CNN
+F 2 "Resistors_SMD:R_0805_HandSoldering" H 5700 6500 60  0001 C CNN
 F 3 "" H 5700 6500 60  0001 C CNN
 	1    5700 6500
@@
 F 0 "R8" V 5780 5850 50  0000 C CNN
 F 1 "10k" V 5700 5850 50  0000 C CNN
-F 2 "Resistors_SMD:R_1206_HandSoldering" H 5700 5850 60  0001 C CNN
+F 2 "Resistors_SMD:R_0805_HandSoldering" H 5700 5850 60  0001 C CNN
 F 3 "" H 5700 5850 60  0001 C CNN
 	1    5700 5850
@@
 P 4750 1850
 F 0 "C8" H 4800 1950 50  0000 L CNN
-F 1 "47m/25V" H 4800 1750 50  0000 L CNN
-F 2 "Capacitors_SMD:c_elec_5x5.8" H 4750 1850 60  0001 C CNN
+F 1 "10m/16V" H 4800 1750 50  0000 L CNN
+F 2 "Capacitors_SMD:CP_Elec_5x5.8" H 4750 1850 60  0001 C CNN
 F 3 "" H 4750 1850 60  0001 C CNN
 	1    4750 1850
@@
 P 4850 3800
 F 0 "C9" H 4900 3900 50  0000 L CNN
-F 1 "47m/25V" H 4900 3700 50  0000 L CNN
-F 2 "Capacitors_SMD:c_elec_5x5.8" H 4850 3800 60  0001 C CNN
+F 1 "10m/16V" H 4900 3700 50  0000 L CNN
+F 2 "Capacitors_SMD:CP_Elec_5x5.8" H 4850 3800 60  0001 C CNN
 F 3 "" H 4850 3800 60  0001 C CNN
 	1    4850 3800
@@
 F 0 "R11" V 2180 4150 50  0000 C CNN
 F 1 "10k" V 2100 4150 50  0000 C CNN
-F 2 "Resistors_SMD:R_1206_HandSoldering" H 2100 4150 60  0001 C CNN
+F 2 "Resistors_SMD:R_0805_HandSoldering" H 2100 4150 60  0001 C CNN
 F 3 "" H 2100 4150 60  0001 C CNN
 	1    2100 4150
@@
 F 0 "R10" V 2230 2200 50  0000 C CNN
 F 1 "10k" V 2150 2200 50  0000 C CNN
-F 2 "Resistors_SMD:R_1206_HandSoldering" H 2150 2200 60  0001 C CNN
+F 2 "Resistors_SMD:R_0805_HandSoldering" H 2150 2200 60  0001 C CNN
 F 3 "" H 2150 2200 60  0001 C CNN
 	1    2150 2200
@@
 F 0 "R13" V 2880 4800 50  0000 C CNN
 F 1 "100k" V 2800 4800 50  0000 C CNN
-F 2 "Resistors_SMD:R_1206_HandSoldering" H 2800 4800 60  0001 C CNN
+F 2 "Resistors_SMD:R_0805_HandSoldering" H 2800 4800 60  0001 C CNN
 F 3 "" H 2800 4800 60  0001 C CNN
 	1    2800 4800
@@
 F 0 "R12" V 2930 2700 50  0000 C CNN
 F 1 "100k" V 2850 2700 50  0000 C CNN
-F 2 "Resistors_SMD:R_1206_HandSoldering" H 2850 2700 60  0001 C CNN
+F 2 "Resistors_SMD:R_0805_HandSoldering" H 2850 2700 60  0001 C CNN
 F 3 "" H 2850 2700 60  0001 C CNN
 	1    2850 2700
@@
 F 0 "R15" V 3430 4850 50  0000 C CNN
 F 1 "100k" V 3350 4850 50  0000 C CNN
-F 2 "Resistors_SMD:R_1206_HandSoldering" H 3350 4850 60  0001 C CNN
+F 2 "Resistors_SMD:R_0805_HandSoldering" H 3350 4850 60  0001 C CNN
 F 3 "" H 3350 4850 60  0001 C CNN
 	1    3350 4850
@@
 F 0 "R14" V 3480 2700 50  0000 C CNN
 F 1 "100k" V 3400 2700 50  0000 C CNN
-F 2 "Resistors_SMD:R_1206_HandSoldering" H 3400 2700 60  0001 C CNN
+F 2 "Resistors_SMD:R_0805_HandSoldering" H 3400 2700 60  0001 C CNN
 F 3 "" H 3400 2700 60  0001 C CNN
 	1    3400 2700
@@
 F 0 "R17" V 4330 4400 50  0000 C CNN
 F 1 "2M2" V 4250 4400 50  0000 C CNN
-F 2 "Resistors_SMD:R_1206_HandSoldering" H 4250 4400 60  0001 C CNN
+F 2 "Resistors_SMD:R_0805_HandSoldering" H 4250 4400 60  0001 C CNN
 F 3 "" H 4250 4400 60  0001 C CNN
 	1    4250 4400
@@
 F 0 "R16" V 4230 2350 50  0000 C CNN
 F 1 "2M2" V 4150 2350 50  0000 C CNN
-F 2 "Resistors_SMD:R_1206_HandSoldering" H 4150 2350 60  0001 C CNN
+F 2 "Resistors_SMD:R_0805_HandSoldering" H 4150 2350 60  0001 C CNN
 F 3 "" H 4150 2350 60  0001 C CNN
 	1    4150 2350
@@
 F 0 "C7" H 2550 3800 50  0000 L CNN
 F 1 "10m/16V" H 2550 3600 50  0000 L CNN
-F 2 "Capacitors_SMD:c_elec_5x5.8" H 2500 3700 60  0001 C CNN
+F 2 "Capacitors_SMD:CP_Elec_5x5.8" H 2500 3700 60  0001 C CNN
 F 3 "" H 2500 3700 60  0001 C CNN
 	1    2500 3700
@@
 F 0 "C6" H 2600 1850 50  0000 L CNN
 F 1 "10m/16V" H 2600 1650 50  0000 L CNN
-F 2 "Capacitors_SMD:c_elec_5x5.8" H 2550 1750 60  0001 C CNN
+F 2 "Capacitors_SMD:CP_Elec_5x5.8" H 2550 1750 60  0001 C CNN
 F 3 "" H 2550 1750 60  0001 C CNN
 	1    2550 1750
@@
 F 0 "U3" H 3800 4000 60  0000 L CNN
 F 1 "TL072" H 3800 3550 60  0000 L CNN
-F 2 "" H 3850 3800 60  0001 C CNN
+F 2 "Housings_SOIC:SOIC-8_3.9x4.9mm_Pitch1.27mm" H 3850 3800 60  0001 C CNN
 F 3 "" H 3850 3800 60  0001 C CNN
 	2    3850 3800
@@
 F 0 "U3" H 3850 2050 60  0000 L CNN
 F 1 "TL072" H 3850 1600 60  0000 L CNN
-F 2 "" H 3900 1850 60  0001 C CNN
+F 2 "Housings_SOIC:SOIC-8_3.9x4.9mm_Pitch1.27mm" H 3900 1850 60  0001 C CNN
 F 3 "" H 3900 1850 60  0001 C CNN
 	1    3900 1850
@@
 F 0 "P3" H 8400 3750 50  0000 C CNN
 F 1 "CONN_01X03" V 8500 3550 50  0000 C CNN
-F 2 "Pin_Headers:Pin_Header_Straight_1x05" H 8400 3550 60  0001 C CNN
+F 2 "Pin_Headers:Pin_Header_Straight_1x05_Pitch2.54mm" H 8400 3550 60  0001 C CNN
 F 3 "" H 8400 3550 60  0000 C CNN
 	1    8400 3550
@@
 F 0 "P2" H 8350 2450 50  0000 C CNN
 F 1 "CONN_01X03" V 8450 2250 50  0000 C CNN
-F 2 "Pin_Headers:Pin_Header_Straight_1x03" H 8350 2250 60  0001 C CNN
+F 2 "Pin_Headers:Pin_Header_Straight_1x03_Pitch2.54mm" H 8350 2250 60  0001 C CNN
 F 3 "" H 8350 2250 60  0000 C CNN
 	1    8350 2250
