File: kicad/motorola_cracker/motorola_cracker.sch (KiCad schematic (older format))
At the start: 13 parts, among them P1 UART, P2 +12V, P3 RTS, U2 68HC05_PLCC, X1 4Mhz

Commit message: to fcking much changes to commit it separatly, lets go with everything in one commit, git will love me for sure :D
Parts:
- C2, C3: symbol C -> motorola_cracker-rescue:C-RESCUE-motorola_cracker
- JP1: symbol JUMPER3 -> motorola_cracker-rescue:JUMPER3-RESCUE-motorola_cracker
- P1: symbol CONN_01X04 -> motorola_cracker-rescue:CONN_01X04-RESCUE-motorola_cracker
- P2: symbol CONN_01X02 -> motorola_cracker-rescue:CONN_01X02-RESCUE-motorola_cracker
- P3: symbol CONN_01X01 -> motorola_cracker-rescue:CONN_01X01-RESCUE-motorola_cracker
- R1, R2, R7, R8, R9: symbol R -> motorola_cracker-rescue:R-RESCUE-motorola_cracker
- U2: symbol 68HC05_PLCC -> motorola_cracker-rescue:68HC05_PLCC-RESCUE-motorola_cracker
- X1: symbol Crystal -> motorola_cracker-rescue:Crystal-RESCUE-motorola_cracker
Connections:
- wire segments 39 -> 45
Changed lines of the file:
@@
-EESchema Schematic File Version 2
-LIBS:motorola_cracker-rescue
-LIBS:power
-LIBS:device
-LIBS:transistors
-LIBS:conn
-LIBS:linear
-LIBS:regul
-LIBS:74xx
-LIBS:cmos4000
-LIBS:adc-dac
-LIBS:memory
-LIBS:xilinx
-LIBS:microcontrollers
-LIBS:dsp
-LIBS:microchip
-LIBS:analog_switches
-LIBS:motorola
-LIBS:texas
-LIBS:intel
-LIBS:audio
-LIBS:interface
-LIBS:digital-audio
-LIBS:philips
-LIBS:display
-LIBS:cypress
-LIBS:siliconi
-LIBS:opto
-LIBS:atmel
-LIBS:contrib
-LIBS:valves
+EESchema Schematic File Version 4
 LIBS:motorola_cracker-cache
-EELAYER 25 0
+EELAYER 26 0
 EELAYER END
 $Descr A4 11693 8268
@@
 $EndDescr
 $Comp
-L +5V #PWR01
+L motorola_cracker-rescue:+5V-RESCUE-motorola_cracker #PWR01
 U 1 1 53AAD03E
 P 3450 2300
@@
 $EndComp
 $Comp
-L GND #PWR02
+L motorola_cracker-rescue:GND-RESCUE-motorola_cracker #PWR02
 U 1 1 53AACF93
 P 8450 3350
@@
 $EndComp
 $Comp
-L GND #PWR03
+L motorola_cracker-rescue:GND-RESCUE-motorola_cracker #PWR03
 U 1 1 52DC243F
 P 7750 1750
@@
 $EndComp
 $Comp
-L GND #PWR04
+L motorola_cracker-rescue:GND-RESCUE-motorola_cracker #PWR04
 U 1 1 52DC243D
 P 7750 1100
@@
 $EndComp
 $Comp
-L C C3
+L motorola_cracker-rescue:C-RESCUE-motorola_cracker C3
 U 1 1 52DC2436
 P 7300 1650
@@
 $EndComp
 $Comp
-L C C2
+L motorola_cracker-rescue:C-RESCUE-motorola_cracker C2
 U 1 1 52DC2429
 P 7300 1050
@@
 $EndComp
 $Comp
-L Crystal X1
+L motorola_cracker-rescue:Crystal-RESCUE-motorola_cracker X1
 U 1 1 52DC241C
 P 6500 1350
@@
 $EndComp
 $Comp
-L CONN_01X02 P2
+L motorola_cracker-rescue:CONN_01X02-RESCUE-motorola_cracker P2
 U 1 1 52DBDB8E
 P 8250 3150
@@
 $EndComp
 $Comp
-L GND #PWR05
+L motorola_cracker-rescue:GND-RESCUE-motorola_cracker #PWR05
 U 1 1 52DBC8C7
 P 9200 1400
@@
 $EndComp
 $Comp
-L CONN_01X04 P1
+L motorola_cracker-rescue:CONN_01X04-RESCUE-motorola_cracker P1
 U 1 1 52DBC7F5
 P 8800 1200
@@
 $EndComp
 $Comp
-L R R8
+L motorola_cracker-rescue:R-RESCUE-motorola_cracker R8
 U 1 1 52DAF95D
 P 3850 2400
@@
 $EndComp
 $Comp
-L R R9
+L motorola_cracker-rescue:R-RESCUE-motorola_cracker R9
 U 1 1 52DAF927
 P 6800 3400
@@
 $EndComp
 $Comp
-L +5V #PWR06
+L motorola_cracker-rescue:+5V-RESCUE-motorola_cracker #PWR06
 U 1 1 52DAF91A
 P 7150 3150
@@
 $EndComp
 $Comp
-L GND #PWR07
+L motorola_cracker-rescue:GND-RESCUE-motorola_cracker #PWR07
 U 1 1 52DAF8D6
 P 5200 5250
@@
 $EndComp
 $Comp
-L +5V #PWR08
+L motorola_cracker-rescue:+5V-RESCUE-motorola_cracker #PWR08
 U 1 1 52DAF45F
 P 9200 950
@@
 $EndComp
 $Comp
-L GND #PWR09
+L motorola_cracker-rescue:GND-RESCUE-motorola_cracker #PWR09
 U 1 1 543000B3
 P 6850 3900
@@
 68HC705
 $Comp
-L R R1
+L motorola_cracker-rescue:R-RESCUE-motorola_cracker R1
 U 1 1 55BA483C
 P 6800 3300
@@
 $EndComp
 $Comp
-L +5V #PWR010
+L motorola_cracker-rescue:+5V-RESCUE-motorola_cracker #PWR010
 U 1 1 55BAE486
 P 5200 1000
@@
 $EndComp
 $Comp
-L R R7
+L motorola_cracker-rescue:R-RESCUE-motorola_cracker R7
 U 1 1 52DAF9A3
 P 6600 2000
@@
 TX
 $Comp
-L CONN_01X01 P3
+L motorola_cracker-rescue:CONN_01X01-RESCUE-motorola_cracker P3
 U 1 1 55BB8CCF
 P 8800 1700
@@
 RESET
 $Comp
-L JUMPER3 JP1
+L motorola_cracker-rescue:JUMPER3-RESCUE-motorola_cracker JP1
 U 1 1 55BBE03F
 P 6850 3700
@@
 +12V
 $Comp
-L R R2
+L motorola_cracker-rescue:R-RESCUE-motorola_cracker R2
 U 1 1 55BA6671
 P 6900 1350
@@
 	5200 1000 5200 1100
 Wire Wire Line
-	6200 3300 6650 3300
+	6200 3300 6450 3300
 Wire Wire Line
 	6950 3400 7150 3400
 Wire Wire Line
-	7150 3400 7150 3150
+	7150 3400 7150 3300
 Wire Wire Line
 	6950 3300 7150 3300
@@
 +12V
 $Comp
-L 68HC05_PLCC U2
+L motorola_cracker-rescue:68HC05_PLCC-RESCUE-motorola_cracker U2
 U 1 1 55BA8732
 P 5200 3100
@@
 $EndComp
 Wire Wire Line
-	6200 1650 7150 1650
-Wire Wire Line
-	6250 1050 7150 1050
+	6200 1650 6500 1650
+Wire Wire Line
+	6250 1050 6500 1050
 Wire Wire Line
 	6900 1500 6900 1650
@@
 	6900 1200 6900 1050
 Connection ~ 6900 1050
+Wire Wire Line
+	7150 3300 7150 3150
+Wire Wire Line
+	6450 3300 6650 3300
+Wire Wire Line
+	6900 1650 7150 1650
+Wire Wire Line
+	6500 1650 6900 1650
+Wire Wire Line
+	6500 1050 6900 1050
+Wire Wire Line
+	6900 1050 7150 1050
 $EndSCHEMATC
