File: kicad/sot23-6_breadboard_adapter/sot23-6_breadboard_adapter.kicad_pcb (KiCad board)
At the start: 2 copper layers, 11.4 x 8.9 mm, 3 parts, among them P1 CONN_01X03, P2 CONN_01X03, U1 MCP3421A0T-E/CH

Commit message: to fcking much changes to commit it separatly, lets go with everything in one commit, git will love me for sure :D
Parts:
- added U2: MCP3421A0T-E/CH, Housings_SOT-23_SOT-143_TSOT-6.pretty:SOT-23-6, B.Cu at (112.0, 87.4)
Routing:
- net Net-(P1-Pad3): track 6.38 -> 12.5 mm
- net Net-(P2-Pad3): track 6.44 -> 12.4 mm
- net Net-(P1-Pad1): track 5.87 -> 11.8 mm
- net Net-(P2-Pad1): track 5.80 -> 11.7 mm
- net Net-(P1-Pad2): track 5.63 -> 11.3 mm
- net Net-(P2-Pad2): track 6.02 -> 11.7 mm
Changed lines of the file:
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@@
-(kicad_pcb (version 4) (host pcbnew 0.201510170916+6271~30~ubuntu14.04.1-product)
+(kicad_pcb (version 20171130) (host pcbnew 5.0-dev-unknown-dd04bcb~61~ubuntu16.04.1)
   (general
-    (links 6)
-    (no_connects 0)
-    (area 106.096999 82.855999 117.753201 91.921401)
     (thickness 1.6)
     (drawings 4)
-    (tracks 29)
+    (tracks 59)
     (zones 0)
-    (modules 3)
+    (modules 4)
     (nets 7)
   )
@@
     (pad_to_mask_clearance 0.2)
     (aux_axis_origin 0 0)
-    (visible_elements FFFEFF7F)
+    (visible_elements FFFFFF7F)
     (pcbplotparams
       (layerselection 0x00030_80000001)
       (usegerberextensions false)
+      (usegerberattributes false)
+      (usegerberadvancedattributes false)
+      (creategerberjobfile false)
       (excludeedgelayer true)
       (linewidth 1.000000)
@@
       (hpglpenspeed 20)
       (hpglpendiameter 15)
-      (hpglpenoverlay 2)
       (psnegative false)
       (psa4output false)
@@
       (net 3 "Net-(P1-Pad3)"))
     (model Pin_Headers.3dshapes/Pin_Header_Straight_1x03.wrl
-      (at (xyz 0 -0.1 0))
+      (offset (xyz 0 -2.539999961853027 0))
       (scale (xyz 1 1 1))
       (rotate (xyz 0 0 90))
@@
       (net 6 "Net-(P2-Pad3)"))
     (model Pin_Headers.3dshapes/Pin_Header_Straight_1x03.wrl
-      (at (xyz 0 -0.1 0))
+      (offset (xyz 0 -2.539999961853027 0))
       (scale (xyz 1 1 1))
       (rotate (xyz 0 0 90))
@@
     )
   )
+  (module Housings_SOT-23_SOT-143_TSOT-6.pretty:SOT-23-6 (layer B.Cu)
+    (at 112.014 87.376 90)
+    (descr "6-pin SOT-23 package")
+    (tags SOT-23-6)
+    (attr smd)
+    (fp_text reference U2 (at 0 2.9 90) (layer B.SilkS)
+      (effects (font (size 1 1) (thickness 0.15)) (justify mirror))
+    )
+    (fp_text value MCP3421A0T-E/CH (at 0 -2.9 90) (layer B.Fab)
+      (effects (font (size 1 1) (thickness 0.15)) (justify mirror))
+    )
+    (fp_circle (center -0.4 1.7) (end -0.3 1.7) (layer B.SilkS) (width 0.15))
+    (fp_line (start 0.25 1.45) (end -0.25 1.45) (layer B.SilkS) (width 0.15))
+    (fp_line (start 0.25 -1.45) (end 0.25 1.45) (layer B.SilkS) (width 0.15))
+    (fp_line (start -0.25 -1.45) (end 0.25 -1.45) (layer B.SilkS) (width 0.15))
+    (fp_line (start -0.25 1.45) (end -0.25 -1.45) (layer B.SilkS) (width 0.15))
+    (pad 1 smd rect (at -1.1 0.95 90) (size 1.06 0.65) (layers B.Cu B.Paste B.Mask)
+      (net 3 "Net-(P1-Pad3)"))
+    (pad 2 smd rect (at -1.1 0 90) (size 1.06 0.65) (layers B.Cu B.Paste B.Mask)
+      (net 2 "Net-(P1-Pad2)"))
+    (pad 3 smd rect (at -1.1 -0.95 90) (size 1.06 0.65) (layers B.Cu B.Paste B.Mask)
+      (net 1 "Net-(P1-Pad1)"))
+    (pad 4 smd rect (at 1.1 -0.95 90) (size 1.06 0.65) (layers B.Cu B.Paste B.Mask)
+      (net 6 "Net-(P2-Pad3)"))
+    (pad 6 smd rect (at 1.1 0.95 90) (size 1.06 0.65) (layers B.Cu B.Paste B.Mask)
+      (net 4 "Net-(P2-Pad1)"))
+    (pad 5 smd rect (at 1.1 0 90) (size 1.06 0.65) (layers B.Cu B.Paste B.Mask)
+      (net 5 "Net-(P2-Pad2)"))
+    (model Housings_SOT-23_SOT-143_TSOT-6.3dshapes/SOT-23-6.wrl
+      (at (xyz 0 0 0))
+      (scale (xyz 1 1 1))
+      (rotate (xyz 0 0 0))
+    )
+  )
   (gr_line (start 106.2482 90.9828) (end 106.2482 83.3882) (angle 90) (layer Edge.Cuts) (width 0.15))
   (gr_line (start 116.967 91.821) (end 106.8578 91.821) (angle 90) (layer Edge.Cuts) (width 0.15))
   (gr_line (start 117.6274 83.7438) (end 117.6274 90.9066) (angle 90) (layer Edge.Cuts) (width 0.15))
   (gr_line (start 106.807 82.9564) (end 117.1448 82.9564) (angle 90) (layer Edge.Cuts) (width 0.15))
+  (segment (start 110.236 88.223) (end 110.236 85.6782) (width 0.25) (layer B.Cu) (net 1))
+  (segment (start 110.489 88.476) (end 110.236 88.223) (width 0.25) (layer B.Cu) (net 1))
+  (segment (start 110.236 85.6782) (end 109.3938 84.836) (width 0.25) (layer B.Cu) (net 1))
+  (segment (start 111.064 88.476) (end 110.489 88.476) (width 0.25) (layer B.Cu) (net 1))
+  (segment (start 109.3938 84.836) (end 108.1278 84.836) (width 0.25) (layer B.Cu) (net 1))
   (segment (start 108.1278 84.836) (end 109.2962 84.836) (width 0.25) (layer F.Cu) (net 1))
   (segment (start 110.4216 88.4506) (end 111.0386 88.4506) (width 0.25) (layer F.Cu) (net 1))
@@
   (segment (start 110.1598 85.6996) (end 110.1598 88.1888) (width 0.25) (layer F.Cu) (net 1))
   (segment (start 109.2962 84.836) (end 110.1598 85.6996) (width 0.25) (layer F.Cu) (net 1))
+  (segment (start 112.014 89.2556) (end 112.014 88.476) (width 0.25) (layer B.Cu) (net 2))
+  (segment (start 111.6838 89.5858) (end 112.014 89.2556) (width 0.25) (layer B.Cu) (net 2))
+  (segment (start 110.49 89.5858) (end 111.6838 89.5858) (width 0.25) (layer B.Cu) (net 2))
+  (segment (start 108.1278 87.376) (end 108.2802 87.376) (width 0.25) (layer B.Cu) (net 2))
+  (segment (start 108.2802 87.376) (end 110.49 89.5858) (width 0.25) (layer B.Cu) (net 2))
   (segment (start 108.1278 87.376) (end 108.331 87.376) (width 0.25) (layer F.Cu) (net 2))
   (segment (start 108.331 87.376) (end 110.4646 89.5096) (width 0.25) (layer F.Cu) (net 2))
@@
   (segment (start 111.6838 89.5096) (end 111.9886 89.2048) (width 0.25) (layer F.Cu) (net 2))
   (segment (start 111.9886 89.2048) (end 111.9886 88.4506) (width 0.25) (layer F.Cu) (net 2))
+  (segment (start 112.136 90.17) (end 109.6478 90.17) (width 0.25) (layer B.Cu) (net 3))
+  (segment (start 109.6478 90.17) (end 109.3938 89.916) (width 0.25) (layer B.Cu) (net 3))
+  (segment (start 109.3938 89.916) (end 108.1278 89.916) (width 0.25) (layer B.Cu) (net 3))
+  (segment (start 112.964 89.342) (end 112.136 90.17) (width 0.25) (layer B.Cu) (net 3))
+  (segment (start 112.964 88.476) (end 112.964 89.342) (width 0.25) (layer B.Cu) (net 3))
   (segment (start 108.1278 89.916) (end 109.5248 89.916) (width 0.25) (layer F.Cu) (net 3))
   (segment (start 112.9386 89.5502) (end 112.9386 88.4506) (width 0.25) (layer F.Cu) (net 3))
@@
   (segment (start 109.9058 90.297) (end 112.1918 90.297) (width 0.25) (layer F.Cu) (net 3))
   (segment (start 109.5248 89.916) (end 109.9058 90.297) (width 0.25) (layer F.Cu) (net 3))
+  (segment (start 114.046 86.783) (end 114.046 89.4802) (width 0.25) (layer B.Cu) (net 4))
+  (segment (start 113.539 86.276) (end 114.046 86.783) (width 0.25) (layer B.Cu) (net 4))
+  (segment (start 114.046 89.4802) (end 114.4818 89.916) (width 0.25) (layer B.Cu) (net 4))
+  (segment (start 112.964 86.276) (end 113.539 86.276) (width 0.25) (layer B.Cu) (net 4))
+  (segment (start 114.4818 89.916) (end 115.7478 89.916) (width 0.25) (layer B.Cu) (net 4))
   (segment (start 112.9386 86.2506) (end 113.327 86.2506) (width 0.25) (layer F.Cu) (net 4))
   (segment (start 114.4778 89.916) (end 115.7478 89.916) (width 0.25) (layer F.Cu) (net 4))
@@
   (segment (start 113.9698 86.8934) (end 113.9698 89.408) (width 0.25) (layer F.Cu) (net 4))
   (segment (start 113.327 86.2506) (end 113.9698 86.8934) (width 0.25) (layer F.Cu) (net 4))
+  (segment (start 112.42 85.09) (end 112.014 85.496) (width 0.25) (layer B.Cu) (net 5))
+  (segment (start 113.3094 85.09) (end 112.42 85.09) (width 0.25) (layer B.Cu) (net 5))
+  (segment (start 115.5954 87.376) (end 113.3094 85.09) (width 0.25) (layer B.Cu) (net 5))
+  (segment (start 115.7478 87.376) (end 115.5954 87.376) (width 0.25) (layer B.Cu) (net 5))
+  (segment (start 112.014 85.496) (end 112.014 86.276) (width 0.25) (layer B.Cu) (net 5))
   (segment (start 115.7478 87.376) (end 115.7478 87.0712) (width 0.25) (layer F.Cu) (net 5))
   (segment (start 115.7478 87.0712) (end 113.6142 84.9376) (width 0.25) (layer F.Cu) (net 5))
@@
   (segment (start 112.395 84.9376) (end 111.9886 85.344) (width 0.25) (layer F.Cu) (net 5))
   (segment (start 111.9886 85.344) (end 111.9886 86.2506) (width 0.25) (layer F.Cu) (net 5))
+  (segment (start 111.064 85.496) (end 112.014 84.546) (width 0.25) (layer B.Cu) (net 6))
+  (segment (start 115.7478 84.836) (end 114.4818 84.836) (width 0.25) (layer B.Cu) (net 6))
+  (segment (start 114.4818 84.836) (end 114.1918 84.546) (width 0.25) (layer B.Cu) (net 6))
+  (segment (start 114.1918 84.546) (end 112.014 84.546) (width 0.25) (layer B.Cu) (net 6))
+  (segment (start 111.064 86.276) (end 111.064 85.496) (width 0.25) (layer B.Cu) (net 6))
   (segment (start 111.0386 86.2506) (end 111.0386 85.3034) (width 0.25) (layer F.Cu) (net 6))
   (segment (start 115.0366 84.1248) (end 115.7478 84.836) (width 0.25) (layer F.Cu) (net 6))
