File: kicad/blk-md-spk-b_breadboard_adapter/blk-md-spk-b_breadboard_adapter.sch (KiCad schematic (older format))
At the start: 12 parts, among them J1 SCJ368R1NUS0B00G, P1 CONNECTOR, P2 CONNECTOR, U1 BLK-MD-SPK-B

Commit message: updated version
Parts:
- removed J1: SCJ368R1NUS0B00G, jacks:3.5mm_stereo_jack_PJ320B, symbol SCJ368R1NUS0B00G
- added BACK1, FWD1, VOL+1, VOL-1: SW_PUSH, Buttons_Switches_SMD:SW_SPST_FSMSM, symbol MiscellaneousDevices:SWITCH_SPST
- added C2: 4u7, Capacitors_SMD:C_1206_HandSoldering, symbol blk-md-spk-b_breadboard_adapter-rescue:C
- added C3: 1u, Capacitors_SMD:C_1206_HandSoldering, symbol blk-md-spk-b_breadboard_adapter-rescue:C
- added C4: 10, Capacitors_SMD:C_0805_HandSoldering, symbol blk-md-spk-b_breadboard_adapter-rescue:C
- added J1, J2: Jack_3.5mm_3pin, jacks:3.5mm_stereo_jack_PJ320B, symbol w_connectors:Jack_3.5mm_3pin
- added L1: 15n, Choke_SMD.pretty:Choke_SMD_1206_Handsoldering, symbol Device:L
- added R4: 2k7, Resistors_SMD:R_0805_HandSoldering, symbol blk-md-spk-b_breadboard_adapter-rescue:R
- C1: symbol C -> Device:C
- D1, D2: symbol LED -> Device:LED
- MFB1: renamed from ON/OFF1; symbol SW_PUSH -> MiscellaneousDevices:SWITCH_SPST
- P1, P2: symbol CONN_10 -> Connector_Generic:Conn_01x10
- R1, R2, R3: symbol R -> Device:R
- RESET1: symbol SW_PUSH -> MiscellaneousDevices:SWITCH_SPST
- U1: symbol BLK-MD-SPK-B -> BLK-MD-SPK-B:BLK-MD-SPK-B
Connections:
- net labels added: 1V8, BACK, BLED, CHG, FWD, MFB, MIC, MUTE, RLED, RST, RXD, SPKLP, SPKN, SPKRP, TXD, VBAT, VMIC, VOL+, VOL-
- wire segments 61 -> 89
