File: kicad/blk-md-spk-b_breadboard_adapter/blk-md-spk-b_breadboard_adapter.sch (KiCad schematic (older format))
At the start: 22 parts, among them J1 Jack_3.5mm_3pin, J2 Jack_3.5mm_3pin, P1 CONNECTOR, P2 CONNECTOR, U1 BLK-MD-SPK-B

Commit message: udpated to version 2.1
Parts:
- added C5, C6, C7: 1u, Capacitors_SMD:C_1206_HandSoldering, symbol blk-md-spk-b_breadboard_adapter-rescue:C
Connections:
- net SPKLP: now also C7.1, C7.2
- net SPKN: now also C5.1, C5.2
- net SPKRP: now also C6.1, C6.2
Other:
- note added: "C5,C6,C7 - optional , no need for headphones"
- moved on the sheet: BACK1, C1, C2, C3, C4, D1, D2, FWD1, J1, J2, L1, MFB1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

Commit message: update
Parts:
- C5, C6, C7: value 1u -> 10uF
Changed lines of the file:
@@
 EESchema Schematic File Version 4
 LIBS:blk-md-spk-b_breadboard_adapter-cache
-EELAYER 26 0
+EELAYER 29 0
 EELAYER END
 $Descr A4 11693 8268
@@
 P 2250 5700
 F 0 "C5" V 2200 5800 50  0000 C CNN
-F 1 "1u" V 2200 5550 50  0000 C CNN
+F 1 "10uF" V 2200 5550 50  0000 C CNN
 F 2 "Capacitors_SMD:C_1206_HandSoldering" H 2288 5550 50  0001 C CNN
 F 3 "" H 2250 5700 50  0000 C CNN
@@
 P 2250 5800
 F 0 "C6" V 2300 5900 50  0000 C CNN
-F 1 "1u" V 2300 5650 50  0000 C CNN
+F 1 "10uF" V 2300 5650 50  0000 C CNN
 F 2 "Capacitors_SMD:C_1206_HandSoldering" H 2288 5650 50  0001 C CNN
 F 3 "" H 2250 5800 50  0000 C CNN
@@
 P 2250 6000
 F 0 "C7" V 2300 6100 50  0000 C CNN
-F 1 "1u" V 2300 5850 50  0000 C CNN
+F 1 "10uF" V 2300 5850 50  0000 C CNN
 F 2 "Capacitors_SMD:C_1206_HandSoldering" H 2288 5850 50  0001 C CNN
 F 3 "" H 2250 6000 50  0000 C CNN
