File: kicad/BM23_breadboard_adapter/BM23_breadboard_adapter.kicad_pcb (KiCad board)
At the start: 2 copper layers, 29.5 x 49.8 mm, 21 parts, among them CON1 CONN_19, CON2 CONN_18, CON3 CONN_2, J1 USB_B_Micro, J2 3.5mmjack, U1 BM23

Commit message: update
Parts:
- added JP1: Jumper_NO_Small, Jumper:SolderJumper-2_P1.3mm_Open_RoundedPad1.0x1.5mm, B.Cu at (170.1, 79.0)
- J2: footprint jacks:3.5mm_stereo_jack_PJ320B_no_up_silkscreen -> jacks:3.5mm_stereo_jack_PJ320B
Routing:
- net Net-(J2-Pad3): track 0.00 -> 6.21 mm, vias 0 -> 1
- net Net-(C8-Pad1): track 42.4 -> 40.0 mm, vias 0 -> 1
Changed lines of the file:
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@@
-(kicad_pcb (version 20171130) (host pcbnew 5.0.0-rc2-dev-unknown-ce1bd4c~62~ubuntu16.04.1)
+(kicad_pcb (version 20171130) (host pcbnew 5.0.0-rc2-dev-unknown-648803d~64~ubuntu16.04.1)
   (general
     (thickness 1.6)
     (drawings 11)
-    (tracks 464)
+    (tracks 475)
     (zones 0)
-    (modules 21)
-    (nets 40)
+    (modules 22)
+    (nets 41)
   )
   (page A4)
@@
   (net 38 "Net-(C10-Pad2)")
   (net 39 "Net-(C8-Pad1)")
+  (net 40 "Net-(J2-Pad3)")
   (net_class Default "This is the default net class."
     (clearance 0.2)
@@
     (add_net "Net-(C5-Pad1)")
     (add_net "Net-(C8-Pad1)")
+    (add_net "Net-(J2-Pad3)")
+  )
+  (module jacks:3.5mm_stereo_jack_PJ320B (layer F.Cu)
+    (at 169.926 75.946)
+    (fp_text reference J2 (at -0.05 -3.3) (layer F.SilkS)
+      (effects (font (size 0.39878 0.39878) (thickness 0.0508)))
+    )
+    (fp_text value 3.5mmjack (at 0.11 2.15 90) (layer F.SilkS) hide
+      (effects (font (size 1.524 1.524) (thickness 0.3048)))
+    )
+    (fp_line (start 3 -2.1) (end 3 -1.05) (layer Dwgs.User) (width 0.15))
+    (fp_line (start 3 3) (end 3 9.1) (layer F.SilkS) (width 0.15))
+    (fp_line (start 3 9.1) (end -3 9.1) (layer F.SilkS) (width 0.15))
+    (fp_line (start -3 9.1) (end -3 8.25) (layer F.SilkS) (width 0.15))
+    (fp_line (start -3 1.25) (end -3 6.2) (layer F.SilkS) (width 0.15))
+    (fp_line (start -3 -1) (end -3 -2.1) (layer Dwgs.User) (width 0.15))
+    (fp_line (start -3 -2.1) (end -2.5 -2.1) (layer Dwgs.User) (width 0.15))
+    (fp_line (start -2.5 -2.1) (end -2.5 -4.8) (layer Dwgs.User) (width 0.15))
+    (fp_line (start -2.5 -4.8) (end 2.5 -4.8) (layer Dwgs.User) (width 0.15))
+    (fp_line (start 2.5 -4.8) (end 2.5 -2.1) (layer Dwgs.User) (width 0.15))
+    (fp_line (start 2.5 -2.1) (end 3 -2.1) (layer Dwgs.User) (width 0.15))
+    (fp_line (start 3 -1) (end 3 1) (layer F.SilkS) (width 0.15))
+    (pad "" np_thru_hole circle (at 0 6) (size 1.2 1.2) (drill 1.2) (layers *.Cu *.Mask F.SilkS))
+    (pad 2 smd rect (at -3.75 7.2) (size 3.5 1.5) (layers F.Cu F.Paste F.Mask)
+      (net 39 "Net-(C8-Pad1)"))
+    (pad 3 smd rect (at 3.75 2) (size 3.5 1.5) (layers F.Cu F.Paste F.Mask)
+      (net 40 "Net-(J2-Pad3)"))
+    (pad 1 smd rect (at -3.75 0.2) (size 3.5 1.5) (layers F.Cu F.Paste F.Mask)
+      (net 38 "Net-(C10-Pad2)"))
+    (pad "" np_thru_hole circle (at 0 0) (size 1.2 1.2) (drill 1.2) (layers *.Cu *.Mask F.SilkS))
   )
   (module modules:BM23_no_silk_screen_under_antena (layer B.Cu)
@@
       (net 15 /15))
   )
-  (module jacks:3.5mm_stereo_jack_PJ320B_no_up_silkscreen (layer F.Cu)
-    (at 169.926 75.946)
-    (fp_text reference J2 (at 1.79 3.79) (layer F.SilkS)
-      (effects (font (size 0.39878 0.39878) (thickness 0.0508)))
-    )
-    (fp_text value 3.5mmjack (at 0.14 3.88 90) (layer F.SilkS) hide
-      (effects (font (size 1.524 1.524) (thickness 0.3048)))
-    )
-    (fp_line (start 3 3) (end 3 9.1) (layer F.SilkS) (width 0.15))
-    (fp_line (start 3 9.1) (end -3 9.1) (layer F.SilkS) (width 0.15))
-    (fp_line (start -3 9.1) (end -3 8) (layer F.SilkS) (width 0.15))
-    (fp_line (start -3 1) (end -3 6) (layer F.SilkS) (width 0.15))
-    (pad "" np_thru_hole circle (at 0 6) (size 1.2 1.2) (drill 1.2) (layers *.Cu *.Mask F.SilkS))
-    (pad 5 smd rect (at -3.75 7) (size 3.5 1.5) (layers F.Cu F.Paste F.Mask)
+  (module Jumper:SolderJumper-2_P1.3mm_Open_RoundedPad1.0x1.5mm (layer B.Cu)
+    (at 170.053 78.994 180)
+    (descr "SMD Solder Jumper, 1x1.5mm, rounded Pads, 0.3mm gap, open")
+    (tags "solder jumper open")
+    (attr virtual)
+    (fp_text reference JP1 (at 0.127 1.651 180) (layer B.SilkS)
+      (effects (font (size 1 1) (thickness 0.15)) (justify mirror))
+    )
+    (fp_text value Jumper_NO_Small (at 0 -1.9 180) (layer B.Fab)
+      (effects (font (size 1 1) (thickness 0.15)) (justify mirror))
+    )
+    (fp_arc (start 0.7 0.3) (end 1.4 0.3) (angle 90) (layer B.SilkS) (width 0.12))
+    (fp_arc (start 0.7 -0.3) (end 0.7 -1) (angle 90) (layer B.SilkS) (width 0.12))
+    (fp_arc (start -0.7 -0.3) (end -1.4 -0.3) (angle 90) (layer B.SilkS) (width 0.12))
+    (fp_arc (start -0.7 0.3) (end -0.7 1) (angle 90) (layer B.SilkS) (width 0.12))
+    (fp_line (start -1.4 -0.3) (end -1.4 0.3) (layer B.SilkS) (width 0.12))
+    (fp_line (start 0.7 -1) (end -0.7 -1) (layer B.SilkS) (width 0.12))
+    (fp_line (start 1.4 0.3) (end 1.4 -0.3) (layer B.SilkS) (width 0.12))
+    (fp_line (start -0.7 1) (end 0.7 1) (layer B.SilkS) (width 0.12))
+    (fp_line (start -1.65 1.25) (end 1.65 1.25) (layer B.CrtYd) (width 0.05))
+    (fp_line (start -1.65 1.25) (end -1.65 -1.25) (layer B.CrtYd) (width 0.05))
+    (fp_line (start 1.65 -1.25) (end 1.65 1.25) (layer B.CrtYd) (width 0.05))
+    (fp_line (start 1.65 -1.25) (end -1.65 -1.25) (layer B.CrtYd) (width 0.05))
+    (pad 2 smd roundrect (at 0.65 0 180) (size 1 1.5) (layers B.Cu B.Mask)(roundrect_rratio 0.5)
       (net 39 "Net-(C8-Pad1)"))
-    (pad 2 smd rect (at 3.75 2) (size 3.5 1.5) (layers F.Cu F.Paste F.Mask)
+    (pad 1 smd roundrect (at -0.65 0 180) (size 1 1.5) (layers B.Cu B.Mask)(roundrect_rratio 0.5)
+      (net 40 "Net-(J2-Pad3)"))
+    (pad 1 smd rect (at -0.4 0 180) (size 0.5 1.5) (layers B.Cu B.Mask)
+      (net 40 "Net-(J2-Pad3)"))
+    (pad 2 smd rect (at 0.4 0 180) (size 0.5 1.5) (layers B.Cu B.Mask)
       (net 39 "Net-(C8-Pad1)"))
-    (pad 1 smd rect (at -3.75 0) (size 3.5 1.5) (layers F.Cu F.Paste F.Mask)
-      (net 38 "Net-(C10-Pad2)"))
-    (pad "" np_thru_hole circle (at 0 0) (size 1.2 1.2) (drill 1.2) (layers *.Cu *.Mask F.SilkS))
   )
   (gr_text "SYSPWR\nBATIN" (at 176.5808 81.5086 180) (layer F.SilkS)
@@
   (segment (start 164.039589 94.021589) (end 164.039589 91.563589) (width 0.2) (layer F.Cu) (net 39))
   (segment (start 166.176 82.946) (end 167.176 82.946) (width 0.2) (layer F.Cu) (net 39))
-  (segment (start 167.176 82.946) (end 172.176 77.946) (width 0.2) (layer F.Cu) (net 39))
-  (segment (start 172.176 77.946) (end 173.676 77.946) (width 0.2) (layer F.Cu) (net 39))
   (segment (start 161.29 88.614) (end 162.29 88.614) (width 0.2) (layer F.Cu) (net 39))
   (segment (start 162.29 88.614) (end 166.176 84.728) (width 0.2) (layer F.Cu) (net 39))
   (segment (start 166.176 84.728) (end 166.176 83.896) (width 0.2) (layer F.Cu) (net 39))
   (segment (start 166.176 83.896) (end 166.176 82.946) (width 0.2) (layer F.Cu) (net 39))
+  (segment (start 167.473 80.899) (end 168.402 80.899) (width 0.2) (layer F.Cu) (net 39))
+  (via (at 168.402 80.899) (size 0.8) (drill 0.4) (layers F.Cu B.Cu) (net 39))
+  (segment (start 166.176 82.196) (end 167.473 80.899) (width 0.2) (layer F.Cu) (net 39))
+  (segment (start 166.176 83.146) (end 166.176 82.196) (width 0.2) (layer F.Cu) (net 39))
+  (segment (start 169.403 79.244) (end 169.653 78.994) (width 0.2) (layer B.Cu) (net 39))
+  (segment (start 169.403 79.898) (end 169.403 79.244) (width 0.2) (layer B.Cu) (net 39))
+  (segment (start 168.402 80.899) (end 169.403 79.898) (width 0.2) (layer B.Cu) (net 39))
+  (segment (start 172.176 77.946) (end 173.676 77.946) (width 0.2) (layer F.Cu) (net 40))
+  (via (at 172.593 79.756) (size 0.8) (drill 0.4) (layers F.Cu B.Cu) (net 40))
+  (segment (start 171.831 78.994) (end 172.593 79.756) (width 0.2) (layer B.Cu) (net 40))
+  (segment (start 170.453 78.994) (end 171.831 78.994) (width 0.2) (layer B.Cu) (net 40))
+  (segment (start 173.676 78.673) (end 173.676 77.946) (width 0.2) (layer F.Cu) (net 40))
+  (segment (start 172.593 79.756) (end 173.676 78.673) (width 0.2) (layer F.Cu) (net 40))
   (zone (net 15) (net_name /15) (layer B.Cu) (hatch edge 0.508)
     (connect_pads (clearance 0.508))
