File: kicad/F-6188_breakout_board/F-6188_breakout_board.kicad_pcb (KiCad board)
At the start: 2 copper layers, 29.5 x 42.2 mm, 34 parts, among them CON1 CONN_16, CON2 CONN_16, SW1 VOLUME UP, SW2 VOLUME DOWN, SW3 NEXT TRACK, SW4 PREVIOUS TRACK, SW5 PLAY/PAUSE, SW6 RESET, U1 F-6188, U2 PJ-320B, U3 PJ-320B, U4 PJ-327A

Commit message: v2
Parts:
- added JP3: Jumper_NO_Small, Jumper:SolderJumper-2_P1.3mm_Open_RoundedPad1.0x1.5mm, B.Cu at (233.9, 120.9)
- C4, C5: value CTS 1u/16V A 10% AVX-TAJ -> 1u/16V X7R; footprint Capacitors_Tantalum_SMD.pretty:TantalC_SizeA_EIA-3216_HandSoldering -> Capacitors_SMD.pretty:C_1206_HandSoldering
- turned C4 to 270 degrees
- turned C5 to 270 degrees
Connections:
- C4 pad 1: Net-(C4-Pad1) -> /MICP
- C4 pad 2: /MICP -> Net-(C4-Pad2)
- C5 pad 1: Net-(C5-Pad1) -> /MICN
- C5 pad 2: /MICN -> Net-(C5-Pad2)
- R4 pad 1: Net-(C4-Pad1) -> Net-(C4-Pad2)
- R5 pad 2: Net-(C5-Pad1) -> Net-(C5-Pad2)
- U2 pad 1: Net-(C5-Pad1) -> Net-(C5-Pad2)
- U2 pad 2: Net-(C4-Pad1) -> Net-(C4-Pad2)
- U2 pad 3: Net-(C4-Pad1) -> Net-(JP3-Pad2)
Routing:
- net Net-(C4-Pad1): track 26.8 -> 0.00 mm, vias 2 -> 0
- net Net-(C5-Pad2): track 0.00 -> 17.0 mm, vias 0 -> 2
- net Net-(C5-Pad1): track 17.0 -> 0.00 mm, vias 2 -> 0
- net Net-(C4-Pad2): track 0.00 -> 16.2 mm, vias 0 -> 1
- net Net-(JP3-Pad2): track 0.00 -> 5.10 mm, vias 0 -> 1
- net GND: track 149.3 -> 145.0 mm, vias 20 -> 19

Commit message: update
Parts:
- removed JP2: Jumper_2, Jumper:SolderJumper-2_P1.3mm_Open_RoundedPad1.0x1.5mm
- removed R2: 1k, Resistors_SMD.pretty:R_0805_HandSoldering
- added C10: 2.2p, Capacitors_SMD.pretty:C_0603_HandSoldering, B.Cu at (250.8, 89.0)
- added L1: 100nH*, Resistors_SMD.pretty:R_0805_HandSoldering, B.Cu at (251.5, 92.2)
- C2: value CTS 1u/16V A 10% AVX-TAJ -> 1u/16V; footprint Capacitors_Tantalum_SMD.pretty:TantalC_SizeA_EIA-3216_HandSoldering -> Capacitors_SMD.pretty:C_1206_HandSoldering
- C3: value 100n/50V X7R!!! -> 10n/50V X7R!!!
- C6, C7: value CKS1206 10u/25V X5R 10% SAMSUNG -> 1u/25V
- R4, R5: value 1k2 -> 1k
- moved R1 2.06 mm to (231.6, 91.9)
- moved D2 1.19 mm to (250.0, 105.2), turned to 270 degrees
- moved C4 0.40 mm to (243.8, 112.8)
Connections:
- CON2 pad 2: /ANT_EXT -> Net-(C10-Pad2)
- CON2 pad 3: GND -> Net-(CON2-Pad3)
- D1 pad 1: GND -> Net-(D1-Pad1)
- D1 pad 2: Net-(D1-Pad2) -> /LED0
- D2 pad 1: GND -> Net-(D1-Pad1)
- D2 pad 2: Net-(D2-Pad2) -> /LED1
- R1 pad 1: /VBAT -> /3V_OUT
- R3 pad 1: /LED1 -> Net-(D1-Pad1)
- R3 pad 2: Net-(D2-Pad2) -> GND
- R9 pad 1: (no net) -> /AUX_INR
- U1 pad 3: GND -> Net-(L1-Pad1)
Routing:
- net Net-(D1-Pad1): track 0.00 -> 20.5 mm
- net GND: track 145.0 -> 127.1 mm, vias 19 -> 20
- net Net-(D2-Pad2): track 7.28 -> 0.00 mm
- net /LED0: track 32.6 -> 37.8 mm, vias 3 -> 1
- net /ANT_EXT: track 6.84 -> 1.73 mm
- net /3V_OUT: track 39.7 -> 44.5 mm
- net Net-(D1-Pad2): track 4.38 -> 0.00 mm
- net Net-(L1-Pad1): track 0.00 -> 3.61 mm
- net Net-(C10-Pad2): track 0.00 -> 3.55 mm
- net /AUDIO_LP: track 40.5 -> 37.1 mm
- net Net-(CON2-Pad3): track 0.00 -> 2.71 mm
- net /MICP: track 43.8 -> 41.9 mm
- net Net-(R1-Pad2): track 36.9 -> 38.8 mm
- net /LED1: track 26.9 -> 25.5 mm
- net /AUX_INR: track 39.4 -> 40.7 mm
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