File: kicad/F-6188_breakout_board/F-6188_breakout_board.sch (KiCad schematic (older format))
At the start: 34 parts, among them CON1 CONN_16, CON2 CONN_16, SW1 VOLUME UP, SW2 VOLUME DOWN, SW3 NEXT TRACK, SW4 PREVIOUS TRACK, SW5 PLAY/PAUSE, SW6 RESET, U1 F-6188, U2 PJ-320B, U3 PJ-320B, U4 PJ-327A

Commit message: v2
Parts:
- removed C4, C5: CTS 1u/16V A 10% AVX-TAJ, Capacitors_Tantalum_SMD.pretty:TantalC_SizeA_EIA-3216_HandSoldering, symbol Device:CP
- added C4, C5: 1u/16V X7R, Capacitors_SMD.pretty:C_1206_HandSoldering, symbol c:C
- added JP3: Jumper_NO_Small, Jumper:SolderJumper-2_P1.3mm_Open_RoundedPad1.0x1.5mm, symbol Device:Jumper_NO_Small
- C6, C7, C8, C9: Manufacturer Part Number (none) -> CL31A106KAHNNNE; gme.sk part number (none) -> 905-207
- U2, U3: symbol PJ-320B:PJ-320B -> jacks:PJ-320B
- U4: symbol PJ_J327A:PJ-327A -> jacks:PJ-327A
Connections:
- net MICN: now also C5.1
- net MICP: now also C4.1
- net at R4.1, U2.2: now also C4.2, JP3.1; no longer U2.3
- net at R5.2, U2.1: now also C5.2
- new net: JP3.2, U2.3
Other:
- moved on the sheet: C6, C7, C8, C9, CON1, CON2, D1, D2, JP1, JP2, R1, R2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

Commit message: update
Parts:
- removed JP2: Jumper_2, Jumper:SolderJumper-2_P1.3mm_Open_RoundedPad1.0x1.5mm, symbol Device:Jumper_NO_Small
- removed R2: 1k, Resistors_SMD.pretty:R_0805_HandSoldering, symbol Device:R
- added C10: 2.2p, Capacitors_SMD.pretty:C_0603_HandSoldering, symbol c:C
- added L1: 100nH*, Resistors_SMD.pretty:R_0805_HandSoldering, symbol Device:L
- C1: symbol c:C -> Device:C
- C2: value CTS 1u/16V A 10% AVX-TAJ -> 1u/16V; footprint Capacitors_Tantalum_SMD.pretty:TantalC_SizeA_EIA-3216_HandSoldering -> Capacitors_SMD.pretty:C_1206_HandSoldering; symbol Device:CP -> Device:C
- C3: value 100n/50V X7R!!! -> 10n/50V X7R!!!
- C6, C7: value CKS1206 10u/25V X5R 10% SAMSUNG -> 1u/25V
- R4, R5: value 1k2 -> 1k
Connections:
- net AUX_INP is gone; now on net AUX_INR: R9.1
- net 3V_OUT: now also R1.1
- net ANT_EXT: now also C10.1; no longer CON2.2
- net GND: now also R3.2; no longer CON2.3, D1.1 (K), D2.1 (K), U1.3 (GND)
- net LED0: now also D1.2 (A)
- net LED1: now also D2.2 (A); no longer R3.1
- net VBAT: no longer R1.1
- new net: L1.1, U1.3 (GND)
- new net: C10.2, CON2.2
- new net: CON2.3, L1.2
- new net: D1.1 (K), D2.1 (K), R3.1
Other:
- note added: "* BK3254 compatibility"
- moved on the sheet: CON1, CON2, D1, D2, R3

Commit message: update
Parts:
- C6, C7: value 1u/25V -> 10u/25V
- C8, C9: value CKS1206 10u/25V X5R 10% SAMSUNG -> 4u7/25V X5R
Changed lines of the file:
@@
 EESchema Schematic File Version 4
 LIBS:F-6188_breakout_board-cache
-EELAYER 26 0
+EELAYER 29 0
 EELAYER END
 $Descr A4 11693 8268
@@
 P 6350 4100
 F 0 "C7" V 6250 4250 60  0000 C CNN
-F 1 "1u/25V" V 6450 4350 60  0000 C CNN
+F 1 "10u/25V" V 6450 4350 60  0000 C CNN
 F 2 "Capacitors_SMD.pretty:C_1206_HandSoldering" H 6350 4100 50  0001 C CNN
 F 3 "" H 6350 4100 50  0001 C CNN
@@
 P 6350 3800
 F 0 "C6" V 6150 3950 60  0000 C CNN
-F 1 "1u/25V" V 6250 4050 60  0000 C CNN
+F 1 "10u/25V" V 6250 4050 60  0000 C CNN
 F 2 "Capacitors_SMD.pretty:C_1206_HandSoldering" H 6350 3800 50  0001 C CNN
 F 3 "" H 6350 3800 50  0001 C CNN
@@
 P 6200 5900
 F 0 "C9" V 6100 6050 60  0000 C CNN
-F 1 "CKS1206 10u/25V X5R 10% SAMSUNG" V 6450 5900 60  0000 C CNN
+F 1 "4u7/25V X5R" V 6450 5900 60  0000 C CNN
 F 2 "Capacitors_SMD.pretty:C_1206_HandSoldering" H 6200 5900 50  0001 C CNN
 F 3 "" H 6200 5900 50  0001 C CNN
@@
 P 6200 5700
 F 0 "C8" V 6100 5850 60  0000 C CNN
-F 1 "CKS1206 10u/25V X5R 10% SAMSUNG" V 5900 5700 60  0000 C CNN
+F 1 "4u7/25V X5R" V 5900 5700 60  0000 C CNN
 F 2 "Capacitors_SMD.pretty:C_1206_HandSoldering" H 6200 5700 50  0001 C CNN
 F 3 "" H 6200 5700 50  0001 C CNN
