File: kicad/F-6888_breakaout_adapter/F-6888_breakaout_adapter.kicad_pcb (KiCad board)
At the start: 2 copper layers, 26.9 x 72.9 mm, 29 parts, among them J1 USB_A, J2 CONN_01X20, J3 MIC, J4 CONN_01X20, J6 Micro_SD_Card_Det, SW1 RESET, SW2 PREV/VOL-, SW3 NEXT/VOL+, SW4 P.P/CALL, SW5 MODE, U1 F-6888

Commit message: update
Parts:
- removed J3: MIC, Pin_Headers:Pin_Header_Straight_1x02_Pitch2.54mm
- removed PJ-327A2: CONN_6, jacks:3.5mm_stereo_jack_PJ3026
- added C10: 1uF, Capacitors_SMD:C_1206_HandSoldering, F.Cu at (112.1, 140.6)
- added C6: 1uF*, Capacitors_SMD:C_1206_HandSoldering, B.Cu at (116.3, 145.3)
- added C7: 10n(*), Capacitors_SMD:C_1206_HandSoldering, B.Cu at (111.8, 143.8)
- added C8: 2.2p, Capacitors_SMD:C_0603_HandSoldering, F.Cu at (124.8, 87.5)
- added C9: 1uF, Capacitors_SMD:C_1206_HandSoldering, F.Cu at (112.1, 137.8)
- added L1: 100nH*, Resistors_SMD.pretty:R_0805_HandSoldering, F.Cu at (124.1, 93.3)
- added R10: 200, Resistors_SMD:R_0805_HandSoldering, B.Cu at (104.4, 147.9)
- added R11: 200, Resistors_SMD:R_0805_HandSoldering, B.Cu at (107.2, 140.4)
- added R8: 1k*, Resistors_SMD:R_0805_HandSoldering, B.Cu at (124.0, 148.6)
- added R9: 10k, Resistors_SMD:R_0805_HandSoldering, B.Cu at (115.0, 111.9)
- added U3: PJ-320B, jacks:3.5mm_stereo_jack_PJ320B, F.Cu at (127.3, 141.7)
- added U4: PJ-320B, jacks:3.5mm_stereo_jack_PJ320B, F.Cu at (127.8, 150.9)
- C4, C5: value CP -> 1uF; footprint Capacitors_SMD:CP_Elec_4x5.3 -> Capacitors_SMD:C_1206_HandSoldering
- R3: value 1k2 -> 1k
- U1: footprint bluetooth:F-6888 -> modules:F-6888
- U2: renamed from PJ-327A1; value CONN_6 -> PJ-327A
- moved C2 6.19 mm to (116.3, 142.7)
- moved R4 4.82 mm to (109.4, 141.2)
- moved C1 3.37 mm to (123.8, 138.7), turned to 90 degrees
- moved C3 3.08 mm to (124.0, 146.3), turned to 0 degrees
- moved R3 2.99 mm to (124.1, 144.1), turned to 0 degrees
- moved D2 1.27 mm to (120.9, 133.9)
- moved D1 1.02 mm to (111.5, 134.1)
- moved D3 0.76 mm to (114.0, 150.9)
- moved U2 0.51 mm to (113.5, 156.7)
- turned SW3 to 90 degrees
Connections:
- C1 pad 1: GND -> /MICBIAS
- C1 pad 2: /MICBIAS -> GND
- C3 pad 1: GND -> Net-(C2-Pad1)
- C3 pad 2: Net-(C2-Pad1) -> GND
- J1 pad 2: /USBD- -> Net-(J1-Pad2)
- J1 pad 3: /USBD+ -> Net-(J1-Pad3)
- J2 pad 2: /FMINP -> Net-(C8-Pad1)
- J2 pad 3: /FMINN -> Net-(J2-Pad3)
- R1 pad 2: /VBAT -> /V3OUT
- R4 pad 2: Net-(PJ-327A1-Pad6) -> Net-(R4-Pad2)
- SW2 pad 1: GND -> Net-(R9-Pad1)
- SW3 pad 1: GND -> Net-(R9-Pad1)
- SW4 pad 1: GND -> Net-(R9-Pad1)
- SW5 pad 1: GND -> Net-(R9-Pad1)
- U2 pad 3: (no net) -> GND
- U2 pad 4: (no net) -> Net-(R4-Pad2)
- U2 pad 6: Net-(PJ-327A1-Pad6) -> (no net)
Routing:
- net GND: track 259.5 -> 182.3 mm, vias 29 -> 21
- net /NC: track 30.3 -> 71.2 mm, vias 1 -> 2
- net Net-(R9-Pad1): track 0.00 -> 35.5 mm, vias 0 -> 4
- net /AUDIORP: track 76.4 -> 54.8 mm
- net Net-(R4-Pad2): track 0.00 -> 18.3 mm, vias 0 -> 1
- net Net-(C10-Pad1): track 0.00 -> 14.8 mm
- net /V3OUT: track 23.8 -> 38.5 mm, vias 1 -> 4
- net Net-(C6-Pad2): track 0.00 -> 13.3 mm, vias 0 -> 1
- net /AUDIOLP: track 67.9 -> 55.0 mm
- net Net-(JP1-Pad2): track 66.7 -> 54.1 mm
- net /USBD-: track 50.3 -> 40.9 mm
- net /NEXT/VOL+: track 48.3 -> 39.5 mm
- net Net-(J1-Pad2): track 0.00 -> 7.02 mm
- net /MICBIAS: track 69.5 -> 75.7 mm
- net Net-(C9-Pad1): track 0.00 -> 6.03 mm
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Other:
- board text added: "SterMIC"
- board text added: "sdcard"
- board text added: "select ground"
- board text removed: "MIC"
- board text removed: "select audio ground for jack"
