File: kicad/F-6888_breakaout_adapter/F-6888_breakaout_adapter.sch (KiCad schematic (older format))
At the start: 29 parts, among them J1 USB_A, J2 CONN_01X20, J3 MIC, J4 CONN_01X20, J6 Micro_SD_Card_Det, SW1 RESET, SW2 PREV/VOL-, SW3 NEXT/VOL+, SW4 P.P/CALL, SW5 MODE, U1 F-6888

Commit message: update
Parts:
- removed J3: MIC, Pin_Headers:Pin_Header_Straight_1x02_Pitch2.54mm, symbol F-6888_breakaout_adapter-rescue:CONN_01X02-RESCUE-F-6888_breakaout_adapter
- removed PJ-327A1: CONN_6, jacks:PJ-327A_no_top_silkscreen, symbol gencon:CONN_6
- removed PJ-327A2: CONN_6, jacks:3.5mm_stereo_jack_PJ320B_no_up_silkscreen, symbol gencon:CONN_6
- added C10, C9: 10uF, Capacitors_SMD:C_1206_HandSoldering, symbol Device:C
- added C6: 1uF*, Capacitors_SMD:C_1206_HandSoldering, symbol F-6888_breakaout_adapter-rescue:C-RESCUE-F-6888_breakaout_adapter
- added C7: 10n(*), Capacitors_SMD:C_0805_HandSoldering, symbol F-6888_breakaout_adapter-rescue:C-RESCUE-F-6888_breakaout_adapter
- added C8: 2.2p, Capacitors_SMD:C_0603_HandSoldering, symbol F-6888_breakaout_adapter-rescue:C-RESCUE-F-6888_breakaout_adapter
- added L1: 100nH*, Resistors_SMD.pretty:R_0805_HandSoldering, symbol Device:L
- added R10, R11: 200, Resistors_SMD:R_0805_HandSoldering, symbol F-6888_breakaout_adapter-rescue:R-RESCUE-F-6888_breakaout_adapter
- added R8: 1k*, Resistors_SMD:R_0805_HandSoldering, symbol F-6888_breakaout_adapter-rescue:R-RESCUE-F-6888_breakaout_adapter
- added R9: 10k, Resistors_SMD:R_0805_HandSoldering, symbol F-6888_breakaout_adapter-rescue:R-RESCUE-F-6888_breakaout_adapter
- added U2: PJ-327A, jacks:PJ-327A, symbol jacks:PJ-327A
- added U3, U4: PJ-320B, jacks:3.5mm_stereo_jack_PJ320B, symbol jacks:PJ-320B
- C4, C5: value CP -> 10uF; footprint Capacitors_SMD:CP_Elec_4x5.3 -> Capacitors_SMD:C_1206_HandSoldering; symbol F-6888_breakaout_adapter-rescue:CP-RESCUE-F-6888_breakaout_adapter -> Device:C
- J1: footprint Connect:USB_A -> modules:USB_A
- R3: value 1k2 -> 1k
Connections:
- net AUDIOLP: now also C9.2
- net AUDIORP: now also C10.2
- net FMINN: now also L1.2; no longer J2.3 (P3)
- net FMINP: now also C8.2; no longer J2.2 (P2)
- net GND: now also C1.2, C3.2, R8.1, U2.3; no longer C1.1, C3.1, SW2.1 (A), SW3.1 (A), SW4.1 (A), SW5.1 (A)
- net MICBIAS: now also C1.1; no longer C1.2
- net MICIP: now also C7.1
- net NC: now also C6.1, C7.2
- net USBD+: now also R10.1; no longer J1.3 (D+)
- net USBD-: now also R11.2; no longer J1.2 (D-)
- net V3OUT: now also R1.2, R9.2
- net VBAT: no longer R1.2
- net at C2.1, R3.1: now also C3.1, U4.2; no longer C3.2
- net at R4.2: now also U2.4
- net at R5.2: now also U2.2
- net at R6.2: now also U2.5
- net at JP1.2: now also U3.1
- new net: C8.1, J2.2 (P2)
- new net: J2.3 (P3), L1.1
- new net: R9.1, SW2.1 (A), SW3.1 (A), SW4.1 (A), SW5.1 (A)
- new net: J1.2 (D-), R11.1
- new net: J1.3 (D+), R10.2
- new net: C9.1, U3.2
- new net: C10.1, U3.3
- new net: C6.2, R8.2, U4.1
Other:
- note added: "* BK8000L compatibility"
- note added: "* for F-6188 compatibility"
- moved on the sheet: C1, C2, C3, D1, D2, D3, J1, J2, J4, J6, JP1, R1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

Commit message: misc
Parts:
- J1: symbol Connector_Specialized:USB_A -> F-6888_breakaout_adapter-rescue:USB_A-Connector_Specialized
- U1: symbol F-6888:F-6888 -> F-6888_breakaout_adapter-rescue:F-6888-F-6888
Changed lines of the file:
@@
 encoding utf-8
 Sheet 1 1
-Title ""
-Date ""
-Rev ""
-Comp ""
-Comment1 ""
-Comment2 ""
-Comment3 ""
+Title "BK3254 adapter"
+Date "1.1.2019"
+Rev "3"
+Comp "kovo"
+Comment1 "firmware version 1.1up"
+Comment2 "buttons on separate IO"
+Comment3 "BK8000L compatible"
 Comment4 ""
 $EndDescr
 $Comp
-L F-6888:F-6888 U1
+L F-6888_breakaout_adapter-rescue:F-6888-F-6888 U1
 U 1 1 59BA8F51
 P 6350 1100
@@
 	1    0    0    1
 $EndComp
-Text Label 4950 950  0    60   ~ 0
+Text Label 4950 950  0    60   ~ 6
 GND
-Text Label 5350 1050 0    60   ~ 0
+Text Label 5350 1050 0    60   ~ 6
 FMINP
-Text Label 5350 1150 0    60   ~ 0
+Text Label 5350 1150 0    60   ~ 6
 FMINN
-Text Label 4850 1250 0    60   ~ 0
+Text Label 4850 1250 0    60   ~ 6
 TMS
-Text Label 4850 1350 0    60   ~ 0
+Text Label 4850 1350 0    60   ~ 6
 TCK
-Text Label 4850 1450 0    60   ~ 0
+Text Label 4850 1450 0    60   ~ 6
 TDO
-Text Label 4850 1550 0    60   ~ 0
+Text Label 4850 1550 0    60   ~ 6
 TDI
-Text Label 4950 1650 0    60   ~ 0
+Text Label 4950 1650 0    60   ~ 6
 RSTN
-Text Label 4950 1750 0    60   ~ 0
+Text Label 4950 1750 0    60   ~ 6
 GPIO6
-Text Label 4950 1850 0    60   ~ 0
+Text Label 4950 1850 0    60   ~ 6
 TX
-Text Label 4950 1950 0    60   ~ 0
+Text Label 4950 1950 0    60   ~ 6
 RX
-Text Label 4950 2050 0    60   ~ 0
+Text Label 4950 2050 0    60   ~ 6
 MUTE
-Text Label 4950 2150 0    60   ~ 0
+Text Label 4950 2150 0    60   ~ 6
 LED1
-Text Label 4950 2250 0    60   ~ 0
+Text Label 4950 2250 0    60   ~ 6
 LED2
-Text Label 4950 2450 0    60   ~ 0
+Text Label 4950 2450 0    60   ~ 6
 GND
-Text Label 4950 2550 0    60   ~ 0
+Text Label 4950 2550 0    60   ~ 6
 GPIO10
-Text Label 4950 2650 0    60   ~ 0
+Text Label 4950 2650 0    60   ~ 6
 SD_CMD
-Text Label 4950 2750 0    60   ~ 0
+Text Label 4950 2750 0    60   ~ 6
 GPIO5
-Text Label 4950 2850 0    60   ~ 0
+Text Label 4950 2850 0    60   ~ 6
 SD_DATA
-Text Label 7800 2550 2    60   ~ 0
+Text Label 7800 2550 2    60   ~ 6
 IRDA
-Text Label 7800 2650 2    60   ~ 0
+Text Label 7800 2650 2    60   ~ 6
 USBD-
-Text Label 7800 2750 2    60   ~ 0
+Text Label 7800 2750 2    60   ~ 6
 USBD+
-Text Label 7800 2850 2    60   ~ 0
+Text Label 7800 2850 2    60   ~ 6
 SD_CLK
-Text Label 7800 2450 2    60   ~ 0
+Text Label 7800 2450 2    60   ~ 6
 GND
-Text Label 7800 2350 2    60   ~ 0
+Text Label 7800 2350 2    60   ~ 6
 AUX_DET
-Text Label 7800 2250 2    60   ~ 0
+Text Label 7800 2250 2    60   ~ 6
 AUXR
-Text Label 7800 2150 2    60   ~ 0
+Text Label 7800 2150 2    60   ~ 6
 AUXL
-Text Label 7800 1950 2    60   ~ 0
+Text Label 7800 1950 2    60   ~ 6
 MICIP
-Text Label 7800 1850 2    60   ~ 0
+Text Label 7800 1850 2    60   ~ 6
 MICBIAS
-Text Label 7800 1750 2    60   ~ 0
+Text Label 7800 1750 2    60   ~ 6
 AUDIOLN
-Text Label 7800 1650 2    60   ~ 0
+Text Label 7800 1650 2    60   ~ 6
 AUDIOLP
-Text Label 7800 1550 2    60   ~ 0
+Text Label 7800 1550 2    60   ~ 6
 AUDIORP
-Text Label 7800 1450 2    60   ~ 0
+Text Label 7800 1450 2    60   ~ 6
 AUDIORN
-Text Label 7800 1350 2    60   ~ 0
+Text Label 7800 1350 2    60   ~ 6
 VCCIO
-Text Label 7800 1250 2    60   ~ 0
+Text Label 7800 1250 2    60   ~ 6
 VBAT
-Text Label 7800 1150 2    60   ~ 0
+Text Label 7800 1150 2    60   ~ 6
 V3OUT
-Text Label 7800 1050 2    60   ~ 0
+Text Label 7800 1050 2    60   ~ 6
 ADC
-Text Label 7800 950  2    60   ~ 0
+Text Label 7800 950  2    60   ~ 6
 GND
-Text Label 5100 1250 0    60   ~ 0
+Text Label 5100 1250 0    60   ~ 6
 PREV/VOL-
-Text Label 5100 1350 0    60   ~ 0
+Text Label 5100 1350 0    60   ~ 6
 NEXT/VOL+
-Text Label 5100 1450 0    60   ~ 0
+Text Label 5100 1450 0    60   ~ 6
 P.P/CALL
-Text Label 5100 1550 0    60   ~ 0
+Text Label 5100 1550 0    60   ~ 6
 MODE
-Text Label 4950 2350 0    60   ~ 0
+Text Label 4950 2350 0    60   ~ 6
 GPIO16
 $Comp
@@
 	1    0    0    -1
 $EndComp
-Text Label 8100 3250 2    60   ~ 0
+Text Label 8100 3250 2    60   ~ 6
 GND
 $Comp
@@
 	0    1    1    0
 $EndComp
-Text Label 1250 800  0    60   ~ 0
+Text Label 1250 800  0    60   ~ 6
 MICBIAS
-Text Label 1200 1600 0    60   ~ 0
+Text Label 1200 1600 0    60   ~ 6
 MICIP
 $Comp
@@
 	1    0    0    -1
 $EndComp
-Text Label 10550 5450 2    60   ~ 0
+Text Label 10550 5450 2    60   ~ 6
 AUXL
-Text Label 10550 5100 2    60   ~ 0
+Text Label 10550 5100 2    60   ~ 6
 AUX_DET
-Text Label 10550 5800 2    60   ~ 0
+Text Label 10550 5800 2    60   ~ 6
 AUXR
 $Comp
@@
 	0    1    1    0
 $EndComp
-Text Label 2950 3700 2    60   ~ 0
+Text Label 2950 3700 2    60   ~ 6
 LED1
-Text Label 2950 4100 2    60   ~ 0
+Text Label 2950 4100 2    60   ~ 6
 LED2
 $Comp
@@
 	1    0    0    -1
 $EndComp
-Text Label 2900 5150 2    60   ~ 0
+Text Label 2900 5150 2    60   ~ 6
 PREV/VOL-
-Text Label 2900 5400 2    60   ~ 0
+Text Label 2900 5400 2    60   ~ 6
 NEXT/VOL+
-Text Label 2900 5650 2    60   ~ 0
+Text Label 2900 5650 2    60   ~ 6
 P.P/CALL
-Text Label 2900 5900 2    60   ~ 0
+Text Label 2900 5900 2    60   ~ 6
 MODE
 $Comp
@@
 	1    0    0    -1
 $EndComp
-Text Label 2800 7100 2    60   ~ 0
+Text Label 2800 7100 2    60   ~ 6
 RSTN
 $Comp
@@
 	1    0    0    -1
 $EndComp
-Text Label 3450 5600 0    60   ~ 0
+Text Label 3450 5600 0    60   ~ 6
 SD_CMD
-Text Label 3450 5700 0    60   ~ 0
+Text Label 3450 5700 0    60   ~ 6
 V3OUT
-Text Label 3450 5800 0    60   ~ 0
+Text Label 3450 5800 0    60   ~ 6
 SD_CLK
 Wire Wire Line
@@
 Wire Wire Line
 	4600 6000 3450 6000
-Text Label 3450 6000 0    60   ~ 0
+Text Label 3450 6000 0    60   ~ 6
 SD_DATA
 Wire Wire Line
@@
 Wire Wire Line
 	2450 7100 2800 7100
-Text Label 9150 1350 0    60   ~ 0
+Text Label 9150 1350 0    60   ~ 6
 AUDIORP
-Text Label 9150 1150 0    60   ~ 0
+Text Label 9150 1150 0    60   ~ 6
 AUDIOLP
 Wire Wire Line
@@
 Wire Wire Line
 	9800 3250 9250 3250
-Text Label 10600 3250 2    60   ~ 0
+Text Label 10600 3250 2    60   ~ 6
 5V
-Text Label 9250 3250 0    60   ~ 0
+Text Label 9250 3250 0    60   ~ 6
 VBAT
 $Comp
-L Connector_Specialized:USB_A J1
+L F-6888_breakaout_adapter-rescue:USB_A-Connector_Specialized J1
 U 1 1 5AC5EC95
 P 8950 2450
@@
 	1    0    0    -1
 $EndComp
-Text Label 10450 2550 2    60   ~ 0
+Text Label 10450 2550 2    60   ~ 6
 USBD-
-Text Label 10450 2450 2    60   ~ 0
+Text Label 10450 2450 2    60   ~ 6
 USBD+
-Text Label 9800 2250 2    60   ~ 0
+Text Label 9800 2250 2    60   ~ 6
 5V
 Wire Wire Line
@@
 Wire Wire Line
 	8850 3000 8850 3150
-Text Label 7500 2950 0    60   ~ 0
+Text Label 7500 2950 0    60   ~ 6
 5V
 Wire Wire Line
@@
 Wire Wire Line
 	1850 2150 1650 2150
-Text Label 1200 2150 0    60   ~ 0
+Text Label 1200 2150 0    60   ~ 6
 NC
-Text Label 7800 2050 2    60   ~ 0
+Text Label 7800 2050 2    60   ~ 6
 NC
 $Comp
@@
 Wire Wire Line
 	1000 4650 1650 4650
-Text Label 1650 4650 2    60   ~ 0
+Text Label 1650 4650 2    60   ~ 6
 V3OUT
 Wire Wire Line
@@
 Wire Wire Line
 	2250 800  2700 800
-Text Notes 3450 7550 0    50   ~ 0
+Text Notes 3450 7550 0    50   ~ 6
 * for F-6188 compatibility
 $Comp
@@
 Wire Wire Line
 	10450 1350 10250 1350
-Text Label 2800 6450 2    60   ~ 0
+Text Label 2800 6450 2    60   ~ 6
 V3OUT
 $Comp
@@
 Wire Wire Line
 	9250 2550 9600 2550
-Text Notes 1000 3150 0    50   ~ 0
+Text Notes 1000 3150 0    50   ~ 6
 * BK8000L compatibility
 $EndSCHEMATC
