File: kicad/XS3868_breadboard_adapter/XS3868_breadboard_adapter.sch (KiCad schematic (older format))
At the start: 12 parts, among them J1 SCJ368R1NUS0B00G, P1 CONN_01X12, P2 CONN_01X12, U1 XS3868

Commit message: to fcking much changes to commit it separatly, lets go with everything in one commit, git will love me for sure :D
Parts:
- C1: symbol C -> XS3868_breadboard_adapter-rescue:C-RESCUE-XS3868_breadboard_adapter
- D1, D2: symbol LED -> XS3868_breadboard_adapter-rescue:LED-RESCUE-XS3868_breadboard_adapter
- J1: symbol SCJ368R1NUS0B00G -> phonejack:SCJ368R1NUS0B00G
- ON/OFF/PLAY1, RESET1: symbol SW_Push -> XS3868_breadboard_adapter-rescue:SW_Push-RESCUE-XS3868_breadboard_adapter
- P1: symbol CONN_01X12 -> XS3868_breadboard_adapter-rescue:CONN_01X12-RESCUE-XS3868_breadboard_adapter
- P2: symbol CONN_01X11 -> XS3868_breadboard_adapter-rescue:CONN_01X11-RESCUE-XS3868_breadboard_adapter
- R1, R2, R3: symbol R -> XS3868_breadboard_adapter-rescue:R-RESCUE-XS3868_breadboard_adapter
- U1: symbol XS3868 -> XS3868_breadboard_adapter-rescue:XS3868-RESCUE-XS3868_breadboard_adapter
Connections:
- wire segments 58 -> 74
Changed lines of the file:
@@
-EESchema Schematic File Version 2
-LIBS:XS3868_breadboard_adapter-rescue
-LIBS:power
-LIBS:device
-LIBS:transistors
-LIBS:conn
-LIBS:linear
-LIBS:regul
-LIBS:74xx
-LIBS:cmos4000
-LIBS:adc-dac
-LIBS:memory
-LIBS:xilinx
-LIBS:microcontrollers
-LIBS:dsp
-LIBS:microchip
-LIBS:analog_switches
-LIBS:motorola
-LIBS:texas
-LIBS:intel
-LIBS:audio
-LIBS:interface
-LIBS:digital-audio
-LIBS:philips
-LIBS:display
-LIBS:cypress
-LIBS:siliconi
-LIBS:opto
-LIBS:atmel
-LIBS:contrib
-LIBS:valves
-LIBS:phonejack
-LIBS:XS3868
-LIBS:switches
+EESchema Schematic File Version 4
 LIBS:XS3868_breadboard_adapter-cache
 EELAYER 26 0
@@
 $EndDescr
 $Comp
-L SCJ368R1NUS0B00G J1
+L phonejack:SCJ368R1NUS0B00G J1
 U 1 1 5576DC76
 P 5650 2550
@@
 $EndComp
 $Comp
-L CONN_01X11 P2
+L XS3868_breadboard_adapter-rescue:CONN_01X11-RESCUE-XS3868_breadboard_adapter P2
 U 1 1 5576DF5A
 P 9300 3800
@@
 $EndComp
 $Comp
-L SW_Push RESET1
+L XS3868_breadboard_adapter-rescue:SW_Push-RESCUE-XS3868_breadboard_adapter RESET1
 U 1 1 56C45A37
 P 5400 4950
@@
 $EndComp
 $Comp
-L R R1
+L XS3868_breadboard_adapter-rescue:R-RESCUE-XS3868_breadboard_adapter R1
 U 1 1 56C47B10
 P 5400 5200
@@
 $EndComp
 $Comp
-L SW_Push ON/OFF/PLAY1
+L XS3868_breadboard_adapter-rescue:SW_Push-RESCUE-XS3868_breadboard_adapter ON/OFF/PLAY1
 U 1 1 56C4875B
 P 5700 5700
@@
 $EndComp
 $Comp
-L R R2
+L XS3868_breadboard_adapter-rescue:R-RESCUE-XS3868_breadboard_adapter R2
 U 1 1 56C48674
 P 5550 5850
@@
 $EndComp
 $Comp
-L R R3
+L XS3868_breadboard_adapter-rescue:R-RESCUE-XS3868_breadboard_adapter R3
 U 1 1 56C48760
 P 5550 6150
@@
 $EndComp
 $Comp
-L LED D1
+L XS3868_breadboard_adapter-rescue:LED-RESCUE-XS3868_breadboard_adapter D1
 U 1 1 56C487CC
 P 6100 5850
@@
 $EndComp
 $Comp
-L LED D2
+L XS3868_breadboard_adapter-rescue:LED-RESCUE-XS3868_breadboard_adapter D2
 U 1 1 56C488F4
 P 6100 6150
@@
 $EndComp
 $Comp
-L CONN_01X12 P1
+L XS3868_breadboard_adapter-rescue:CONN_01X12-RESCUE-XS3868_breadboard_adapter P1
 U 1 1 5576DE6D
 P 3400 3850
@@
 	6250 3800 9100 3800
 Wire Wire Line
-	3600 3300 5050 3300
-Wire Wire Line
-	3600 3400 5050 3400
-Wire Wire Line
-	3600 3500 5050 3500
+	3600 3300 4900 3300
+Wire Wire Line
+	3600 3400 4950 3400
+Wire Wire Line
+	3600 3500 5000 3500
 Wire Wire Line
 	3600 3600 5050 3600
@@
 	3600 3700 5050 3700
 Wire Wire Line
-	3600 3800 5050 3800
-Wire Wire Line
-	3600 3900 5050 3900
+	3600 3800 4850 3800
+Wire Wire Line
+	3600 3900 4800 3900
 Wire Wire Line
 	3600 4000 5050 4000
@@
 	5000 5700 5500 5700
 Wire Wire Line
-	5000 4400 5000 6500
+	5000 4400 5000 5700
 Connection ~ 5000 4400
 Wire Wire Line
@@
 	6250 5850 6400 5850
 Wire Wire Line
-	6400 5850 6400 6500
+	6400 5850 6400 6150
 Wire Wire Line
 	6250 6150 6400 6150
@@
 	5250 5200 4950 5200
 Wire Wire Line
-	5600 4950 9000 4950
+	5600 4950 5800 4950
 Wire Wire Line
 	5800 4950 5800 5200
@@
 Connection ~ 5800 4950
 Wire Wire Line
-	3600 4400 5050 4400
+	3600 4400 5000 4400
 Wire Wire Line
 	4800 6150 4800 3900
@@
 Connection ~ 4850 3800
 Wire Wire Line
-	3600 4300 5050 4300
+	3600 4300 4450 4300
 Wire Wire Line
 	3600 4100 5050 4100
 Wire Wire Line
-	3600 4200 5050 4200
+	3600 4200 3800 4200
 Wire Wire Line
 	9100 3900 6250 3900
@@
 	5100 4950 5100 5350
 Wire Wire Line
-	5100 5350 3800 5350
+	5100 5350 4450 5350
 Wire Wire Line
 	6250 4000 9100 4000
@@
 	6250 4100 9100 4100
 Wire Wire Line
-	6250 4200 9100 4200
-Wire Wire Line
-	6250 4300 9100 4300
+	6250 4200 6300 4200
+Wire Wire Line
+	6250 4300 9000 4300
 Wire Wire Line
 	3800 5350 3800 4200
@@
 Connection ~ 6300 4200
 $Comp
-L XS3868 U1
+L XS3868_breadboard_adapter-rescue:XS3868-RESCUE-XS3868_breadboard_adapter U1
 U 1 1 59A82016
 P 5650 3750
@@
 $EndComp
 $Comp
-L C C1
+L XS3868_breadboard_adapter-rescue:C-RESCUE-XS3868_breadboard_adapter C1
 U 1 1 59A824D9
 P 4450 4950
@@
 Connection ~ 4450 4300
 Wire Wire Line
-	4450 5100 4450 5500
+	4450 5100 4450 5350
 Connection ~ 4450 5350
 $Comp
-L GND #PWR?
+L power:GND #PWR?
 U 1 1 59A82F11
 P 4450 5500
@@
 	1    0    0    -1
 $EndComp
+Wire Wire Line
+	5000 3500 5050 3500
+Wire Wire Line
+	4950 3400 5050 3400
+Wire Wire Line
+	4900 3300 5050 3300
+Wire Wire Line
+	4950 4300 5050 4300
+Wire Wire Line
+	5000 4400 5050 4400
+Wire Wire Line
+	5000 5700 5000 6500
+Wire Wire Line
+	6400 6150 6400 6500
+Wire Wire Line
+	5800 4950 9000 4950
+Wire Wire Line
+	4800 3900 5050 3900
+Wire Wire Line
+	4850 3800 5050 3800
+Wire Wire Line
+	3800 4200 5050 4200
+Wire Wire Line
+	9000 4300 9100 4300
+Wire Wire Line
+	6300 4200 9100 4200
+Wire Wire Line
+	4450 4300 4950 4300
+Wire Wire Line
+	4450 5350 3800 5350
+Wire Wire Line
+	4450 5350 4450 5500
 $EndSCHEMATC

Commit message: update
Parts:
- removed C1: 100n, Capacitors_SMD:C_1206, symbol XS3868_breadboard_adapter-rescue:C-RESCUE-XS3868_breadboard_adapter
- removed J1: SCJ368R1NUS0B00G, jacks:3.5mm_stereo_jack_PJ320B, symbol phonejack:SCJ368R1NUS0B00G
- removed U1: XS3868, modules:XS3868, symbol XS3868_breadboard_adapter-rescue:XS3868-RESCUE-XS3868_breadboard_adapter
- added C1: 100n, Capacitors_SMD.pretty:C_0805_HandSoldering, symbol c:C
- added C2: 4u7, Capacitors_SMD.pretty:C_1206_HandSoldering, symbol c:C
- added C3: 2u2/6.5V, Capacitors_SMD.pretty:C_0805_HandSoldering, symbol c:C
- added C4: 220p/optional, Capacitors_SMD.pretty:C_0805_HandSoldering, symbol c:C
- added C5, C6, C7: 10uF, Capacitors_SMD.pretty:C_1206_HandSoldering, symbol c:C
- added J1: OUT, jacks:3.5mm_stereo_jack_PJ320B, symbol jacks:PJ-320B
- added J2: MIC, jacks:3.5mm_stereo_jack_PJ320B, symbol jacks:PJ-320B
- added L1: 15n, Choke_SMD.pretty:Choke_SMD_1206_Handsoldering, symbol Device:L
- added R4: 2k2, Resistors_SMD:R_0805_HandSoldering, symbol Device:R
- added R5: 2k, Resistors_SMD:R_0805_HandSoldering, symbol Device:R
- added SW1: PREVIOUS, Buttons_Switches_SMD:SW_SPST_FSMSM, symbol switch:SW_PUSH
- added SW2: NEXT, Buttons_Switches_SMD:SW_SPST_FSMSM, symbol switch:SW_PUSH
- added SW3: VOL-, Buttons_Switches_SMD:SW_SPST_FSMSM, symbol switch:SW_PUSH
- added SW4: VOL+, Buttons_Switches_SMD:SW_SPST_FSMSM, symbol switch:SW_PUSH
- added U1: XS3868, bluetooth:XS3868, symbol xs3868:XS3868
- DG1: renamed from D1; value LED -> GREEN; footprint LEDs:LED_1206 -> LEDs:LED-1206; symbol XS3868_breadboard_adapter-rescue:LED-RESCUE-XS3868_breadboard_adapter -> Device:LED
- DR2: renamed from D2; value LED -> RED; footprint LEDs:LED_1206 -> LEDs:LED-1206; symbol XS3868_breadboard_adapter-rescue:LED-RESCUE-XS3868_breadboard_adapter -> Device:LED
- P1: footprint Pin_Headers.pretty:Pin_Header_Straight_1x12 -> Pin_Headers:Pin_Header_Straight_1x12_Pitch2.54mm; symbol XS3868_breadboard_adapter-rescue:CONN_01X12-RESCUE-XS3868_breadboard_adapter -> Connector_Generic:Conn_01x12_Male
- P2: footprint Pin_Headers.pretty:Pin_Header_Straight_1x11 -> Pin_Headers:Pin_Header_Straight_1x12_Pitch2.54mm; symbol XS3868_breadboard_adapter-rescue:CONN_01X11-RESCUE-XS3868_breadboard_adapter -> Connector_Generic:Conn_01x12_Male
- R1: renamed from R2; symbol XS3868_breadboard_adapter-rescue:R-RESCUE-XS3868_breadboard_adapter -> Device:R
- R2: renamed from R3; symbol XS3868_breadboard_adapter-rescue:R-RESCUE-XS3868_breadboard_adapter -> Device:R
- R3: renamed from R1; symbol XS3868_breadboard_adapter-rescue:R-RESCUE-XS3868_breadboard_adapter -> Device:R
- SW5: renamed from ON/OFF/PLAY1; symbol XS3868_breadboard_adapter-rescue:SW_Push-RESCUE-XS3868_breadboard_adapter -> switch:SW_PUSH
- SW6: renamed from RESET1; value 1 -> RESET; symbol XS3868_breadboard_adapter-rescue:SW_Push-RESCUE-XS3868_breadboard_adapter -> switch:SW_PUSH
Connections:
- net labels added: 1V8, AOL, AOM, AOR, LED1, LED2, MFB1, MIC+, MICBIAS, MODE, MUTE, NEXT, ONKEY, PREVIOUS, RESET, UART_RX, UART_TX, VBAT, VBUCK, VCC, VOL+, VOL-
- wire segments 74 -> 89
- no-connect marks 0 -> 1
Other:
- note added: "this is at blk "datasheet"\nI put it here just in case\ns3860-m "datasheet"\nis missing this parts"

Commit message: update
Changed lines of the file:
@@
 Text Label 7000 2150 0    50   ~ 0
 VCC
-Text Label 7000 2250 0    50   ~ 0
+Text Label 6950 2350 0    50   ~ 0
 VBUCK
 $Comp
@@
 	-1   0    0    1
 $EndComp
-Text Label 7000 2350 0    50   ~ 0
+Text Label 7000 2250 0    50   ~ 0
 GND
 Wire Wire Line

Commit message: update xs3868 kicad project files
Parts:
- C1, C2, C3, C4, C5, C6, C7: symbol c:C -> XS3868_breadboard_adapter-rescue:C-c
- P1, P2: symbol Connector_Generic:Conn_01x12_Male -> XS3868_breadboard_adapter-rescue:Conn_01x12_Male-Connector_Generic
- SW1, SW2, SW3, SW4, SW5, SW6: symbol switch:SW_PUSH -> XS3868_breadboard_adapter-rescue:SW_PUSH-switch
- U1: symbol xs3868:XS3868 -> XS3868_breadboard_adapter-rescue:XS3868-xs3868
Changed lines of the file:
@@
-EESchema Schematic File Version 4
+EESchema Schematic File Version 5
 LIBS:XS3868_breadboard_adapter-cache
 EELAYER 29 0
@@
 $EndDescr
 $Comp
-L xs3868:XS3868 U1
+L XS3868_breadboard_adapter-rescue:XS3868-xs3868 U1
 U 1 1 5576DBD3
 P 7950 1900
@@
 $EndComp
 $Comp
-L switch:SW_PUSH SW6
+L XS3868_breadboard_adapter-rescue:SW_PUSH-switch SW6
 U 1 1 56C45A37
 P 8350 6000
@@
 $EndComp
 $Comp
-L switch:SW_PUSH SW5
+L XS3868_breadboard_adapter-rescue:SW_PUSH-switch SW5
 U 1 1 56C4875B
 P 8350 5650
@@
 VBUCK
 $Comp
-L c:C C1
+L XS3868_breadboard_adapter-rescue:C-c C1
 U 1 1 5A910B1E
 P 4350 6100
@@
 Connection ~ 8750 6000
 $Comp
-L switch:SW_PUSH SW4
+L XS3868_breadboard_adapter-rescue:SW_PUSH-switch SW4
 U 1 1 5BD7EF33
 P 8350 5250
@@
 	8050 5250 7650 5250
 $Comp
-L switch:SW_PUSH SW3
+L XS3868_breadboard_adapter-rescue:SW_PUSH-switch SW3
 U 1 1 5BD80C91
 P 8350 4800
@@
 $EndComp
 $Comp
-L switch:SW_PUSH SW2
+L XS3868_breadboard_adapter-rescue:SW_PUSH-switch SW2
 U 1 1 5BD80C9A
 P 8350 4400
@@
 $EndComp
 $Comp
-L switch:SW_PUSH SW1
+L XS3868_breadboard_adapter-rescue:SW_PUSH-switch SW1
 U 1 1 5BD82B1B
 P 8350 3950
@@
 $EndComp
 $Comp
-L c:C C4
+L XS3868_breadboard_adapter-rescue:C-c C4
 U 1 1 5BD9018D
 P 3700 4000
@@
 $EndComp
 $Comp
-L c:C C3
+L XS3868_breadboard_adapter-rescue:C-c C3
 U 1 1 5BD903C6
 P 3200 3650
@@
 	9350 2050 8550 2050
 $Comp
-L Connector_Generic:Conn_01x12_Male P2
+L XS3868_breadboard_adapter-rescue:Conn_01x12_Male-Connector_Generic P2
 U 1 1 5576DF5A
 P 10550 1950
@@
 	7350 2450 6650 2450
 $Comp
-L Connector_Generic:Conn_01x12_Male P1
+L XS3868_breadboard_adapter-rescue:Conn_01x12_Male-Connector_Generic P1
 U 1 1 5576DE6D
 P 6450 2050
@@
 	4100 3850 4200 3850
 $Comp
-L c:C C6
+L XS3868_breadboard_adapter-rescue:C-c C6
 U 1 1 5BE2591C
 P 3250 1550
@@
 $EndComp
 $Comp
-L c:C C7
+L XS3868_breadboard_adapter-rescue:C-c C7
 U 1 1 5BE2604A
 P 3250 1750
@@
 $EndComp
 $Comp
-L c:C C5
+L XS3868_breadboard_adapter-rescue:C-c C5
 U 1 1 5BE26205
 P 3250 1950
@@
 	2400 3250 2200 3250
 $Comp
-L c:C C2
+L XS3868_breadboard_adapter-rescue:C-c C2
 U 1 1 5BD76587
 P 2200 3600
