File: kicad/audi_trunk_led_light/audi_trunk_led_light.sch (KiCad schematic (older format))
At the start: 77 parts, among them P1 CONN_01X02, P2 CONN_01X02

Commit message: update
Parts:
- D1, D10, D11, D12, D13, D14, D15, D16, D17, D18, D19, D2, D20, D21, D22, D23, D24, D25, D26, D27, D28, D29, D3, D30, D31, D32, D33, D34, D35, D36, D4, D5, D6, D7, D8, D9: symbol LED_RGB -> audi_trunk_led_light-rescue:LED_RGB
- P1, P2: symbol CONN_01X01 -> audi_trunk_led_light-rescue:CONN_01X01
- R1, R10, R11, R12, R13, R14, R15, R16, R17, R18, R19, R2, R20, R21, R22, R23, R24, R25, R26, R27, R28, R29, R3, R30, R31, R32, R33, R34, R35, R36, R37, R38, R39, R4, R5, R6, R7, R8, R9: symbol R -> rgb_led_toy:R
Connections:
- wire segments 194 -> 270
