File: kicad/42mm_car_interior_LED/42mm_cat_interior_LED.sch (KiCad schematic (older format))
At the start: 39 parts, among them P1 CONN_01X01, P2 CONN_01X01, P3 CONN_01X01, P4 CONN_01X01

Commit message: update
Parts:
- C1, C2, C3: symbol CP -> 42mm_cat_interior_LED-rescue:CP
- D1, D10, D11, D12, D13, D14, D15, D16, D2, D3, D4, D5, D6, D7, D8, D9: symbol LED_RGB -> 42mm_cat_interior_LED-rescue:LED_RGB
- D17, D18, D20, D21: symbol D -> 42mm_cat_interior_LED-rescue:D
- P1, P2, P3, P4: symbol CONN_01X01 -> 42mm_cat_interior_LED-rescue:CONN_01X01
- R13, R14, R15, R16, R17, R18, R19, R20, R21, R22, R23, R24: symbol R -> 42mm_cat_interior_LED-rescue:R
Changed lines of the file:
@@
-EESchema Schematic File Version 2
-LIBS:power
-LIBS:device
-LIBS:transistors
-LIBS:conn
-LIBS:linear
-LIBS:regul
-LIBS:74xx
-LIBS:cmos4000
-LIBS:adc-dac
-LIBS:memory
-LIBS:xilinx
-LIBS:microcontrollers
-LIBS:dsp
-LIBS:microchip
-LIBS:analog_switches
-LIBS:motorola
-LIBS:texas
-LIBS:intel
-LIBS:audio
-LIBS:interface
-LIBS:digital-audio
-LIBS:philips
-LIBS:display
-LIBS:cypress
-LIBS:siliconi
-LIBS:opto
-LIBS:atmel
-LIBS:contrib
-LIBS:valves
+EESchema Schematic File Version 4
 LIBS:42mm_cat_interior_LED-cache
-EELAYER 25 0
+EELAYER 29 0
 EELAYER END
 $Descr A4 11693 8268
@@
 $EndDescr
 $Comp
-L LED_RGB D10
+L 42mm_cat_interior_LED-rescue:LED_RGB D10
 U 1 1 5652DCB5
 P 4600 2500
@@
 $EndComp
 $Comp
-L LED_RGB D7
+L 42mm_cat_interior_LED-rescue:LED_RGB D7
 U 1 1 5652E21C
 P 4050 2500
@@
 $EndComp
 $Comp
-L LED_RGB D4
+L 42mm_cat_interior_LED-rescue:LED_RGB D4
 U 1 1 5652E253
 P 3500 2500
@@
 $EndComp
 $Comp
-L LED_RGB D1
+L 42mm_cat_interior_LED-rescue:LED_RGB D1
 U 1 1 5652E287
 P 3000 2500
@@
 $EndComp
 $Comp
-L LED_RGB D11
+L 42mm_cat_interior_LED-rescue:LED_RGB D11
 U 1 1 5652E995
 P 4600 3300
@@
 $EndComp
 $Comp
-L LED_RGB D8
+L 42mm_cat_interior_LED-rescue:LED_RGB D8
 U 1 1 5652E9AD
 P 4050 3300
@@
 $EndComp
 $Comp
-L LED_RGB D5
+L 42mm_cat_interior_LED-rescue:LED_RGB D5
 U 1 1 5652E9B3
 P 3500 3300
@@
 $EndComp
 $Comp
-L LED_RGB D2
+L 42mm_cat_interior_LED-rescue:LED_RGB D2
 U 1 1 5652E9B9
 P 3000 3300
@@
 $EndComp
 $Comp
-L LED_RGB D12
+L 42mm_cat_interior_LED-rescue:LED_RGB D12
 U 1 1 5652EBAE
 P 5050 4050
@@
 $EndComp
 $Comp
-L LED_RGB D9
+L 42mm_cat_interior_LED-rescue:LED_RGB D9
 U 1 1 5652EBC6
 P 4500 4050
@@
 $EndComp
 $Comp
-L LED_RGB D6
+L 42mm_cat_interior_LED-rescue:LED_RGB D6
 U 1 1 5652EBCC
 P 3950 4050
@@
 $EndComp
 $Comp
-L LED_RGB D3
+L 42mm_cat_interior_LED-rescue:LED_RGB D3
 U 1 1 5652EBD2
 P 3450 4050
@@
 $EndComp
 $Comp
-L CONN_01X01 P1
+L 42mm_cat_interior_LED-rescue:CONN_01X01 P1
 U 1 1 5652FEAD
 P 9100 2200
@@
 $EndComp
 $Comp
-L CONN_01X01 P2
+L 42mm_cat_interior_LED-rescue:CONN_01X01 P2
 U 1 1 5652FFE0
 P 9050 1500
@@
 $EndComp
 $Comp
-L LED_RGB D16
+L 42mm_cat_interior_LED-rescue:LED_RGB D16
 U 1 1 56530B8D
 P 5050 4850
@@
 $EndComp
 $Comp
-L LED_RGB D15
+L 42mm_cat_interior_LED-rescue:LED_RGB D15
 U 1 1 56530BA5
 P 4500 4850
@@
 $EndComp
 $Comp
-L LED_RGB D14
+L 42mm_cat_interior_LED-rescue:LED_RGB D14
 U 1 1 56530BAB
 P 3950 4850
@@
 $EndComp
 $Comp
-L LED_RGB D13
+L 42mm_cat_interior_LED-rescue:LED_RGB D13
 U 1 1 56530BB1
 P 3450 4850
@@
 MINUS
 $Comp
-L D D20
+L 42mm_cat_interior_LED-rescue:D D20
 U 1 1 5654878B
 P 8400 4850
@@
 $EndComp
 $Comp
-L D D17
+L 42mm_cat_interior_LED-rescue:D D17
 U 1 1 565488BC
 P 7800 4850
@@
 $EndComp
 $Comp
-L D D21
+L 42mm_cat_interior_LED-rescue:D D21
 U 1 1 565489C7
 P 8400 5150
@@
 $EndComp
 $Comp
-L D D18
+L 42mm_cat_interior_LED-rescue:D D18
 U 1 1 56548A77
 P 7800 5150
@@
 IN1
 $Comp
-L R R19
+L 42mm_cat_interior_LED-rescue:R R19
 U 1 1 56548B2B
 P 5100 2300
@@
 $EndComp
 $Comp
-L R R20
+L 42mm_cat_interior_LED-rescue:R R20
 U 1 1 56548C8F
 P 5100 2500
@@
 $EndComp
 $Comp
-L R R21
+L 42mm_cat_interior_LED-rescue:R R21
 U 1 1 56548D12
 P 5100 2700
@@
 $EndComp
 $Comp
-L R R22
+L 42mm_cat_interior_LED-rescue:R R22
 U 1 1 56548F64
 P 5100 3100
@@
 $EndComp
 $Comp
-L R R23
+L 42mm_cat_interior_LED-rescue:R R23
 U 1 1 56548FF7
 P 5100 3300
@@
 $EndComp
 $Comp
-L R R24
+L 42mm_cat_interior_LED-rescue:R R24
 U 1 1 565490AB
 P 5100 3500
@@
 $EndComp
 $Comp
-L R R13
+L 42mm_cat_interior_LED-rescue:R R13
 U 1 1 56549779
 P 2950 3850
@@
 $EndComp
 $Comp
-L R R14
+L 42mm_cat_interior_LED-rescue:R R14
 U 1 1 5654984D
 P 2950 4050
@@
 $EndComp
 $Comp
-L R R15
+L 42mm_cat_interior_LED-rescue:R R15
 U 1 1 565498E2
 P 2950 4250
@@
 $EndComp
 $Comp
-L R R16
+L 42mm_cat_interior_LED-rescue:R R16
 U 1 1 56549D46
 P 2950 4650
@@
 $EndComp
 $Comp
-L R R17
+L 42mm_cat_interior_LED-rescue:R R17
 U 1 1 56549DEB
 P 2950 4850
@@
 $EndComp
 $Comp
-L R R18
+L 42mm_cat_interior_LED-rescue:R R18
 U 1 1 56549E89
 P 2950 5050
@@
 Connection ~ 5350 3500
 Wire Wire Line
-	5250 3300 6200 3300
+	5250 3300 5350 3300
 Connection ~ 5350 3300
 Wire Wire Line
@@
 Connection ~ 2300 3500
 Wire Wire Line
-	1750 3300 2800 3300
+	1750 3300 2300 3300
 Connection ~ 2300 3300
 Wire Wire Line
@@
 Connection ~ 2300 4250
 Wire Wire Line
-	2300 2300 2300 5050
+	2300 2300 2300 2500
 Wire Wire Line
 	8550 4850 8650 4850
 Wire Wire Line
-	8650 4850 8650 5150
+	8650 4850 8650 5000
 Wire Wire Line
 	8650 5150 8550 5150
 Wire Wire Line
-	7550 4850 7550 5150
+	7550 4850 7550 5000
 Wire Wire Line
 	7550 5150 7650 5150
@@
 	7650 4850 7550 4850
 Wire Wire Line
-	7950 4850 8250 4850
-Wire Wire Line
-	7950 5150 8250 5150
+	7950 4850 8100 4850
+Wire Wire Line
+	7950 5150 8100 5150
 Connection ~ 8100 4850
 Connection ~ 8100 5150
@@
 	8100 5400 8100 5150
 $Comp
-L CP C1
+L 42mm_cat_interior_LED-rescue:CP C1
 U 1 1 56654E40
 P 8050 2900
@@
 	7600 2900 7900 2900
 $Comp
-L CP C2
+L 42mm_cat_interior_LED-rescue:CP C2
 U 1 1 566552E6
 P 8050 3400
@@
 	7600 3400 7900 3400
 $Comp
-L CP C3
+L 42mm_cat_interior_LED-rescue:CP C3
 U 1 1 566553F8
 P 8050 4050
@@
 	7600 4050 7900 4050
 $Comp
-L CONN_01X01 P4
+L 42mm_cat_interior_LED-rescue:CONN_01X01 P4
 U 1 1 56658CEF
 P 7850 2200
@@
 $EndComp
 $Comp
-L CONN_01X01 P3
+L 42mm_cat_interior_LED-rescue:CONN_01X01 P3
 U 1 1 56658CF5
 P 7800 1500
@@
 	6950 2200 7650 2200
 Wire Wire Line
-	5350 2300 5350 5050
+	5350 2300 5350 2500
+Wire Wire Line
+	5350 4050 5350 4250
+Wire Wire Line
+	5350 3850 5350 4050
+Wire Wire Line
+	5350 3500 5350 3850
+Wire Wire Line
+	5350 3300 6200 3300
+Wire Wire Line
+	5350 3300 5350 3500
+Wire Wire Line
+	5350 3100 5350 3300
+Wire Wire Line
+	5350 2700 5350 3100
+Wire Wire Line
+	2300 4050 2300 4250
+Wire Wire Line
+	2300 3850 2300 4050
+Wire Wire Line
+	2300 3500 2300 3850
+Wire Wire Line
+	2300 3300 2800 3300
+Wire Wire Line
+	2300 3300 2300 3500
+Wire Wire Line
+	2300 3100 2300 3300
+Wire Wire Line
+	2300 2700 2300 3100
+Wire Wire Line
+	2300 2500 2300 2700
+Wire Wire Line
+	5350 2500 5350 2700
+Wire Wire Line
+	5350 4850 5350 5050
+Wire Wire Line
+	5350 4650 5350 4850
+Wire Wire Line
+	2300 4850 2300 5050
+Wire Wire Line
+	2300 4650 2300 4850
+Wire Wire Line
+	5350 4250 5350 4650
+Wire Wire Line
+	2300 4250 2300 4650
+Wire Wire Line
+	8100 4850 8250 4850
+Wire Wire Line
+	8100 5150 8250 5150
+Wire Wire Line
+	7550 5000 7550 5150
+Wire Wire Line
+	8650 5000 8650 5150
 $EndSCHEMATC
