File: kicad/F-6888_breakaout_adapter/old/v1/F-6888_breakout_board.sch (KiCad schematic (older format))
At the start: 5 parts, among them CON1 CONN_20, CON2 CONN_20, J1 Jack_3.5mm_5pin, U1 F-6888

Commit message: update
Parts:
- CON1, CON2: symbol gencon:CONN_20 -> F-6888_breakout_board-rescue:CONN_20-gencon
- U1: symbol F-6888:F-6888 -> F-6888_breakout_board-rescue:F-6888-F-6888
Changed lines of the file:
@@
 EESchema Schematic File Version 4
-EELAYER 26 0
+LIBS:F-6888_breakout_board-cache
+EELAYER 29 0
 EELAYER END
 $Descr A4 11693 8268
@@
 $EndDescr
 $Comp
-L gencon:CONN_20 CON1
+L F-6888_breakout_board-rescue:CONN_20-gencon CON1
 U 1 1 5A847A68
 P 2800 3850
@@
 	3200 4100 3550 4100
 $Comp
-L gencon:CONN_20 CON2
+L F-6888_breakout_board-rescue:CONN_20-gencon CON2
 U 1 1 5A84AD5B
 P 5850 3850
@@
 	3250 4400 3550 4400
 $Comp
-L F-6888:F-6888 U1
+L F-6888_breakout_board-rescue:F-6888-F-6888 U1
 U 1 1 5AA6C3D3
 P 4300 3050
