File: kicad/F-6888_breakaout_adapter/old/v2/F-6888_breakaout_adapter.sch (KiCad schematic (older format))
At the start: 29 parts, among them J1 USB_A, J2 CONN_01X20, J3 MIC, J4 CONN_01X20, J6 Micro_SD_Card_Det, SW1 RESET, SW2 PREV/VOL-, SW3 NEXT/VOL+, SW4 P.P/CALL, SW5 MODE, U1 F-6888

Commit message: update
Parts:
- J1: symbol Connector_Specialized:USB_A -> F-6888_breakaout_adapter-rescue:USB_A-Connector_Specialized
- J6: symbol Connector_Specialized:Micro_SD_Card_Det_Hirose_DM3AT -> F-6888_breakaout_adapter-rescue:Micro_SD_Card_Det_Hirose_DM3AT-Connector_Specialized
- PJ-327A1, PJ-327A2: symbol gencon:CONN_6 -> F-6888_breakaout_adapter-rescue:CONN_6-gencon
- U1: symbol F-6888:F-6888 -> F-6888_breakaout_adapter-rescue:F-6888-F-6888
Changed lines of the file:
@@
 EESchema Schematic File Version 4
 LIBS:F-6888_breakaout_adapter-cache
-EELAYER 26 0
+EELAYER 29 0
 EELAYER END
 $Descr A4 11693 8268
@@
 $EndDescr
 $Comp
-L F-6888:F-6888 U1
+L F-6888_breakaout_adapter-rescue:F-6888-F-6888 U1
 U 1 1 59BA8F51
 P 5850 2600
@@
 VBAT
 $Comp
-L Connector_Specialized:Micro_SD_Card_Det_Hirose_DM3AT J6
+L F-6888_breakaout_adapter-rescue:Micro_SD_Card_Det_Hirose_DM3AT-Connector_Specialized J6
 U 1 1 59BB90AF
 P 5550 6600
@@
 	2700 2600 3050 2600
 $Comp
-L gencon:CONN_6 PJ-327A1
+L F-6888_breakaout_adapter-rescue:CONN_6-gencon PJ-327A1
 U 1 1 5A90F45F
 P 8200 1450
@@
 	8950 1700 8950 1900
 $Comp
-L gencon:CONN_6 PJ-327A2
+L F-6888_breakaout_adapter-rescue:CONN_6-gencon PJ-327A2
 U 1 1 5A92B891
 P 9150 2550
@@
 VBAT
 $Comp
-L Connector_Specialized:USB_A J1
+L F-6888_breakaout_adapter-rescue:USB_A-Connector_Specialized J1
 U 1 1 5AC5EC95
 P 8450 3950
