File: kicad/arduino_nanoXX4/arduino_nano324.kicad_pcb (KiCad board)
At the start: 2 copper layers, 24.4 x 64.5 mm, 51 parts, among them J1 USB_B_Micro, P1 Digital, P2 Analog, P3 CONN_01X01, P4 CONN_01X01, P5 CONN_01X01, P6 CONN_01X01, P7 CONN_6, SW1 SW_PUSH, U1 ATMEGA324PB-AU, U2 CP2102N-A01-GQFN28, U3 AP1117-50, U4 AP1117-33, X1 CRYSTAL, Y1 16Mhz

Commit message: init public commit
Other:
- board text added: "7: D|X"
- board text added: "8: D|X"
Changed lines of the file:
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@@
-(kicad_pcb (version 20190331) (host pcbnew "6.0.0-unknown-a40367c~86~ubuntu16.04.1")
+(kicad_pcb (version 20190605) (host pcbnew "6.0.0-unknown-dd938b0~86~ubuntu16.04.1")
   (general
     (thickness 1.6)
@@
     (uvia_min_size 0.2)
     (uvia_min_drill 0.1)
-    (edge_width 0.5)
-    (segment_width 0.15)
-    (pcb_text_width 0.1)
-    (pcb_text_size 0.8 0.8)
-    (mod_edge_width 0.15)
-    (mod_text_size 0.8 0.8)
-    (mod_text_width 0.1)
+    (max_error 0.005)
+    (defaults
+      (edge_clearance 0.01)
+      (edge_cuts_line_width 0.5)
+      (courtyard_line_width 0.05)
+      (copper_line_width 0.15)
+      (copper_text_dims (size 0.8 0.8) (thickness 0.1) keep_upright)
+      (silk_line_width 0.15)
+      (silk_text_dims (size 0.8 0.8) (thickness 0.1) keep_upright)
+      (other_layers_line_width 0.1)
+      (other_layers_text_dims (size 1 1) (thickness 0.15) keep_upright)
+    )
     (pad_size 1.5 1.5)
     (pad_drill 0.6)
@@
     (visible_elements FFFFFF7F)
     (pcbplotparams
-      (layerselection 0x00020_7ffffffe)
+      (layerselection 0x30030_7ffffffe)
       (usegerberextensions true)
       (usegerberattributes false)
@@
       (plotreference true)
       (plotvalue true)
-      (plotinvisibletext false)
+      (plotinvisibletext true)
       (padsonsilk false)
       (subtractmaskfromsilk true)
@@
       (drillshape 2)
       (scaleselection 1)
-      (outputdirectory ""))
+      (outputdirectory "AP/"))
   )
   (net 0 "")
@@
     (effects (font (size 0.8 0.8) (thickness 0.1)) (justify mirror))
   )
-  (gr_text "PB|PA" (at 192.6844 98.7171 270) (layer "B.SilkS")
+  (gr_text "7: D|X" (at 192.3796 99.6188 270) (layer "B.SilkS")
     (effects (font (size 0.8 0.8) (thickness 0.1)) (justify mirror))
   )
-  (gr_text "PB|PA" (at 196.56044 98.77552 270) (layer "B.SilkS")
+  (gr_text "8: D|X" (at 196.342 99.7204 270) (layer "B.SilkS")
     (effects (font (size 0.8 0.8) (thickness 0.1)) (justify mirror))
   )
@@
     (connect_pads (clearance 0.2))
     (min_thickness 0.254)
-    (fill yes (arc_segments 32) (thermal_gap 0.508) (thermal_bridge_width 0.508))
+    (fill yes (thermal_gap 0.508) (thermal_bridge_width 0.508))
     (polygon
       (pts
@@
     (connect_pads (clearance 0.2))
     (min_thickness 0.254)
-    (fill yes (arc_segments 32) (thermal_gap 0.508) (thermal_bridge_width 0.508))
+    (fill yes (thermal_gap 0.508) (thermal_bridge_width 0.508))
     (polygon
       (pts
