File: kicad/arduino_mega_all_pins/arduino_mega_all_pins.kicad_pcb (KiCad board)
At the start: 2 copper layers, 101.6 x 53.3 mm, 75 parts, among them J1 USB_B, J2 USB_B_Micro, J3 DC_JACK, J4 USB_B_Micro, P1 Digital, P10 CONN_01X01, P11 CONN_01X01, P12 CONN_01X01, P13 CONN_01X01, P14 xx2, P15 CP2102, P16 CONN_6, P17 CONN_1x1, P19 Digital, P2 Power, P20 Analog, P21 Digital, P22 Digital, P3 Analog, P4 Analog, P5 PWM, P6 PWM, P7 Communication, P8 CONN_01X01, P9 CONN_01X01, SW1 SW_PUSH, SW2 SW_PUSH, U1 CP2104, U2 ATMEGA2560-16AU, U3 AP1117-50, U4 AP1117-50, X1 32.768kHz (optional), X2 16MHz, X3 16MHz, Y1 Resonator 16MHz, Y2 Crystal_GND23 16MHz

Commit message: pcb v2.0
Parts:
- added R10: 1k, Resistors_SMD.pretty:R_0805_HandSoldering, F.Cu at (128.9, 80.5)
- added R11: 1k, Resistors_SMD.pretty:R_0805_HandSoldering, F.Cu at (130.3, 102.4)
- F1: value Fuse -> 0.5A
- JP1: footprint Jumper:SolderJumper-2_P1.3mm_Bridged_RoundedPad1.0x1.5mm -> Jumper:SolderJumper-2_P1.3mm_Open_RoundedPad1.0x1.5mm
- L2: value L -> bead_30
- U4: value AP1117-50 -> AP1117-33
- moved JP1 0.99 mm to (131.7, 98.3), turned to -90 degrees
- moved P2 0.25 mm to (131.3, 119.1)
- turned C7 to 0 degrees
Connections:
- JP1 pad 2: /DTR -> Net-(C6-Pad2)
- R5 pad 1: /RXLED -> /0(Rx0)
- R6 pad 1: /TXLED -> /1(Tx0)
- U1 pad 13: /RXLED -> (no net)
- U1 pad 14: /TXLED -> (no net)
- U1 pad 20: /1(Tx0) -> Net-(R10-Pad2)
- U2 pad 43: (no net) -> /21(SCL)
- U2 pad 44: (no net) -> /20(SDA)
Routing:
- net /0(Rx0): track 67.1 -> 101.6 mm, vias 2 -> 4
- net /RXLED: track 24.7 -> 0.00 mm, vias 2 -> 0
- net /1(Tx0): track 66.8 -> 86.6 mm, vias 1 -> 3
- net /TXLED: track 18.0 -> 0.00 mm, vias 2 -> 0
- net /DTR: track 26.8 -> 34.8 mm
- net Net-(R10-Pad2): track 0.00 -> 5.61 mm
- net Net-(C7-Pad1): track 19.5 -> 14.9 mm
- net Net-(C6-Pad2): track 10.2 -> 14.5 mm, vias 2 -> 0
- net GND: track 365.7 -> 368.6 mm
