File: kicad/BM20_breadboard_adapter/BM20_breadboard_adapter.kicad_sch (KiCad schematic)
At the start: 28 parts, among them CON1 CONN_18, CON2 CONN_18, CON3 batt, J1 PJ-320B, J2 PJ-320B, J3 USB_B_Micro, SW1 SWITCH_SPST, SW2 SWITCH_SPST, U1 BM20, U2 PJ-3027F

Commit message: new module hw
Parts:
- removed U2: PJ-3027F, jacks:PJ-3027F-S, symbol jacks:PJ-3027F
- added U2: PJ-3027F, jacks:PJ-327A, symbol jacks:PJ-327A
Connections:
- net 15: no longer C11.2
- net 3: now also U2.3
- net GND: now also U2.4
- net at C11.1: now also U2.2, U2.6
- net at C10.2: now also U2.5
Changed lines of the file:
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@@
   (page 1 1)
   (paper "A4")
+  (junction (at 47.371 87.63))
   (junction (at 49.53 62.23))
   (junction (at 49.53 125.73))
@@
     (stroke (width 0) (type solid) (color 0 0 0 0))
   )
-  (wire (pts (xy 44.45 87.63) (xy 57.15 87.63))
-    (stroke (width 0) (type solid) (color 0 0 0 0))
-  )
-  (wire (pts (xy 44.45 92.71) (xy 49.53 92.71))
+  (wire (pts (xy 44.45 85.09) (xy 47.371 85.09))
+    (stroke (width 0) (type solid) (color 0 0 0 0))
+  )
+  (wire (pts (xy 44.45 87.63) (xy 47.371 87.63))
+    (stroke (width 0) (type solid) (color 0 0 0 0))
+  )
+  (wire (pts (xy 44.45 90.17) (xy 49.53 90.17))
+    (stroke (width 0) (type solid) (color 0 0 0 0))
+  )
+  (wire (pts (xy 47.371 85.09) (xy 47.371 87.63))
+    (stroke (width 0) (type solid) (color 0 0 0 0))
+  )
+  (wire (pts (xy 47.371 87.63) (xy 57.15 87.63))
     (stroke (width 0) (type solid) (color 0 0 0 0))
   )
@@
     (stroke (width 0) (type solid) (color 0 0 0 0))
   )
-  (wire (pts (xy 49.53 92.71) (xy 49.53 104.14))
+  (wire (pts (xy 49.53 90.17) (xy 49.53 104.14))
     (stroke (width 0) (type solid) (color 0 0 0 0))
   )
@@
     (effects (font (size 1.27 1.27)) (justify right bottom))
   )
-  (label "AIL" (at 82.55 87.63 180)
+  (label "AIL" (at 82.55 90.17 180)
     (effects (font (size 1.27 1.27)) (justify right bottom))
   )
@@
     )
   )
-  (symbol (lib_id "jacks:PJ-3027F") (at 35.56 85.09 0) (unit 1)
-    (in_bom yes)
-    (property "Reference" "U2" (id 0) (at 37.6174 71.755 0))
-    (property "Value" "PJ-3027F" (id 1) (at 37.6174 74.0664 0))
-    (property "Footprint" "jacks:PJ-3027F-S" (id 2) (at 35.56 87.63 0)
-      (effects (font (size 1.27 1.27)) hide)
-    )
-    (property "Datasheet" "" (id 3) (at 35.56 87.63 0)
+  (symbol (lib_id "jacks:PJ-327A") (at 34.29 85.09 0) (unit 1)
+    (in_bom yes)
+    (property "Reference" "U2" (id 0) (at 36.3474 71.755 0))
+    (property "Value" "PJ-3027F" (id 1) (at 36.3474 74.0664 0))
+    (property "Footprint" "jacks:PJ-327A" (id 2) (at 34.29 87.63 0)
+      (effects (font (size 1.27 1.27)) hide)
+    )
+    (property "Datasheet" "" (id 3) (at 34.29 87.63 0)
       (effects (font (size 1.27 1.27)) hide)
     )
@@
       (reference "U1") (unit 1)
     )
-    (path "/00000000-0000-0000-0000-00005adfde17"
+    (path "/fecea5d8-056f-4fab-9941-7c70f3e31e92"
       (reference "U2") (unit 1)
     )
