File: kicad/BM20_breadboard_adapter/BM20_breadboard_adapter.sch (KiCad schematic (older format))
At the start: 23 parts, among them CON1 CONN_18, CON2 CONN_18, CON3 batt, J1 3.5mmjack, J2 3.5mmjack, J3 USB_B_Micro, SW1 SWITCH_SPST, SW2 SWITCH_SPST, U1 BM20

Commit message: update
Parts:
- removed J1, J2: 3.5mmjack, jacks:3.5mm_stereo_jack_PJ320B_no_up_silkscreen, symbol phonejack:3.5mmjack
- added C10: 10uF/16V, Capacitors_SMD.pretty:C_1206_HandSoldering, symbol c:C
- added C11: 10u/16V, Capacitors_SMD.pretty:C_1206_HandSoldering, symbol c:C
- added C9: 100n, Capacitors_SMD.pretty:C_0805_HandSoldering, symbol c:C
- added J1, J2: PJ-320B, jacks:3.5mm_stereo_jack_PJ320B, symbol jacks:PJ-320B
- added JP1: Jumper_NO_Small, Jumper:SolderJumper-2_P1.3mm_Open_RoundedPad1.0x1.5mm, symbol Device:Jumper_NO_Small
- added U2: PJ-3027F, jacks:PJ-3027F-S, symbol jacks:PJ-3027F
Connections:
- net labels added: AIL, AIR, AUX_DET
- wire segments 144 -> 152
Other:
- moved on the sheet: C1, C2, C3, C4, C5, C6, C7, C8, CON1, CON2, CON3, D1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

Commit message: new module hw
Parts:
- J3: symbol Connector_Specialized:USB_B_Micro -> BM20_breadboard_adapter-rescue:USB_B_Micro-Connector_Specialized
- SW1, SW2: symbol MiscellaneousDevices:SWITCH_SPST -> BM20_breadboard_adapter-rescue:SWITCH_SPST-MiscellaneousDevices
Changed lines of the file:
@@
-EESchema Schematic File Version 4
+EESchema Schematic File Version 5
 LIBS:BM20_breadboard_adapter-cache
-EELAYER 29 0
+EELAYER 30 0
 EELAYER END
 $Descr A4 11693 8268
@@
 GND
 $Comp
-L MiscellaneousDevices:SWITCH_SPST SW1
+L BM20_breadboard_adapter-rescue:SWITCH_SPST-MiscellaneousDevices SW1
 U 1 1 5AA8F0C8
 P 8100 2700
@@
 $EndComp
 $Comp
-L MiscellaneousDevices:SWITCH_SPST SW2
+L BM20_breadboard_adapter-rescue:SWITCH_SPST-MiscellaneousDevices SW2
 U 1 1 5AA97138
 P 8100 3050
@@
 	7500 3050 7800 3050
 $Comp
-L Connector_Specialized:USB_B_Micro J3
+L BM20_breadboard_adapter-rescue:USB_B_Micro-Connector_Specialized J3
 U 1 1 5AA4246D
 P 6600 1350
