File: kicad/arduino_based_cdc_emulator/atmegax8_with_F6188/atmegax8_with_bluetooth.kicad_pcb (KiCad board)
At the start: 2 copper layers, 41.4 x 36.1 mm, 75 parts, among them IC1 ATMEGA88-A, J1 Ant, J2 TMS, J3 TCK, J4 TDO, J5 TDI, P1 CONN_10, P2 SPI, P3 CONN_4, P4 SERIAL, P5 CONN_4, U1 AP1117, U2 F-6188, U3 TL072, U4 MAX809, U5 MAX809, Y1 16MHz

Commit message: rename conn4 to 7805
Parts:
- P5: value CONN_4 -> LM7805
Changed lines of the file:
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@@
       (effects (font (size 1 1) (thickness 0.15)))
     )
-    (fp_text value "CONN_4" (at 0 -3.1) (layer "F.Fab") hide
+    (fp_text value "LM7805" (at 0 -3.1) (layer "F.Fab") hide
       (effects (font (size 1 1) (thickness 0.15)))
     )
