File: kicad/headlight_washer_pump_controler/headlight_washer_pump_controler.kicad_sch (KiCad schematic)
At the start: 17 parts, among them Q1 BSS138, U1 AP1117, U2 ATtiny25-20PU

Commit message: comment about R1
Other:
- note added: "do we need this R1? probably no, it is mosfet ..."
Changed lines of the file:
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@@
+    (effects (font (size 1.27 1.27)) (justify right bottom))
+  )
+  (text "do we need this R1?\nprobably no, \nit is mosfet ... "
+    (at 124.1298 121.1072 0)
     (effects (font (size 1.27 1.27)) (justify right bottom))
   )
