File: kicad/fake_xenon4/fake_xenon4.kicad_sch (KiCad schematic)
At the start: 22 parts, among them J1 Conn_01x03_Male, J2 Conn_01x03_Male, J3 Conn_01x04_Female, J4 Conn_01x04_Female, Q1 BSS138, U1 AP1117, U2 ATtiny25-20PU, U3 Fujitsu_NA-Series, U4 MAX809

Commit message: fake_xenon4_update
Connections:
- net at R6.2, RV1.2, RV1.3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: now also R5.1
Changed lines of the file:
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@@
     (stroke (width 0) (type solid) (color 0 0 0 0))
   )
-  (wire (pts (xy 196.85 92.075) (xy 196.85 109.22))
+  (wire (pts (xy 196.85 91.44) (xy 196.85 109.22))
     (stroke (width 0) (type solid) (color 0 0 0 0))
   )
